File: Tangenta/USB_OTG.kicad_sch (KiCad schematic)
At the start: 0 parts

Commit message: ...
Parts:
- added J11: TYPEC-304-ACP16, USB_TYPEC:USB_TYPEC, symbol USB_TYPEC:TYPEC-304-ACP16
Changed lines of the file:
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@@
 (kicad_sch (version 20230121) (generator eeschema)
   (paper "A4")
+  (symbol (lib_id "USB_TYPEC:TYPEC-304-ACP16") (at 82.55 61.595 180) (unit 1)
+    (in_bom yes) (on_board yes) (dnp no)
+    (property "Reference" "J11" (at 81.28 49.53 0)
+      (effects (font (size 1.27 1.27)))
+    )
+    (property "Value" "TYPEC-304-ACP16" (at 82.55 76.2 0)
+      (effects (font (size 1.27 1.27)))
+    )
+    (property "Footprint" "USB_TYPEC:USB_TYPEC" (at 80.01 47.625 0)
+      (effects (font (size 1.27 1.27) italic) hide)
+    )
+    (property "Datasheet" "https://img.jlc.com/pdf/applyPasteComponent/2022-02-23/91586W/67ceeeb81a9f4c1f8ea00a3628213c3d/USBC16P.pdf" (at 91.44 42.545 0)
+      (effects (font (size 1.27 1.27)) (justify left) hide)
+    )
+    (property "LCSC" "C2982555" (at 80.01 45.085 0)
+      (effects (font (size 1.27 1.27)) hide)
+    )
+    (pin "13")
+    (pin "A1_B12")
+    (pin "A4_B9")
+    (pin "A5")
+    (pin "A6")
+    (pin "A7")
+    (pin "A8")
+    (pin "B1_A12")
+    (pin "B4_A9")
+    (pin "B5")
+    (pin "B6")
+    (pin "B7")
+    (pin "B8")
+    (instances
+      (project "Tangenta"
+        (path "/358d1bcf-7599-4352-8c4d-baa18a5f09e6/e56d8c10-557c-47b7-a4d3-5b3b43580080"
+          (reference "J11") (unit 1)
+        )
+      )
+    )
+  )
 )
