File: Tangenta/USB.kicad_sch (KiCad schematic)
At the start: 0 parts

Commit message: ...
Parts:
- added J12: 907-211A1019D10200, USB_2_CONNECTOR:USB_2_CONNECTOR, symbol USB_2_CONNECTOR:907-211A1019D10200
- added J13: 906-861A2116D10210, USB_VERTICAL:USB_Vertical, symbol USB_VERTICAL:906-861A2116D10210
Changed lines of the file:
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@@
 (kicad_sch (version 20230121) (generator eeschema)
   (paper "A4")
+  (symbol (lib_id "USB_VERTICAL:906-861A2116D10210") (at 122.555 46.355 0) (unit 1)
+    (in_bom yes) (on_board yes) (dnp no) (fields_autoplaced)
+    (property "Reference" "J13" (at 122.555 36.83 0)
+      (effects (font (size 1.27 1.27)))
+    )
+    (property "Value" "906-861A2116D10210" (at 122.555 39.37 0)
+      (effects (font (size 1.27 1.27)))
+    )
+    (property "Footprint" "USB_VERTICAL:USB_Vertical" (at 126.365 61.595 0)
+      (effects (font (size 1.27 1.27) italic) hide)
+    )
+    (property "Datasheet" "https://atta.szlcsc.com/upload/public/pdf/source/20210526/C2763350_E0D561271332FF88E1B9AF264603FE9E.pdf" (at 113.665 64.135 0)
+      (effects (font (size 1.27 1.27)) (justify left) hide)
+    )
+    (property "LCSC" "C2763350" (at 118.745 59.055 0)
+      (effects (font (size 1.27 1.27)) hide)
+    )
+    (pin "1")
+    (pin "2")
+    (pin "3")
+    (pin "4")
+    (pin "5")
+    (pin "6")
+    (instances
+      (project "Tangenta"
+        (path "/358d1bcf-7599-4352-8c4d-baa18a5f09e6/b1871a4d-6a35-44e2-a9a2-9a4af684371d"
+          (reference "J13") (unit 1)
+        )
+      )
+    )
+  )
+  (symbol (lib_id "USB_2_CONNECTOR:907-211A1019D10200") (at 76.2 53.975 0) (unit 1)
+    (in_bom yes) (on_board yes) (dnp no) (fields_autoplaced)
+    (property "Reference" "J12" (at 80.01 51.435 0)
+      (effects (font (size 1.27 1.27)) (justify left))
+    )
+    (property "Value" "907-211A1019D10200" (at 80.01 53.975 0)
+      (effects (font (size 1.27 1.27)) (justify left))
+    )
+    (property "Footprint" "USB_2_CONNECTOR:USB_2_CONNECTOR" (at 99.06 56.515 0)
+      (effects (font (size 1.27 1.27) italic) hide)
+    )
+    (property "Datasheet" "https://item.szlcsc.com/2892241.html" (at 80.01 53.975 0)
+      (effects (font (size 1.27 1.27)) (justify left) hide)
+    )
+    (property "LCSC" "C2763029" (at 71.12 65.405 0)
+      (effects (font (size 1.27 1.27)) hide)
+    )
+    (pin "1")
+    (pin "10")
+    (pin "2")
+    (pin "3")
+    (pin "4")
+    (pin "5")
+    (pin "6")
+    (pin "7")
+    (pin "8")
+    (pin "9")
+    (instances
+      (project "Tangenta"
+        (path "/358d1bcf-7599-4352-8c4d-baa18a5f09e6/b1871a4d-6a35-44e2-a9a2-9a4af684371d"
+          (reference "J12") (unit 1)
+        )
+      )
+    )
+  )
 )

Commit message: Current progress with the USB schematics...
Parts:
- added C1 (x6): 100nF, Capacitor_SMD:C_0402_1005Metric, symbol Device:C_Small
- added FB1: GZ2012D101TF, footprint:L0805, symbol Ferrite_Bead_100:GZ2012D101TF
- added U8: USB2514B-I_M2, USB_HUB:USB_HUB, symbol USB_HUB:USB2514B-I_M2
Connections:
- new net 3V3: C1.2, C1.2, C1.2, FB1.1
- new net 3V3A: C1.2, C1.2, C1.2, FB1.2
- new net GNDREF: C1.1, C1.1, C1.1, C1.1, C1.1, C1.1

Commit message: ...
Parts:
- added C1 (x2): 18pF, Capacitor_SMD:C_0402_1005Metric, symbol Device:C_Small
Changed lines of the file:
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@@
+    )
+  )
+  (symbol (lib_id "Device:C_Small") (at 34.29 159.512 180) (unit 1)
+    (in_bom yes) (on_board yes) (dnp no)
+    (property "Reference" "C1" (at 32.131 157.988 0)
+      (effects (font (size 1.27 1.27)))
+    )
+    (property "Value" "18pF" (at 31.115 161.163 0)
+      (effects (font (size 1.27 1.27)))
+    )
+    (property "Footprint" "Capacitor_SMD:C_0402_1005Metric" (at 34.29 159.512 0)
+      (effects (font (size 1.27 1.27)) hide)
+    )
+    (property "Datasheet" "~" (at 34.29 159.512 0)
+      (effects (font (size 1.27 1.27)) hide)
+    )
+    (pin "1")
+    (pin "2")
+    (instances
+      (project "Tangenta"
+        (path "/358d1bcf-7599-4352-8c4d-baa18a5f09e6/8215796b-9611-4f43-bcc5-319f8414b8a6"
+          (reference "C1") (unit 1)
+        )
+        (path "/358d1bcf-7599-4352-8c4d-baa18a5f09e6/d6c05402-162e-441f-bed8-be7996260fb4"
+          (reference "C9") (unit 1)
+        )
+        (path "/358d1bcf-7599-4352-8c4d-baa18a5f09e6/b1871a4d-6a35-44e2-a9a2-9a4af684371d"
+          (reference "C41") (unit 1)
+        )
+      )
     )
   )
@@
         )
       )
+    )
+  )
+  (symbol (lib_id "Device:C_Small") (at 43.815 159.512 180) (unit 1)
+    (in_bom yes) (on_board yes) (dnp no)
+    (property "Reference" "C1" (at 41.656 157.988 0)
+      (effects (font (size 1.27 1.27)))
+    )
+    (property "Value" "18pF" (at 40.64 161.163 0)
+      (effects (font (size 1.27 1.27)))
+    )
+    (property "Footprint" "Capacitor_SMD:C_0402_1005Metric" (at 43.815 159.512 0)
+      (effects (font (size 1.27 1.27)) hide)
+    )
+    (property "Datasheet" "~" (at 43.815 159.512 0)
+      (effects (font (size 1.27 1.27)) hide)
+    )
+    (pin "1")
+    (pin "2")
+    (instances
+      (project "Tangenta"
+        (path "/358d1bcf-7599-4352-8c4d-baa18a5f09e6/8215796b-9611-4f43-bcc5-319f8414b8a6"
+          (reference "C1") (unit 1)
+        )
+        (path "/358d1bcf-7599-4352-8c4d-baa18a5f09e6/d6c05402-162e-441f-bed8-be7996260fb4"
+          (reference "C9") (unit 1)
+        )
+        (path "/358d1bcf-7599-4352-8c4d-baa18a5f09e6/b1871a4d-6a35-44e2-a9a2-9a4af684371d"
+          (reference "C42") (unit 1)
+        )
+      )

Commit message: Current progress, USB...
Parts:
- added C1 (x3): 100nF, Capacitor_SMD:C_0402_1005Metric, symbol Device:C_Small
- added C1 (x2): 1uF, Capacitor_SMD:C_0402_1005Metric, symbol Device:C_Small
- added R2 (x9): 10k, Resistor_SMD:R_0402_1005Metric, symbol Device:R_Small_US
- added R2: 1M, Resistor_SMD:R_0402_1005Metric, symbol Device:R_Small_US
- added R2: 12k, Resistor_SMD:R_0402_1005Metric, symbol Device:R_Small_US
- added X1: X322524MOB4SI, XTAL_24MHZ:XTAL_24MHZ, symbol XTAL_24MHZ:X322524MOB4SI
Connections:
- net 3V3: now also U8.15 (VDD33), U8.23 (VDD33), U8.27 (VBUS_DET), R2.1, R2.1, R2.1, R2.1, R2.1
- net 3V3A: now also U8.10 (VDDA33), U8.29 (VDDA33), U8.36 (VDDA33), U8.5 (VDDA33)
- net GNDREF: now also C1.1, C1.1, U8.11 (TEST), U8.37 (EP), C1.1, C1.1, C1.1, C1.1, C1.1, R2.1, R2.1, R2.1, R2.1, R2.1, X1.2 (GND), X1.4 (GND)
- net XTALIN: now reaches C1.2
- net XTALIN: now also U8.33 (XTALIN/CLKIN), R2.1, X1.3 (OSC2)
- net USB_D1_N: now reaches U8.1 (USBDM_DN1/PRT_DIS_M1)
- net at U8.13 (OCS_N1): now also R2.2
- net at U8.14 (CRFILT): now also C1.2, C1.2
- net at U8.17 (OCS_N2): now also R2.2
- net at U8.19 (OCS_N3): now also R2.2
- net USB_D1_P: now reaches U8.2 (USBDP_DN1/PRT_DIS_P1)
- net at U8.21 (OCS_N4): now also R2.2
- net at U8.22 (SDA/SMBBATA/NON_REM1): now also R2.2
- net at U8.24 (SCL/SMBCLK/CFG_SEL0): now also R2.2
- net at U8.25 (HS_IND/CFG_SEL1): now also R2.2
- net at U8.26 (RESET_N): now also C1.2, R2.2
- net at U8.28 (SUSP_IND/LOCAL_PWR/NON_REM0): now also R2.2
- net USB_D2_N: now reaches U8.3 (USBDM_DN2/PRT_DIS_M2)
- net USB_U_N: now reaches U8.30 (USBDM_UP)
- net USB_U_P: now reaches U8.31 (USBDP_UP)
- net XTALOUT: now reaches U8.32 (XTALOUT)
- net XTALOUT: now also C1.2, R2.2, X1.1 (OSC1)
- net at U8.34 (PLLFILT): now also C1.2, C1.2
- net at U8.35 (RBIAS): now also R2.2
- net USB_D2_P: now reaches U8.4 (USBDP_DN2/PRT_DIS_P2)
- net USB_D3_N: now reaches U8.6 (USBDM_DN3/PRT_DIS_M3)
- net USB_D3_P: now reaches U8.7 (USBDP_DN3/PRT_DIS_P3)
- net USB_MODEM_N: now reaches U8.8 (USBDM_DN4/PRT_DIS_M4)
- net USB_MODEM_P: now reaches U8.9 (USBDP_DN4/PRT_DIS_P4)
- net CHASSIS: now reaches J13.5 (SHELL)
- net CHASSIS: now also J12.10 (EH), J12.9 (EH), J13.6 (SHELL)
Other:
- moved on the sheet: C1, FB1, J12, J13, U8

Commit message: USB, continued...
Connections:
- net 5V: now also J12.1 (VCC), J12.5 (VCC), J13.4 (VCC)
- net GNDREF: now also J12.4 (GND), J12.8 (GND), J13.1 (GND)
- net USB_D1_N: now also J12.2 (D1-)
- net USB_D1_P: now also J12.3 (D1+)
- net USB_D2_N: now also J12.6 (D2-)
- net USB_D2_P: now also J12.7 (D2+)
- net USB_D3_N: now also J13.3 (D-)
- net USB_D3_P: now also J13.2 (D+)
- net USB_MODEM_N renamed USB_MODEM.N
- net USB_MODEM_P renamed USB_MODEM.P
Changed lines of the file:
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@@
   (junction (at 38.862 173.609) (diameter 0) (color 0 0 0 0)
   )
+  (bus_entry (at 63.5 189.23) (size 2.54 2.54)
+    (stroke (width 0) (type default))
+  )
+  (bus_entry (at 54.61 189.23) (size 2.54 2.54)
+    (stroke (width 0) (type default))
+  )
   (wire (pts (xy 28.702 192.024) (xy 39.497 192.024))
     (stroke (width 0) (type default))
@@
     (stroke (width 0) (type default))
   )
+  (wire (pts (xy 245.745 69.85) (xy 255.905 69.85))
+    (stroke (width 0) (type default))
+  )
+  (wire (pts (xy 245.745 62.23) (xy 255.905 62.23))
+    (stroke (width 0) (type default))
+  )
   (wire (pts (xy 167.6402 67.31) (xy 177.8 67.31))
     (stroke (width 0) (type default))
@@
     (stroke (width 0) (type default))
   )
+  (wire (pts (xy 45.72 186.055) (xy 60.325 186.055))
+    (stroke (width 0) (type default))
+  )
   (wire (pts (xy 53.848 163.83) (xy 55.118 163.83))
     (stroke (width 0) (type default))
@@
     (stroke (width 0) (type default))
   )
+  (wire (pts (xy 245.745 72.39) (xy 255.905 72.39))
+    (stroke (width 0) (type default))
+  )
   (wire (pts (xy 167.6402 90.17) (xy 201.295 90.17))
     (stroke (width 0) (type default))
@@
     (stroke (width 0) (type default))
   )
-  (wire (pts (xy 255.905 69.85) (xy 245.7452 69.85))
-    (stroke (width 0) (type default))
-  )
   (wire (pts (xy 71.12 62.23) (xy 33.655 62.23))
     (stroke (width 0) (type default))
@@
     (stroke (width 0) (type default))
   )
-  (wire (pts (xy 255.905 88.265) (xy 245.7452 88.265))
+  (wire (pts (xy 245.745 57.15) (xy 255.905 57.15))
     (stroke (width 0) (type default))
   )
@@
     (stroke (width 0) (type default))
   )
+  (wire (pts (xy 245.745 54.61) (xy 255.905 54.61))
+    (stroke (width 0) (type default))
+  )
   (wire (pts (xy 70.104 173.609) (xy 70.104 171.45))
     (stroke (width 0) (type default))
   )
+  (wire (pts (xy 245.745 95.885) (xy 255.905 95.885))
+    (stroke (width 0) (type default))
+  )
   (wire (pts (xy 167.6402 100.33) (xy 177.8 100.33))
     (stroke (width 0) (type default))
@@
     (stroke (width 0) (type default))
   )
-  (wire (pts (xy 255.905 72.39) (xy 245.7452 72.39))
-    (stroke (width 0) (type default))
-  )
   (wire (pts (xy 206.375 97.79) (xy 206.375 96.52))
     (stroke (width 0) (type default))
@@
     (stroke (width 0) (type default))
   )
-  (wire (pts (xy 255.905 57.15) (xy 245.7452 57.15))
-    (stroke (width 0) (type default))
-  )
-  (wire (pts (xy 255.905 67.31) (xy 245.7452 67.31))
+  (wire (pts (xy 63.5 189.23) (xy 60.325 186.055))
     (stroke (width 0) (type default))
   )
@@
     (stroke (width 0) (type default))
   )
+  (bus (pts (xy 57.15 191.77) (xy 66.04 191.77))
+    (stroke (width 0) (type default))
+  )
   (wire (pts (xy 63.5 80.01) (xy 71.12 80.01))
     (stroke (width 0) (type default))
@@
     (stroke (width 0) (type default))
   )
+  (wire (pts (xy 245.745 88.265) (xy 255.905 88.265))
+    (stroke (width 0) (type default))
+  )
   (wire (pts (xy 63.5 77.47) (xy 71.12 77.47))
     (stroke (width 0) (type default))
@@
     (stroke (width 0) (type default))
   )
+  (wire (pts (xy 245.745 59.69) (xy 255.905 59.69))
+    (stroke (width 0) (type default))
+  )
   (wire (pts (xy 43.815 82.55) (xy 71.12 82.55))
     (stroke (width 0) (type default))
@@
     (stroke (width 0) (type default))
   )
-  (wire (pts (xy 255.905 64.77) (xy 245.7452 64.77))
-    (stroke (width 0) (type default))
-  )
   (wire (pts (xy 167.6402 87.63) (xy 180.975 87.63))
     (stroke (width 0) (type default))
@@
     (stroke (width 0) (type default))
   )
+  (wire (pts (xy 245.745 67.31) (xy 255.905 67.31))
+    (stroke (width 0) (type default))
+  )
   (wire (pts (xy 114.3 163.83) (xy 120.65 163.83))
     (stroke (width 0) (type default))
@@
     (stroke (width 0) (type default))
   )
+  (wire (pts (xy 245.745 90.805) (xy 255.905 90.805))
+    (stroke (width 0) (type default))
+  )
   (wire (pts (xy 31.369 163.83) (xy 31.369 166.37))
     (stroke (width 0) (type default))
@@
     (stroke (width 0) (type default))
   )
-  (wire (pts (xy 255.905 90.805) (xy 245.7452 90.805))
-    (stroke (width 0) (type default))
-  )
-  (wire (pts (xy 255.905 62.23) (xy 245.7452 62.23))
-    (stroke (width 0) (type default))
-  )
   (wire (pts (xy 167.6402 95.25) (xy 177.8 95.25))
     (stroke (width 0) (type default))
@@
     (stroke (width 0) (type default))
   )
-  (wire (pts (xy 255.905 54.61) (xy 245.7452 54.61))
-    (stroke (width 0) (type default))
-  )
   (wire (pts (xy 28.575 90.17) (xy 43.815 90.17))
     (stroke (width 0) (type default))
   )
-  (wire (pts (xy 255.905 59.69) (xy 245.7452 59.69))
+  (bus (pts (xy 66.04 191.77) (xy 71.755 191.77))
     (stroke (width 0) (type default))
   )
@@
     (stroke (width 0) (type default))
   )
+  (wire (pts (xy 245.745 93.345) (xy 255.905 93.345))
+    (stroke (width 0) (type default))
+  )
   (wire (pts (xy 167.6402 64.77) (xy 177.8 64.77))
     (stroke (width 0) (type default))
@@
     (stroke (width 0) (type default))
   )
-  (wire (pts (xy 255.905 95.885) (xy 245.7452 95.885))
-    (stroke (width 0) (type default))
-  )
   (wire (pts (xy 60.325 69.85) (xy 71.12 69.85))
     (stroke (width 0) (type default))
@@
     (stroke (width 0) (type default))
   )
+  (wire (pts (xy 245.745 64.77) (xy 255.905 64.77))
+    (stroke (width 0) (type default))
+  )
   (wire (pts (xy 167.6402 92.71) (xy 177.8 92.71))
     (stroke (width 0) (type default))
@@
     (stroke (width 0) (type default))
   )
-  (wire (pts (xy 255.905 93.345) (xy 245.7452 93.345))
+  (wire (pts (xy 45.72 189.23) (xy 54.61 189.23))
     (stroke (width 0) (type default))
   )
@@
     (effects (font (size 1.27 1.27)) (justify right bottom))
   )
+  (label "USB_MODEM.P" (at 189.23 77.47 180) (fields_autoplaced)
+    (effects (font (size 1.27 1.27)) (justify right bottom))
+  )
   (label "3V3A" (at 63.5 57.15 0) (fields_autoplaced)
     (effects (font (size 1.27 1.27)) (justify left bottom))
   )
+  (label "USB_MODEM.N" (at 189.23 74.93 180) (fields_autoplaced)
+    (effects (font (size 1.27 1.27)) (justify right bottom))
+  )
   (label "CHASSIS" (at 279.4 46.99 180) (fields_autoplaced)
     (effects (font (size 1.27 1.27)) (justify right bottom))
@@
     (effects (font (size 1.27 1.27)) (justify left bottom))
   )
-  (label "USB_D4_N" (at 177.8 74.93 180) (fields_autoplaced)
-    (effects (font (size 1.27 1.27)) (justify right bottom))
-  )
   (label "GND" (at 245.745 72.39 0) (fields_autoplaced)
     (effects (font (size 1.27 1.27)) (justify left bottom))
@@
     (effects (font (size 1.27 1.27)) (justify left bottom))
   )
-  (label "USB_D4_P" (at 177.8 77.47 180) (fields_autoplaced)
-    (effects (font (size 1.27 1.27)) (justify right bottom))
-  )
   (label "USB_U_P" (at 60.325 69.85 0) (fields_autoplaced)
     (effects (font (size 1.27 1.27)) (justify left bottom))
@@
     (effects (font (size 1.27 1.27)) (justify left bottom))
   )
+  (label "USB_MODEM.N" (at 45.72 189.23 0) (fields_autoplaced)
+    (effects (font (size 1.27 1.27)) (justify left bottom))
+  )
   (label "3V3" (at 28.575 97.79 0) (fields_autoplaced)
     (effects (font (size 1.27 1.27)) (justify left bottom))
@@
     (effects (font (size 1.27 1.27)) (justify right bottom))
   )
+  (label "USB_MODEM.P" (at 45.72 186.055 0) (fields_autoplaced)
+    (effects (font (size 1.27 1.27)) (justify left bottom))
+  )
   (label "USB_D1_P" (at 245.745 59.69 0) (fields_autoplaced)
     (effects (font (size 1.27 1.27)) (justify left bottom))
@@
   (label "XTALOUT" (at 120.65 163.83 180) (fields_autoplaced)
     (effects (font (size 1.27 1.27)) (justify right bottom))
-  )
-  (hierarchical_label "USB_MODEM_N" (shape output) (at 189.23 74.93 0) (fields_autoplaced)
-    (effects (font (size 1.27 1.27)) (justify left))
   )
   (hierarchical_label "GND" (shape bidirectional) (at 29.464 182.88 180) (fields_autoplaced)
     (effects (font (size 1.27 1.27)) (justify right))
   )
+  (hierarchical_label "USB_MODEM{P N}" (shape output) (at 71.755 191.77 0) (fields_autoplaced)
+    (effects (font (size 1.27 1.27)) (justify left))
+  )
   (hierarchical_label "5V" (shape input) (at 28.702 187.579 180) (fields_autoplaced)
     (effects (font (size 1.27 1.27)) (justify right))
@@
     (effects (font (size 1.27 1.27)) (justify right))
   )
-  (hierarchical_label "USB_MODEM_P" (shape output) (at 189.23 77.47 0) (fields_autoplaced)
-    (effects (font (size 1.27 1.27)) (justify left))
-  )
   (symbol (lib_id "Device:R_Small_US") (at 184.15 97.79 270) (mirror x) (unit 1)
