File: Tangenta/USB.kicad_sch (KiCad schematic)
At the start: 29 parts, among them J4 906-151A1058D10200, J5 907-211A1019D10200, U14 USB2514B-I_M2, X1 X322524MOB4SI

Commit message: Removing component association with previous project (local) libraries.
Parts:
- C49, C50, C51, C52, C53, C54, C55, C57, C58, C60, C61, C62, C63: symbol CholaSymbolsPrjLib:C_Small -> C_Small:C_Small
- C56, C59: footprint CholaFootprintsPrjLib:CAP_L5 -> CAP_L5:CAP_L5; symbol CholaSymbolsPrjLib:16CE47FSS -> 16CE47FSS:16CE47FSS
- FB1: footprint CholaFootprintsPrjLib:Ferrite_Bead_100 -> Ferrite_Bead_100:Ferrite_Bead_100; symbol CholaSymbolsPrjLib:GZ2012D101TF -> GZ2012D101TF:GZ2012D101TF
- J4: footprint CholaFootprintsPrjLib:USB_VERTICAL_BLUE -> USB_VERTICAL_BLUE:USB_VERTICAL_BLUE; symbol CholaSymbolsPrjLib:906-151A1058D10200 -> 906-151A1058D10200:906-151A1058D10200
- J5: footprint CholaFootprintsPrjLib:USB_2_CONNECTOR -> USB_2_CONNECTOR:USB_2_CONNECTOR; symbol CholaSymbolsPrjLib:907-211A1019D10200 -> 907-211A1019D10200:907-211A1019D10200
- R33, R34, R35, R36, R37, R38, R39, R40, R41: symbol CholaSymbolsPrjLib:R_Small_US -> R_Small_US:R_Small_US
- U14: footprint CholaFootprintsPrjLib:USB_HUB -> USB_HUB:USB_HUB; symbol CholaSymbolsPrjLib:USB2514B-I_M2 -> USB2514B-I_M2:USB2514B-I_M2
- X1: footprint CholaFootprintsPrjLib:XTAL_24MHZ -> XTAL_24MHZ:XTAL_24MHZ; symbol CholaSymbolsPrjLib:X322524MOB4SI -> X322524MOB4SI:X322524MOB4SI
Changed lines of the file:
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@@
 	)
 	(symbol
-		(lib_id "CholaSymbolsPrjLib:R_Small_US")
+		(lib_id "R_Small_US:R_Small_US")
 		(at 184.15 97.79 270)
 		(mirror x)
@@
 	)
 	(symbol
-		(lib_id "CholaSymbolsPrjLib:C_Small")
+		(lib_id "C_Small:C_Small")
 		(at 62.611 168.91 180)
 		(unit 1)
@@
 	)
 	(symbol
-		(lib_id "CholaSymbolsPrjLib:C_Small")
+		(lib_id "C_Small:C_Small")
 		(at 38.862 168.91 180)
 		(unit 1)
@@
 	)
 	(symbol
-		(lib_id "CholaSymbolsPrjLib:C_Small")
+		(lib_id "C_Small:C_Small")
 		(at 55.118 168.91 180)
 		(unit 1)
@@
 	)
 	(symbol
-		(lib_id "CholaSymbolsPrjLib:X322524MOB4SI")
+		(lib_id "X322524MOB4SI:X322524MOB4SI")
 		(at 104.775 166.37 180)
 		(unit 1)
@@
 			)
 		)
-		(property "Footprint" "CholaFootprintsPrjLib:XTAL_24MHZ"
+		(property "Footprint" "XTAL_24MHZ:XTAL_24MHZ"
 			(at 113.411 150.114 0)
 			(effects
@@
 	)
 	(symbol
-		(lib_id "CholaSymbolsPrjLib:C_Small")
+		(lib_id "C_Small:C_Small")
 		(at 46.355 168.91 180)
 		(unit 1)
@@
 	)
 	(symbol
-		(lib_id "CholaSymbolsPrjLib:C_Small")
+		(lib_id "C_Small:C_Small")
 		(at 95.25 180.34 180)
 		(unit 1)
@@
 	)
 	(symbol
-		(lib_id "CholaSymbolsPrjLib:C_Small")
+		(lib_id "C_Small:C_Small")
 		(at 33.655 66.04 180)
 		(unit 1)
@@
 	)
 	(symbol
-		(lib_id "CholaSymbolsPrjLib:R_Small_US")
+		(lib_id "R_Small_US:R_Small_US")
 		(at 60.96 77.47 90)
 		(unit 1)
@@
 	)
 	(symbol
-		(lib_id "CholaSymbolsPrjLib:USB2514B-I_M2")
+		(lib_id "USB2514B-I_M2:USB2514B-I_M2")
 		(at 118.1101 76.2 0)
 		(mirror y)
@@
 			)
 		)
-		(property "Footprint" "CholaFootprintsPrjLib:USB_HUB"
+		(property "Footprint" "USB_HUB:USB_HUB"
 			(at 156.2101 115.57 0)
 			(effects
@@
 	)
 	(symbol
-		(lib_id "CholaSymbolsPrjLib:R_Small_US")
+		(lib_id "R_Small_US:R_Small_US")
 		(at 60.96 100.33 90)
 		(unit 1)
@@
 	)
 	(symbol
-		(lib_id "CholaSymbolsPrjLib:C_Small")
+		(lib_id "C_Small:C_Small")
 		(at 206.375 93.98 180)
 		(unit 1)
@@
 	)
 	(symbol
-		(lib_id "CholaSymbolsPrjLib:R_Small_US")
+		(lib_id "R_Small_US:R_Small_US")
 		(at 60.96 95.25 90)
 		(unit 1)
@@
 	)
 	(symbol
-		(lib_id "CholaSymbolsPrjLib:907-211A1019D10200")
+		(lib_id "907-211A1019D10200:907-211A1019D10200")
 		(at 268.605 64.77 0)
 		(unit 1)
@@
 			)
 		)
-		(property "Footprint" "CholaFootprintsPrjLib:USB_2_CONNECTOR"
+		(property "Footprint" "USB_2_CONNECTOR:USB_2_CONNECTOR"
 			(at 291.465 67.31 0)
 			(effects
@@
 	)
 	(symbol
-		(lib_id "CholaSymbolsPrjLib:R_Small_US")
+		(lib_id "R_Small_US:R_Small_US")
 		(at 183.515 87.63 270)
 		(mirror x)
@@
 	)
 	(symbol
-		(lib_id "CholaSymbolsPrjLib:C_Small")
+		(lib_id "C_Small:C_Small")
 		(at 114.3 180.34 180)
 		(unit 1)
@@
 	)
 	(symbol
-		(lib_id "CholaSymbolsPrjLib:GZ2012D101TF")
+		(lib_id "GZ2012D101TF:GZ2012D101TF")
 		(at 50.673 163.83 0)
 		(unit 1)
@@
 			)
 		)
-		(property "Footprint" "CholaFootprintsPrjLib:Ferrite_Bead_100"
+		(property "Footprint" "Ferrite_Bead_100:Ferrite_Bead_100"
 			(at 63.246 173.863 0)
 			(effects
@@
 	)
 	(symbol
-		(lib_id "CholaSymbolsPrjLib:906-151A1058D10200")
+		(lib_id "906-151A1058D10200:906-151A1058D10200")
 		(at 266.7 93.98 0)
 		(unit 1)
@@
 			)
 		)
-		(property "Footprint" "CholaFootprintsPrjLib:USB_VERTICAL_BLUE"
+		(property "Footprint" "USB_VERTICAL_BLUE:USB_VERTICAL_BLUE"
 			(at 267.589 108.585 0)
 			(effects
@@
 	)
 	(symbol
-		(lib_id "CholaSymbolsPrjLib:16CE47FSS")
+		(lib_id "16CE47FSS:16CE47FSS")
 		(at 62.103 187.071 0)
 		(unit 1)
@@
 			)
 		)
-		(property "Footprint" "CholaFootprintsPrjLib:CAP_L5"
+		(property "Footprint" "CAP_L5:CAP_L5"
 			(at 60.833 204.851 0)
 			(effects
@@
 	)
 	(symbol
-		(lib_id "CholaSymbolsPrjLib:R_Small_US")
+		(lib_id "R_Small_US:R_Small_US")
 		(at 105.41 177.8 90)
 		(unit 1)
@@
 	(symbol
 		(lib_name "16CE47FSS_1")
-		(lib_id "CholaSymbolsPrjLib:16CE47FSS")
+		(lib_id "16CE47FSS:16CE47FSS")
 		(at 70.104 187.071 0)
 		(unit 1)
@@
 			)
 		)
-		(property "Footprint" "CholaFootprintsPrjLib:CAP_L5"
+		(property "Footprint" "CAP_L5:CAP_L5"
 			(at 68.834 204.851 0)
 			(effects
@@
 	)
 	(symbol
-		(lib_id "CholaSymbolsPrjLib:C_Small")
+		(lib_id "C_Small:C_Small")
 		(at 201.295 93.98 180)
 		(unit 1)
@@
 	)
 	(symbol
-		(lib_id "CholaSymbolsPrjLib:C_Small")
+		(lib_id "C_Small:C_Small")
 		(at 70.104 168.91 180)
 		(unit 1)
@@
 	)
 	(symbol
-		(lib_id "CholaSymbolsPrjLib:C_Small")
+		(lib_id "C_Small:C_Small")
 		(at 43.815 86.36 180)
 		(unit 1)
@@
 	)
 	(symbol
-		(lib_id "CholaSymbolsPrjLib:C_Small")
+		(lib_id "C_Small:C_Small")
 		(at 28.575 66.04 180)
 		(unit 1)
@@
 	)
 	(symbol
-		(lib_id "CholaSymbolsPrjLib:R_Small_US")
+		(lib_id "R_Small_US:R_Small_US")
 		(at 60.96 59.69 90)
 		(unit 1)
@@
 	)
 	(symbol
-		(lib_id "CholaSymbolsPrjLib:R_Small_US")
+		(lib_id "R_Small_US:R_Small_US")
 		(at 60.96 85.09 90)
 		(unit 1)
@@
 	)
 	(symbol
-		(lib_id "CholaSymbolsPrjLib:R_Small_US")
+		(lib_id "R_Small_US:R_Small_US")
 		(at 40.005 82.55 90)
 		(unit 1)
@@
 	)
 	(symbol
-		(lib_id "CholaSymbolsPrjLib:C_Small")
+		(lib_id "C_Small:C_Small")
 		(at 31.369 168.91 180)
 		(unit 1)
