File: Tangenta/PCIExpress.kicad_sch (KiCad schematic)
At the start: 0 parts

Commit message: ...
Other:
- sheet PCIE_Slot_1 ports: added 3V3, 3V3_STANDBY, GND; removed none
- sheet PCIE_Slot_2 ports: added 3V3, 3V3_STANDBY, GND; removed none
- sheet PCIE_Slot_3 ports: added 3V3, 3V3_STANDBY, GND; removed none
Changed lines of the file:
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@@
     (stroke (width 0) (type default))
   )
-  (wire (pts (xy 215.9 194.945) (xy 220.98 194.945))
+  (wire (pts (xy 215.9 195.58) (xy 223.52 195.58))
     (stroke (width 0) (type default))
   )
@@
     (stroke (width 0) (type default))
   )
+  (wire (pts (xy 215.9 95.25) (xy 223.52 95.25))
+    (stroke (width 0) (type default))
+  )
   (wire (pts (xy 226.06 115.57) (xy 226.06 166.37))
     (stroke (width 0) (type default))
   )
+  (wire (pts (xy 215.9 146.05) (xy 223.52 146.05))
+    (stroke (width 0) (type default))
+  )
   (wire (pts (xy 227.965 168.91) (xy 227.965 118.11))
     (stroke (width 0) (type default))
@@
     (stroke (width 0) (type default))
   )
+  (wire (pts (xy 215.9 97.79) (xy 223.52 97.79))
+    (stroke (width 0) (type default))
+  )
+  (wire (pts (xy 215.9 198.12) (xy 223.52 198.12))
+    (stroke (width 0) (type default))
+  )
   (wire (pts (xy 101.6 120.015) (xy 124.46 120.015))
     (stroke (width 0) (type default))
@@
     (stroke (width 0) (type default))
   )
+  (wire (pts (xy 215.9 138.43) (xy 223.52 138.43))
+    (stroke (width 0) (type default))
+  )
   (wire (pts (xy 101.6 137.795) (xy 124.46 137.795))
     (stroke (width 0) (type default))
@@
     (stroke (width 0) (type default))
   )
+  (wire (pts (xy 215.9 193.04) (xy 223.52 193.04))
+    (stroke (width 0) (type default))
+  )
   (bus (pts (xy 57.785 126.365) (xy 64.135 126.365))
     (stroke (width 0) (type default))
@@
     (stroke (width 0) (type default))
   )
-  (wire (pts (xy 215.9 95.885) (xy 220.98 95.885))
+  (wire (pts (xy 215.9 92.71) (xy 223.52 92.71))
     (stroke (width 0) (type default))
   )
@@
     (stroke (width 0) (type default))
   )
+  (wire (pts (xy 215.9 140.97) (xy 223.52 140.97))
+    (stroke (width 0) (type default))
+  )
   (wire (pts (xy 101.6 132.08) (xy 124.46 132.08))
     (stroke (width 0) (type default))
@@
     (stroke (width 0) (type default))
   )
+  (wire (pts (xy 215.9 90.17) (xy 223.52 90.17))
+    (stroke (width 0) (type default))
+  )
   (wire (pts (xy 176.53 184.15) (xy 187.96 184.15))
     (stroke (width 0) (type default))
@@
     (stroke (width 0) (type default))
   )
-  (wire (pts (xy 215.9 144.145) (xy 220.98 144.145))
+  (wire (pts (xy 215.9 143.51) (xy 223.52 143.51))
     (stroke (width 0) (type default))
   )
@@
     (stroke (width 0) (type default))
   )
+  (wire (pts (xy 215.9 190.5) (xy 223.52 190.5))
+    (stroke (width 0) (type default))
+  )
   (wire (pts (xy 176.53 87.63) (xy 187.96 87.63))
     (stroke (width 0) (type default))
@@
     (effects (font (size 1.27 1.27)) (justify left bottom))
   )
-  (label "12V" (at 220.98 144.145 180) (fields_autoplaced)
+  (label "12V" (at 223.52 143.51 180) (fields_autoplaced)
     (effects (font (size 1.27 1.27)) (justify right bottom))
   )
@@
     (effects (font (size 1.27 1.27)) (justify right bottom))
   )
+  (label "GND" (at 223.52 97.79 180) (fields_autoplaced)
+    (effects (font (size 1.27 1.27)) (justify right bottom))
+  )
+  (label "GND" (at 223.52 198.12 180) (fields_autoplaced)
+    (effects (font (size 1.27 1.27)) (justify right bottom))
+  )
   (label "PCIE_X1_JTAG.TCK" (at 85.09 160.02 180) (fields_autoplaced)
     (effects (font (size 1.27 1.27)) (justify right bottom))
@@
     (effects (font (size 1.27 1.27)) (justify right bottom))
   )
+  (label "3V3" (at 223.52 190.5 180) (fields_autoplaced)
+    (effects (font (size 1.27 1.27)) (justify right bottom))
+  )
+  (label "3V3" (at 223.52 90.17 180) (fields_autoplaced)
+    (effects (font (size 1.27 1.27)) (justify right bottom))
+  )
   (label "PCIE_X1_CLK.P" (at 101.6 110.49 0) (fields_autoplaced)
     (effects (font (size 1.27 1.27)) (justify left bottom))
@@
     (effects (font (size 1.27 1.27)) (justify right bottom))
   )
+  (label "GND" (at 223.52 146.05 180) (fields_autoplaced)
+    (effects (font (size 1.27 1.27)) (justify right bottom))
+  )
   (label "PCIE_X1_DATA.RX_P" (at 85.09 107.95 180) (fields_autoplaced)
     (effects (font (size 1.27 1.27)) (justify right bottom))
@@
     (effects (font (size 1.27 1.27)) (justify right bottom))
   )
-  (label "12V" (at 220.98 95.885 180) (fields_autoplaced)
+  (label "3V3SB" (at 223.52 140.97 180) (fields_autoplaced)
+    (effects (font (size 1.27 1.27)) (justify right bottom))
+  )
+  (label "3V3" (at 223.52 138.43 180) (fields_autoplaced)
+    (effects (font (size 1.27 1.27)) (justify right bottom))
+  )
+  (label "12V" (at 223.52 95.25 180) (fields_autoplaced)
     (effects (font (size 1.27 1.27)) (justify right bottom))
   )
@@
     (effects (font (size 1.27 1.27)) (justify left bottom))
   )
-  (label "12V" (at 220.98 194.945 180) (fields_autoplaced)
+  (label "12V" (at 223.52 195.58 180) (fields_autoplaced)
     (effects (font (size 1.27 1.27)) (justify right bottom))
   )
@@
     (effects (font (size 1.27 1.27)) (justify left bottom))
   )
+  (label "3V3SB" (at 223.52 193.04 180) (fields_autoplaced)
+    (effects (font (size 1.27 1.27)) (justify right bottom))
+  )
   (label "PCIE_X1_CTRL.nRST" (at 86.36 130.81 180) (fields_autoplaced)
     (effects (font (size 1.27 1.27)) (justify right bottom))
@@
     (effects (font (size 1.27 1.27)) (justify right bottom))
   )
+  (label "3V3SB" (at 223.52 92.71 180) (fields_autoplaced)
+    (effects (font (size 1.27 1.27)) (justify right bottom))
+  )
   (label "PCIE_X1_JTAG.TRST" (at 101.6 147.955 0) (fields_autoplaced)
     (effects (font (size 1.27 1.27)) (justify left bottom))
@@
     (effects (font (size 1.27 1.27)) (justify right))
   )
-  (sheet (at 124.46 66.04) (size 52.07 132.08) (fields_autoplaced)
+  (sheet (at 124.46 66.04) (size 52.07 133.35) (fields_autoplaced)
     (stroke (width 0.1524) (type solid))
     (fill (color 0 0 0 0.0000))
@@
       (effects (font (size 1.27 1.27)) (justify left bottom))
     )
-    (property "Sheetfile" "PCIE_Switch.kicad_sch" (at 124.46 198.7046 0)
+    (property "Sheetfile" "PCIE_Switch.kicad_sch" (at 124.46 199.9746 0)
       (effects (font (size 1.27 1.27)) (justify left top))
     )
@@
       (effects (font (size 1.27 1.27)) (justify right))
     )
-    (pin "12V" input (at 215.9 95.885 0)
+    (pin "12V" input (at 215.9 95.25 0)
       (effects (font (size 1.27 1.27)) (justify right))
     )
@@
     )
     (pin "PCIE1_SMBCLK" input (at 215.9 69.85 0)
+      (effects (font (size 1.27 1.27)) (justify right))
+    )
+    (pin "3V3_STANDBY" input (at 215.9 92.71 0)
+      (effects (font (size 1.27 1.27)) (justify right))
+    )
+    (pin "3V3" input (at 215.9 90.17 0)
+      (effects (font (size 1.27 1.27)) (justify right))
+    )
+    (pin "GND" bidirectional (at 215.9 97.79 0)
       (effects (font (size 1.27 1.27)) (justify right))
     )
@@
       (effects (font (size 1.27 1.27)) (justify right))
     )
-    (pin "12V" input (at 215.9 144.145 0)
+    (pin "12V" input (at 215.9 143.51 0)
       (effects (font (size 1.27 1.27)) (justify right))
     )
@@
     )
     (pin "PCIE2_SMBCLK" input (at 215.9 118.11 0)
+      (effects (font (size 1.27 1.27)) (justify right))
+    )
+    (pin "3V3" input (at 215.9 138.43 0)
+      (effects (font (size 1.27 1.27)) (justify right))
+    )
+    (pin "3V3_STANDBY" input (at 215.9 140.97 0)
+      (effects (font (size 1.27 1.27)) (justify right))
+    )
+    (pin "GND" bidirectional (at 215.9 146.05 0)
       (effects (font (size 1.27 1.27)) (justify right))
     )
@@
     )
   )
-  (sheet (at 187.96 165.1) (size 27.94 33.02) (fields_autoplaced)
+  (sheet (at 187.96 165.1) (size 27.94 34.29) (fields_autoplaced)
     (stroke (width 0.1524) (type solid))
     (fill (color 0 0 0 0.0000))
@@
       (effects (font (size 1.27 1.27)) (justify left bottom))
     )
-    (property "Sheetfile" "PCIE_Slot_3.kicad_sch" (at 187.96 198.7046 0)
+    (property "Sheetfile" "PCIE_Slot_3.kicad_sch" (at 187.96 199.9746 0)
       (effects (font (size 1.27 1.27)) (justify left top))
     )
@@
       (effects (font (size 1.27 1.27)) (justify right))
     )
-    (pin "12V" input (at 215.9 194.945 0)
+    (pin "12V" input (at 215.9 195.58 0)
       (effects (font (size 1.27 1.27)) (justify right))
     )
@@
       (effects (font (size 1.27 1.27)) (justify right))
     )
+    (pin "3V3_STANDBY" input (at 215.9 193.04 0)
+      (effects (font (size 1.27 1.27)) (justify right))
+    )
+    (pin "GND" bidirectional (at 215.9 198.12 0)
+      (effects (font (size 1.27 1.27)) (justify right))
+    )
+    (pin "3V3" input (at 215.9 190.5 0)
+      (effects (font (size 1.27 1.27)) (justify right))
+    )

Commit message: Schematic improvements.
Other:
- sheet PCIE_Switch ports: added none; removed PCIE_SW_TCK, PCIE_SW_TDI, PCIE_SW_TDO, PCIE_SW_TMS, PCIE_SW_TRST_L
Changed lines of the file:
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@@
   (junction (at 229.87 71.755) (diameter 0) (color 0 0 0 0)
   )
-  (bus_entry (at 64.135 165.735) (size 2.54 -2.54)
-    (stroke (width 0) (type default))
-  )
   (bus_entry (at 64.135 136.525) (size 2.54 -2.54)
     (stroke (width 0) (type default))
   )
-  (bus_entry (at 64.135 162.56) (size 2.54 -2.54)
-    (stroke (width 0) (type default))
-  )
-  (bus_entry (at 64.135 175.26) (size 2.54 -2.54)
-    (stroke (width 0) (type default))
-  )
   (bus_entry (at 64.135 113.665) (size 2.54 -2.54)
     (stroke (width 0) (type default))
   )
-  (bus_entry (at 64.135 172.085) (size 2.54 -2.54)
-    (stroke (width 0) (type default))
-  )
   (bus_entry (at 64.135 116.84) (size 2.54 -2.54)
     (stroke (width 0) (type default))
@@
     (stroke (width 0) (type default))
   )
-  (bus_entry (at 64.135 168.91) (size 2.54 -2.54)
-    (stroke (width 0) (type default))
-  )
   (bus_entry (at 64.135 110.49) (size 2.54 -2.54)
     (stroke (width 0) (type default))
@@
     (stroke (width 0) (type default))
   )
-  (bus (pts (xy 64.135 165.735) (xy 64.135 168.91))
-    (stroke (width 0) (type default))
-  )
   (wire (pts (xy 176.53 81.28) (xy 187.96 81.28))
     (stroke (width 0) (type default))
@@
     (stroke (width 0) (type default))
   )
-  (wire (pts (xy 101.6 145.415) (xy 124.46 145.415))
-    (stroke (width 0) (type default))
-  )
   (wire (pts (xy 215.9 138.43) (xy 223.52 138.43))
     (stroke (width 0) (type default))
   )
-  (wire (pts (xy 101.6 137.795) (xy 124.46 137.795))
-    (stroke (width 0) (type default))
-  )
-  (wire (pts (xy 101.6 147.955) (xy 124.46 147.955))
-    (stroke (width 0) (type default))
-  )
   (wire (pts (xy 226.06 67.31) (xy 215.9 67.31))
     (stroke (width 0) (type default))
@@
     (stroke (width 0) (type default))
   )
-  (wire (pts (xy 66.675 160.02) (xy 85.09 160.02))
-    (stroke (width 0) (type default))
-  )
   (wire (pts (xy 124.46 76.2) (xy 101.6 76.2))
     (stroke (width 0) (type default))
@@
     (stroke (width 0) (type default))
   )
-  (wire (pts (xy 66.675 169.545) (xy 85.09 169.545))
-    (stroke (width 0) (type default))
-  )
   (wire (pts (xy 66.675 144.145) (xy 85.09 144.145))
     (stroke (width 0) (type default))
@@
     (stroke (width 0) (type default))
   )
-  (wire (pts (xy 101.6 142.875) (xy 124.46 142.875))
-    (stroke (width 0) (type default))
-  )
   (wire (pts (xy 101.6 117.475) (xy 124.46 117.475))
     (stroke (width 0) (type default))
   )
-  (bus (pts (xy 64.135 172.085) (xy 64.135 175.26))
-    (stroke (width 0) (type default))
-  )
   (wire (pts (xy 227.965 118.11) (xy 215.9 118.11))
     (stroke (width 0) (type default))
@@
     (stroke (width 0) (type default))
   )
-  (wire (pts (xy 66.675 166.37) (xy 85.09 166.37))
-    (stroke (width 0) (type default))
-  )
   (wire (pts (xy 176.53 74.93) (xy 187.96 74.93))
     (stroke (width 0) (type default))
@@
     (stroke (width 0) (type default))
   )
-  (bus (pts (xy 57.785 178.435) (xy 64.135 178.435))
-    (stroke (width 0) (type default))
-  )
   (wire (pts (xy 101.6 125.095) (xy 124.46 125.095))
     (stroke (width 0) (type default))
@@
     (stroke (width 0) (type default))
   )
-  (wire (pts (xy 101.6 140.335) (xy 124.46 140.335))
-    (stroke (width 0) (type default))
-  )
-  (wire (pts (xy 66.675 172.72) (xy 85.09 172.72))
-    (stroke (width 0) (type default))
-  )
   (wire (pts (xy 215.9 190.5) (xy 223.52 190.5))
     (stroke (width 0) (type default))
@@
     (stroke (width 0) (type default))
   )
-  (wire (pts (xy 66.675 163.195) (xy 85.09 163.195))
-    (stroke (width 0) (type default))
-  )
   (wire (pts (xy 229.87 120.015) (xy 215.9 120.015))
     (stroke (width 0) (type default))
@@
     (stroke (width 0) (type default))
   )
-  (bus (pts (xy 64.135 175.26) (xy 64.135 178.435))
-    (stroke (width 0) (type default))
-  )
   (wire (pts (xy 229.87 71.755) (xy 215.9 71.755))
     (stroke (width 0) (type default))
@@
     (stroke (width 0) (type default))
   )
-  (bus (pts (xy 64.135 162.56) (xy 64.135 165.735))
-    (stroke (width 0) (type default))
-  )
-  (bus (pts (xy 64.135 168.91) (xy 64.135 172.085))
-    (stroke (width 0) (type default))
-  )
   (wire (pts (xy 124.46 68.58) (xy 101.6 68.58))
     (stroke (width 0) (type default))
@@
     (effects (font (size 1.27 1.27)) (justify right bottom))
   )
-  (label "PCIE_X1_JTAG.TCK" (at 85.09 160.02 180) (fields_autoplaced)
-    (effects (font (size 1.27 1.27)) (justify right bottom))
-  )
   (label "SMBUS.SDA" (at 101.6 132.08 0) (fields_autoplaced)
     (effects (font (size 1.27 1.27)) (justify left bottom))
@@
     (effects (font (size 1.27 1.27)) (justify left bottom))
   )
-  (label "PCIE_X1_JTAG.TMS" (at 101.6 145.415 0) (fields_autoplaced)
-    (effects (font (size 1.27 1.27)) (justify left bottom))
-  )
   (label "PCIE_X1_DATA.RX_N" (at 85.09 111.125 180) (fields_autoplaced)
     (effects (font (size 1.27 1.27)) (justify right bottom))
@@
     (effects (font (size 1.27 1.27)) (justify left bottom))
   )
-  (label "PCIE_X1_JTAG.TDI" (at 85.09 163.195 180) (fields_autoplaced)
-    (effects (font (size 1.27 1.27)) (justify right bottom))
-  )
   (label "PCIE_X1_DATA.TX_N" (at 101.6 125.095 0) (fields_autoplaced)
     (effects (font (size 1.27 1.27)) (justify left bottom))
   )
-  (label "PCIE_X1_JTAG.TDO" (at 85.09 166.37 180) (fields_autoplaced)
-    (effects (font (size 1.27 1.27)) (justify right bottom))
-  )
-  (label "PCIE_X1_JTAG.TCK" (at 101.6 137.795 0) (fields_autoplaced)
-    (effects (font (size 1.27 1.27)) (justify left bottom))
-  )
   (label "SMBUS.SDA" (at 101.6 46.355 0) (fields_autoplaced)
     (effects (font (size 1.27 1.27)) (justify left bottom))
@@
     (effects (font (size 1.27 1.27)) (justify left bottom))
   )
-  (label "PCIE_X1_JTAG.TDO" (at 101.6 142.875 0) (fields_autoplaced)
-    (effects (font (size 1.27 1.27)) (justify left bottom))
-  )
   (label "SMBUS.SDA" (at 85.09 147.32 180) (fields_autoplaced)
     (effects (font (size 1.27 1.27)) (justify right bottom))
   )
-  (label "PCIE_X1_JTAG.TDI" (at 101.6 140.335 0) (fields_autoplaced)
-    (effects (font (size 1.27 1.27)) (justify left bottom))
-  )
   (label "12V" (at 111.76 66.04 180) (fields_autoplaced)
     (effects (font (size 1.27 1.27)) (justify right bottom))
@@
     (effects (font (size 1.27 1.27)) (justify left bottom))
   )
+  (label "PCIE_X1_CTRL.nRST" (at 101.6 106.045 0) (fields_autoplaced)
+    (effects (font (size 1.27 1.27)) (justify left bottom))
+  )
   (label "12V" (at 223.52 195.58 180) (fields_autoplaced)
     (effects (font (size 1.27 1.27)) (justify right bottom))
@@
     (effects (font (size 1.27 1.27)) (justify right bottom))
   )
-  (label "PCIE_X1_JTAG.TMS" (at 85.09 169.545 180) (fields_autoplaced)
-    (effects (font (size 1.27 1.27)) (justify right bottom))
-  )
   (label "1V0SB" (at 107.95 76.2 0) (fields_autoplaced)
     (effects (font (size 1.27 1.27)) (justify left bottom))
   )
-  (label "PCIE_X1_JTAG.TRST" (at 85.09 172.72 180) (fields_autoplaced)
-    (effects (font (size 1.27 1.27)) (justify right bottom))
-  )
   (label "3V3SB" (at 223.52 92.71 180) (fields_autoplaced)
     (effects (font (size 1.27 1.27)) (justify right bottom))
   )
-  (label "PCIE_X1_JTAG.TRST" (at 101.6 147.955 0) (fields_autoplaced)
-    (effects (font (size 1.27 1.27)) (justify left bottom))
-  )
   (label "PCIE_X1_DATA.RX_N" (at 101.6 120.015 0) (fields_autoplaced)
     (effects (font (size 1.27 1.27)) (justify left bottom))
@@
     (effects (font (size 1.27 1.27)) (justify right bottom))
   )
-  (label "PCIE_X1_RST.nRST" (at 101.6 106.045 0) (fields_autoplaced)
-    (effects (font (size 1.27 1.27)) (justify left bottom))
-  )
   (label "PCIE_X1_CLK.N" (at 81.915 93.345 180) (fields_autoplaced)
     (effects (font (size 1.27 1.27)) (justify right bottom))
@@
   )
   (hierarchical_label "GND" (shape bidirectional) (at 101.6 78.74 180) (fields_autoplaced)
-    (effects (font (size 1.27 1.27)) (justify right))
-  )
-  (hierarchical_label "PCIE_X1_JTAG{TCK TDI TDO TMS TRST}" (shape input) (at 57.785 178.435 180) (fields_autoplaced)
     (effects (font (size 1.27 1.27)) (justify right))
   )
@@
       (effects (font (size 1.27 1.27)) (justify left))
     )
-    (pin "PCIE_SW_TCK" input (at 124.46 137.795 180)
-      (effects (font (size 1.27 1.27)) (justify left))
-    )
-    (pin "PCIE_SW_TRST_L" input (at 124.46 147.955 180)
-      (effects (font (size 1.27 1.27)) (justify left))
-    )
-    (pin "PCIE_SW_TMS" input (at 124.46 145.415 180)
-      (effects (font (size 1.27 1.27)) (justify left))
-    )
-    (pin "PCIE_SW_TDO" input (at 124.46 142.875 180)
-      (effects (font (size 1.27 1.27)) (justify left))
-    )
-    (pin "PCIE_SW_TDI" input (at 124.46 140.335 180)
-      (effects (font (size 1.27 1.27)) (justify left))
-    )
