File: Tangenta/CAN_Channel_2.kicad_sch (KiCad schematic)
At the start: 21 parts, among them J33 Conn_01x02_Pin, Q21 BSS138, Q22 BSS138, U23 ADM3053

Commit message: Removing component association with previous project (local) libraries.
Parts:
- C205, C206, C207, C208, C209, C210, C211, C212: symbol CholaSymbolsPrjLib:C_Small -> C_Small:C_Small
- FB12, FB13: footprint CholaFootprintsPrjLib:Ferrite_Bead_100 -> Ferrite_Bead_100:Ferrite_Bead_100; symbol CholaSymbolsPrjLib:GZ2012D101TF -> GZ2012D101TF:GZ2012D101TF
- J33: symbol CholaSymbolsPrjLib:Conn_01x02_Pin -> Conn_01x02_Pin:Conn_01x02_Pin
- Q21, Q22: symbol CholaSymbolsPrjLib:BSS138 -> BSS138:BSS138
- R193, R194, R195, R196, R197, R198, R199: symbol CholaSymbolsPrjLib:R_Small_US -> R_Small_US:R_Small_US
- U23: symbol CholaSymbolsPrjLib:ADM3053 -> ADM3053:ADM3053
Changed lines of the file:
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@@
 	)
 	(symbol
-		(lib_id "CholaSymbolsPrjLib:R_Small_US")
+		(lib_id "R_Small_US:R_Small_US")
 		(at 80.01 134.62 180)
 		(unit 1)
@@
 	)
 	(symbol
-		(lib_id "CholaSymbolsPrjLib:BSS138")
+		(lib_id "BSS138:BSS138")
 		(at 66.04 138.43 270)
 		(unit 1)
@@
 	)
 	(symbol
-		(lib_id "CholaSymbolsPrjLib:C_Small")
+		(lib_id "C_Small:C_Small")
 		(at 132.08 135.89 180)
 		(unit 1)
@@
 	)
 	(symbol
-		(lib_id "CholaSymbolsPrjLib:C_Small")
+		(lib_id "C_Small:C_Small")
 		(at 124.46 116.84 180)
 		(unit 1)
@@
 	)
 	(symbol
-		(lib_id "CholaSymbolsPrjLib:R_Small_US")
+		(lib_id "R_Small_US:R_Small_US")
 		(at 53.34 134.62 180)
 		(unit 1)
@@
 	)
 	(symbol
-		(lib_id "CholaSymbolsPrjLib:BSS138")
+		(lib_id "BSS138:BSS138")
 		(at 66.04 117.475 270)
 		(unit 1)
@@
 	)
 	(symbol
-		(lib_id "CholaSymbolsPrjLib:Conn_01x02_Pin")
+		(lib_id "Conn_01x02_Pin:Conn_01x02_Pin")
 		(at 139.065 153.67 270)
 		(unit 1)
@@
 	)
 	(symbol
-		(lib_id "CholaSymbolsPrjLib:C_Small")
+		(lib_id "C_Small:C_Small")
 		(at 159.385 135.89 0)
 		(mirror x)
@@
 	)
 	(symbol
-		(lib_id "CholaSymbolsPrjLib:R_Small_US")
+		(lib_id "R_Small_US:R_Small_US")
 		(at 80.01 113.665 180)
 		(unit 1)
@@
 	)
 	(symbol
-		(lib_id "CholaSymbolsPrjLib:C_Small")
+		(lib_id "C_Small:C_Small")
 		(at 124.46 135.89 180)
 		(unit 1)
@@
 	)
 	(symbol
-		(lib_id "CholaSymbolsPrjLib:C_Small")
+		(lib_id "C_Small:C_Small")
 		(at 132.08 116.84 180)
 		(unit 1)
@@
 	)
 	(symbol
-		(lib_id "CholaSymbolsPrjLib:C_Small")
+		(lib_id "C_Small:C_Small")
 		(at 141.605 116.84 0)
 		(mirror x)
@@
 	)
 	(symbol
-		(lib_id "CholaSymbolsPrjLib:R_Small_US")
+		(lib_id "R_Small_US:R_Small_US")
 		(at 193.675 73.66 0)
 		(unit 1)
@@
 	(symbol
 		(lib_name "GZ2012D101TF_1")
-		(lib_id "CholaSymbolsPrjLib:GZ2012D101TF")
+		(lib_id "GZ2012D101TF:GZ2012D101TF")
 		(at 168.91 130.81 0)
 		(unit 1)
@@
 			)
 		)
-		(property "Footprint" "CholaFootprintsPrjLib:Ferrite_Bead_100"
+		(property "Footprint" "Ferrite_Bead_100:Ferrite_Bead_100"
 			(at 181.483 140.843 0)
 			(effects
@@
 	)
 	(symbol
-		(lib_id "CholaSymbolsPrjLib:C_Small")
+		(lib_id "C_Small:C_Small")
 		(at 160.655 116.84 0)
 		(mirror x)
@@
 	)
 	(symbol
-		(lib_id "CholaSymbolsPrjLib:R_Small_US")
+		(lib_id "R_Small_US:R_Small_US")
 		(at 53.34 113.665 180)
 		(unit 1)
@@
 	)
 	(symbol
-		(lib_id "CholaSymbolsPrjLib:R_Small_US")
+		(lib_id "R_Small_US:R_Small_US")
 		(at 186.69 77.47 270)
 		(unit 1)
@@
 	)
 	(symbol
-		(lib_id "CholaSymbolsPrjLib:R_Small_US")
+		(lib_id "R_Small_US:R_Small_US")
 		(at 186.69 69.85 270)
 		(unit 1)
@@
 	)
 	(symbol
-		(lib_id "CholaSymbolsPrjLib:ADM3053")
+		(lib_id "ADM3053:ADM3053")
 		(at 137.16 74.93 0)
 		(unit 1)
@@
 	)
 	(symbol
-		(lib_id "CholaSymbolsPrjLib:GZ2012D101TF")
+		(lib_id "GZ2012D101TF:GZ2012D101TF")
 		(at 168.91 140.97 0)
 		(unit 1)
@@
 			)
 		)
-		(property "Footprint" "CholaFootprintsPrjLib:Ferrite_Bead_100"
+		(property "Footprint" "Ferrite_Bead_100:Ferrite_Bead_100"
 			(at 181.483 151.003 0)
 			(effects
@@
 	)
 	(symbol
-		(lib_id "CholaSymbolsPrjLib:C_Small")
+		(lib_id "C_Small:C_Small")
 		(at 178.435 135.89 0)
 		(mirror x)

Commit message: Fixes, continued...
Parts:
- C205, C206, C207, C208, C209, C210, C211, C212: symbol C_Small:C_Small -> Device:C_Small
- J33: symbol Conn_01x02_Pin:Conn_01x02_Pin -> Connector_Generic:Conn_01x02_Pin
- Q21, Q22: symbol BSS138:BSS138 -> Transistor_FET:BSS138
- R193, R194, R195, R196, R197, R198, R199: symbol R_Small_US:R_Small_US -> Device:R_Small_US
- U23: symbol ADM3053:ADM3053 -> ADM3053BRWZ:ADM3053BRWZ-REEL7
Connections:
- net 1V8: no longer Q21.1 (G), Q22.1 (G), R193.2, R194.2
- net 5V: no longer C205.2, C206.2, C207.2, C208.2, R195.2, R196.2, U23.6 (VIO), U23.8 (VCC)
- net CAN_2_CONN_GND: no longer J33.1 (Pin_1)
- net CAN_2_H: no longer R197.1, R199.1
- net CAN_2_H_IC: no longer R197.2, U23.17 (CANH)
- net CAN_2_L: no longer R198.1, R199.2
- net CAN_2_L_IC: no longer R198.2, U23.15 (CANL)
- net CAN_2_RX: no longer Q22.2 (S), R194.1
- net CAN_2_TX: no longer Q21.2 (S), R193.1
- net CAN_ISO_GND: no longer C209.1, C210.1, C211.1, J33.2 (Pin_2), U23.11 (GND2), U23.13 (GND2), U23.16 (GND2), U23.18 (RS), U23.20 (GND2)
- net CAN_ISO_VCC: no longer C209.2, C210.2, C211.2, U23.12 (VISOOUT), U23.19 (VISOIN)
- net GNDREF: no longer C205.1, C206.1, C207.1, C208.1, U23.1 (GND1), U23.10 (GND1), U23.3 (GND1), U23.7 (GND1), U23.9 (GND1)
- net RX_SHIFT: no longer Q22.3 (D), R196.1, U23.4 (RXD)
- net TX_SHIFT: no longer Q21.3 (D), R195.1, U23.5 (TXD)
- net at FB12.2: no longer C212.2
- net at FB13.2: no longer C212.1
Changed lines of the file:
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@@
 	)
 	(symbol
-		(lib_id "R_Small_US:R_Small_US")
+		(lib_id "Device:R_Small_US")
 		(at 80.01 134.62 180)
 		(unit 1)
@@
 	)
 	(symbol
-		(lib_id "BSS138:BSS138")
+		(lib_id "Transistor_FET:BSS138")
 		(at 66.04 138.43 270)
 		(unit 1)
@@
 	)
 	(symbol
-		(lib_id "C_Small:C_Small")
+		(lib_id "Device:C_Small")
 		(at 132.08 135.89 180)
 		(unit 1)
@@
 	)
 	(symbol
-		(lib_id "C_Small:C_Small")
+		(lib_id "Device:C_Small")
 		(at 124.46 116.84 180)
 		(unit 1)
@@
 	)
 	(symbol
-		(lib_id "R_Small_US:R_Small_US")
+		(lib_id "Device:R_Small_US")
 		(at 53.34 134.62 180)
 		(unit 1)
@@
 	)
 	(symbol
-		(lib_id "BSS138:BSS138")
+		(lib_id "Transistor_FET:BSS138")
 		(at 66.04 117.475 270)
 		(unit 1)
@@
 	)
 	(symbol
-		(lib_id "Conn_01x02_Pin:Conn_01x02_Pin")
+		(lib_id "Connector_Generic:Conn_01x02_Pin")
 		(at 139.065 153.67 270)
 		(unit 1)
@@
 	)
 	(symbol
-		(lib_id "C_Small:C_Small")
+		(lib_id "Device:C_Small")
 		(at 159.385 135.89 0)
 		(mirror x)
@@
 	)
 	(symbol
-		(lib_id "R_Small_US:R_Small_US")
+		(lib_id "Device:R_Small_US")
 		(at 80.01 113.665 180)
 		(unit 1)
@@
 	)
 	(symbol
-		(lib_id "C_Small:C_Small")
+		(lib_id "Device:C_Small")
 		(at 124.46 135.89 180)
 		(unit 1)
@@
 	)
 	(symbol
-		(lib_id "C_Small:C_Small")
+		(lib_id "Device:C_Small")
 		(at 132.08 116.84 180)
 		(unit 1)
@@
 	)
 	(symbol
-		(lib_id "C_Small:C_Small")
+		(lib_id "Device:C_Small")
 		(at 141.605 116.84 0)
 		(mirror x)
@@
 	)
 	(symbol
-		(lib_id "R_Small_US:R_Small_US")
+		(lib_id "Device:R_Small_US")
 		(at 193.675 73.66 0)
 		(unit 1)
@@
 	)
 	(symbol
-		(lib_id "C_Small:C_Small")
+		(lib_id "Device:C_Small")
 		(at 160.655 116.84 0)
 		(mirror x)
@@
 	)
 	(symbol
-		(lib_id "R_Small_US:R_Small_US")
+		(lib_id "Device:R_Small_US")
 		(at 53.34 113.665 180)
 		(unit 1)
@@
 	)
 	(symbol
-		(lib_id "R_Small_US:R_Small_US")
+		(lib_id "Device:R_Small_US")
 		(at 186.69 77.47 270)
 		(unit 1)
@@
 	)
 	(symbol
-		(lib_id "R_Small_US:R_Small_US")
+		(lib_id "Device:R_Small_US")
 		(at 186.69 69.85 270)
 		(unit 1)
@@
 	)
 	(symbol
-		(lib_id "ADM3053:ADM3053")
+		(lib_id "ADM3053BRWZ:ADM3053BRWZ-REEL7")
 		(at 137.16 74.93 0)
 		(unit 1)
@@
 	)
 	(symbol
-		(lib_id "C_Small:C_Small")
+		(lib_id "Device:C_Small")
 		(at 178.435 135.89 0)
 		(mirror x)

Commit message: Fixes, continued...
Parts:
- C205, C206, C207, C208, C209, C210, C211, C212: symbol Device:C_Small -> C_Small:C_Small
- J33: symbol Connector_Generic:Conn_01x02_Pin -> Conn_01x02_Pin:Conn_01x02_Pin
- Q21, Q22: symbol Transistor_FET:BSS138 -> BSS138:BSS138
- R193, R194, R195, R196, R197, R198, R199: symbol Device:R_Small_US -> R_Small_US:R_Small_US
- U23: symbol ADM3053BRWZ:ADM3053BRWZ-REEL7 -> ADM3053:ADM3053
Connections:
- net 1V8: now also Q21.1 (G), Q22.1 (G), R193.2, R194.2
- net 5V: now also C205.2, C206.2, C207.2, C208.2, R195.2, R196.2, U23.6 (VIO), U23.8 (VCC)
- net CAN_2_CONN_GND: now also J33.1 (Pin_1)
- net CAN_2_H: now also R197.1, R199.1
- net CAN_2_H_IC: now also R197.2, U23.17 (CANH)
- net CAN_2_L: now also R198.1, R199.2
- net CAN_2_L_IC: now also R198.2, U23.15 (CANL)
- net CAN_2_RX: now also Q22.2 (S), R194.1
- net CAN_2_TX: now also Q21.2 (S), R193.1
- net CAN_ISO_GND: now also C209.1, C210.1, C211.1, J33.2 (Pin_2), U23.11 (GND2), U23.13 (GND2), U23.16 (GND2), U23.18 (RS), U23.20 (GND2)
- net CAN_ISO_VCC: now also C209.2, C210.2, C211.2, U23.12 (VISOOUT), U23.19 (VISOIN)
- net GNDREF: now also C205.1, C206.1, C207.1, C208.1, U23.1 (GND1), U23.10 (GND1), U23.3 (GND1), U23.7 (GND1), U23.9 (GND1)
- net RX_SHIFT: now also Q22.3 (D), R196.1, U23.4 (RXD)
- net TX_SHIFT: now also Q21.3 (D), R195.1, U23.5 (TXD)
- net at FB12.2: now also C212.2
- net at FB13.2: now also C212.1
Changed lines of the file:
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@@
 	)
 	(symbol
-		(lib_id "Device:R_Small_US")
+		(lib_id "R_Small_US:R_Small_US")
 		(at 80.01 134.62 180)
 		(unit 1)
@@
 	)
 	(symbol
-		(lib_id "Transistor_FET:BSS138")
+		(lib_id "BSS138:BSS138")
 		(at 66.04 138.43 270)
 		(unit 1)
@@
 	)
 	(symbol
-		(lib_id "Device:C_Small")
+		(lib_id "C_Small:C_Small")
 		(at 132.08 135.89 180)
 		(unit 1)
@@
 	)
 	(symbol
-		(lib_id "Device:C_Small")
+		(lib_id "C_Small:C_Small")
 		(at 124.46 116.84 180)
 		(unit 1)
@@
 	)
 	(symbol
-		(lib_id "Device:R_Small_US")
+		(lib_id "R_Small_US:R_Small_US")
 		(at 53.34 134.62 180)
 		(unit 1)
@@
 	)
 	(symbol
-		(lib_id "Transistor_FET:BSS138")
+		(lib_id "BSS138:BSS138")
 		(at 66.04 117.475 270)
 		(unit 1)
@@
 	)
 	(symbol
-		(lib_id "Connector_Generic:Conn_01x02_Pin")
+		(lib_id "Conn_01x02_Pin:Conn_01x02_Pin")
 		(at 139.065 153.67 270)
 		(unit 1)
@@
 	)
 	(symbol
-		(lib_id "Device:C_Small")
+		(lib_id "C_Small:C_Small")
 		(at 159.385 135.89 0)
 		(mirror x)
@@
 	)
 	(symbol
-		(lib_id "Device:R_Small_US")
+		(lib_id "R_Small_US:R_Small_US")
 		(at 80.01 113.665 180)
 		(unit 1)
@@
 	)
 	(symbol
-		(lib_id "Device:C_Small")
+		(lib_id "C_Small:C_Small")
 		(at 124.46 135.89 180)
 		(unit 1)
@@
 	)
 	(symbol
-		(lib_id "Device:C_Small")
+		(lib_id "C_Small:C_Small")
 		(at 132.08 116.84 180)
 		(unit 1)
@@
 	)
 	(symbol
-		(lib_id "Device:C_Small")
+		(lib_id "C_Small:C_Small")
 		(at 141.605 116.84 0)
 		(mirror x)
@@
 	)
 	(symbol
-		(lib_id "Device:R_Small_US")
+		(lib_id "R_Small_US:R_Small_US")
 		(at 193.675 73.66 0)
 		(unit 1)
@@
 	)
 	(symbol
-		(lib_id "Device:C_Small")
+		(lib_id "C_Small:C_Small")
 		(at 160.655 116.84 0)
 		(mirror x)
@@
 	)
 	(symbol
-		(lib_id "Device:R_Small_US")
+		(lib_id "R_Small_US:R_Small_US")
 		(at 53.34 113.665 180)
 		(unit 1)
@@
 	)
 	(symbol
-		(lib_id "Device:R_Small_US")
+		(lib_id "R_Small_US:R_Small_US")
 		(at 186.69 77.47 270)
 		(unit 1)
@@
 	)
 	(symbol
-		(lib_id "Device:R_Small_US")
+		(lib_id "R_Small_US:R_Small_US")
 		(at 186.69 69.85 270)
 		(unit 1)
@@
 	)
 	(symbol
-		(lib_id "ADM3053BRWZ:ADM3053BRWZ-REEL7")
+		(lib_id "ADM3053:ADM3053")
 		(at 137.16 74.93 0)
 		(unit 1)
@@
 	)
 	(symbol
-		(lib_id "Device:C_Small")
+		(lib_id "C_Small:C_Small")
 		(at 178.435 135.89 0)
 		(mirror x)

Commit message: Fixes, before checks.
Parts:
- C205, C206, C207, C208, C209, C210, C211, C212: symbol C_Small:C_Small -> Device:C_Small
- FB12, FB13: symbol GZ2012D101TF:GZ2012D101TF -> Ferrite_Bead_100:GZ2012D101TF
- J33: symbol Conn_01x02_Pin:Conn_01x02_Pin -> Connector_Generic:Conn_01x02
- Q21, Q22: symbol BSS138:BSS138 -> Transistor_FET:BSS138
- R193, R194, R195, R196, R197, R198, R199: symbol R_Small_US:R_Small_US -> Device:R_Small_US
- U23: symbol ADM3053:ADM3053 -> ADM3053BRWZ:ADM3053
Changed lines of the file:
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@@
 	)
 	(symbol
-		(lib_id "R_Small_US:R_Small_US")
+		(lib_id "Device:R_Small_US")
 		(at 80.01 134.62 180)
 		(unit 1)
@@
 	)
 	(symbol
-		(lib_id "BSS138:BSS138")
+		(lib_id "Transistor_FET:BSS138")
 		(at 66.04 138.43 270)
 		(unit 1)
@@
 	)
 	(symbol
-		(lib_id "C_Small:C_Small")
+		(lib_id "Device:C_Small")
 		(at 132.08 135.89 180)
 		(unit 1)
@@
 	)
 	(symbol
-		(lib_id "C_Small:C_Small")
+		(lib_id "Device:C_Small")
 		(at 124.46 116.84 180)
 		(unit 1)
@@
 	)
 	(symbol
-		(lib_id "R_Small_US:R_Small_US")
+		(lib_id "Device:R_Small_US")
 		(at 53.34 134.62 180)
 		(unit 1)
@@
 	)
 	(symbol
-		(lib_id "BSS138:BSS138")
+		(lib_id "Transistor_FET:BSS138")
 		(at 66.04 117.475 270)
 		(unit 1)
@@
 	)
 	(symbol
-		(lib_id "Conn_01x02_Pin:Conn_01x02_Pin")
+		(lib_id "Connector_Generic:Conn_01x02")
 		(at 139.065 153.67 270)
 		(unit 1)
@@
 	)
 	(symbol
-		(lib_id "C_Small:C_Small")
+		(lib_id "Device:C_Small")
 		(at 159.385 135.89 0)
 		(mirror x)
@@
 	)
 	(symbol
-		(lib_id "R_Small_US:R_Small_US")
+		(lib_id "Device:R_Small_US")
 		(at 80.01 113.665 180)
 		(unit 1)
@@
 	)
 	(symbol
-		(lib_id "C_Small:C_Small")
+		(lib_id "Device:C_Small")
 		(at 124.46 135.89 180)
 		(unit 1)
@@
 	)
 	(symbol
-		(lib_id "C_Small:C_Small")
+		(lib_id "Device:C_Small")
 		(at 132.08 116.84 180)
 		(unit 1)
@@
 	)
 	(symbol
-		(lib_id "C_Small:C_Small")
+		(lib_id "Device:C_Small")
 		(at 141.605 116.84 0)
 		(mirror x)
@@
 	)
 	(symbol
-		(lib_id "R_Small_US:R_Small_US")
+		(lib_id "Device:R_Small_US")
 		(at 193.675 73.66 0)
 		(unit 1)
@@
 	(symbol
 		(lib_name "GZ2012D101TF_1")
-		(lib_id "GZ2012D101TF:GZ2012D101TF")
+		(lib_id "Ferrite_Bead_100:GZ2012D101TF")
 		(at 168.91 130.81 0)
 		(unit 1)
@@
 	)
 	(symbol
-		(lib_id "C_Small:C_Small")
+		(lib_id "Device:C_Small")
 		(at 160.655 116.84 0)
 		(mirror x)
@@
 	)
 	(symbol
-		(lib_id "R_Small_US:R_Small_US")
+		(lib_id "Device:R_Small_US")
 		(at 53.34 113.665 180)
 		(unit 1)
@@
 	)
 	(symbol
-		(lib_id "R_Small_US:R_Small_US")
+		(lib_id "Device:R_Small_US")
 		(at 186.69 77.47 270)
 		(unit 1)
@@
 	)
 	(symbol
-		(lib_id "R_Small_US:R_Small_US")
+		(lib_id "Device:R_Small_US")
 		(at 186.69 69.85 270)
 		(unit 1)
@@
 	)
 	(symbol
-		(lib_id "ADM3053:ADM3053")
+		(lib_id "ADM3053BRWZ:ADM3053")
 		(at 137.16 74.93 0)
 		(unit 1)
@@
 	)
 	(symbol
-		(lib_id "GZ2012D101TF:GZ2012D101TF")
+		(lib_id "Ferrite_Bead_100:GZ2012D101TF")
 		(at 168.91 140.97 0)
 		(unit 1)
@@
 	)
 	(symbol
-		(lib_id "C_Small:C_Small")
+		(lib_id "Device:C_Small")
 		(at 178.435 135.89 0)
 		(mirror x)

Commit message: Fixes, continued...
Parts:
- U23: value ADM3053 -> ADM3053BRWZ-REEL7; footprint Package_SO:SOIC-20W_7.5x12.8mm_P1.27mm -> ADM3053BRWZ:ADM3053BRWZ; symbol ADM3053BRWZ:ADM3053 -> ADM3053BRWZ:ADM3053BRWZ-REEL7
Connections:
- net 5V: no longer U23.6 (VIO), U23.8 (VCC)
- net CAN_2_H_IC: no longer U23.17 (CANH)
- net CAN_2_L_IC: no longer U23.15 (CANL)
- net CAN_ISO_GND: no longer U23.11 (GND2), U23.13 (GND2), U23.16 (GND2), U23.18 (RS), U23.20 (GND2)
- net CAN_ISO_VCC: no longer U23.12 (VISOOUT), U23.19 (VISOIN)
- net GNDREF: no longer U23.1 (GND1), U23.10 (GND1), U23.3 (GND1), U23.7 (GND1), U23.9 (GND1)
- net RX_SHIFT: no longer U23.4 (RXD)
- net TX_SHIFT: no longer U23.5 (TXD)
Changed lines of the file:
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@@
 	)
 	(symbol
-		(lib_id "ADM3053BRWZ:ADM3053")
+		(lib_id "ADM3053BRWZ:ADM3053BRWZ-REEL7")
 		(at 137.16 74.93 0)
 		(unit 1)
@@
 			)
 		)
-		(property "Value" "ADM3053"
+		(property "Value" "ADM3053BRWZ-REEL7"
 			(at 137.16 54.61 0)
 			(effects
@@
 			)
 		)
-		(property "Footprint" "Package_SO:SOIC-20W_7.5x12.8mm_P1.27mm"
+		(property "Footprint" "ADM3053BRWZ:ADM3053BRWZ"
 			(at 137.16 96.52 0)
 			(effects

Commit message: Reverting to the original design.
Parts:
- C1: renamed from C208; symbol Device:C_Small -> CholaSymbolsPrjLib:C_Small
- C1: renamed from C205; symbol Device:C_Small -> CholaSymbolsPrjLib:C_Small
- C1: renamed from C210; symbol Device:C_Small -> CholaSymbolsPrjLib:C_Small
- C1: renamed from C206; symbol Device:C_Small -> CholaSymbolsPrjLib:C_Small
- C1: renamed from C207; symbol Device:C_Small -> CholaSymbolsPrjLib:C_Small
- C1: renamed from C209; symbol Device:C_Small -> CholaSymbolsPrjLib:C_Small
- C1: renamed from C211; symbol Device:C_Small -> CholaSymbolsPrjLib:C_Small
- C1: renamed from C212; symbol Device:C_Small -> CholaSymbolsPrjLib:C_Small
- FB1: renamed from FB12; symbol Ferrite_Bead_100:GZ2012D101TF -> CholaSymbolsPrjLib:GZ2012D101TF
- FB1: renamed from FB13; symbol Ferrite_Bead_100:GZ2012D101TF -> CholaSymbolsPrjLib:GZ2012D101TF
- J22: renamed from J33; symbol Connector_Generic:Conn_01x02 -> CholaSymbolsPrjLib:Conn_01x02_Pin
- Q3: renamed from Q22; symbol Transistor_FET:BSS138 -> CholaSymbolsPrjLib:BSS138
- Q3: renamed from Q21; symbol Transistor_FET:BSS138 -> CholaSymbolsPrjLib:BSS138
- R2: renamed from R196; symbol Device:R_Small_US -> CholaSymbolsPrjLib:R_Small_US
- R2: renamed from R194; symbol Device:R_Small_US -> CholaSymbolsPrjLib:R_Small_US
- R2: renamed from R195; symbol Device:R_Small_US -> CholaSymbolsPrjLib:R_Small_US
- R2: renamed from R193; symbol Device:R_Small_US -> CholaSymbolsPrjLib:R_Small_US
- R2: renamed from R198; symbol Device:R_Small_US -> CholaSymbolsPrjLib:R_Small_US
- R2: renamed from R197; symbol Device:R_Small_US -> CholaSymbolsPrjLib:R_Small_US
- R4: renamed from R199; symbol Device:R_Small_US -> CholaSymbolsPrjLib:R_Small_US
- U20: renamed from U23; value ADM3053BRWZ-REEL7 -> ADM3053; footprint ADM3053BRWZ:ADM3053BRWZ -> Package_SO:SOIC-20W_7.5x12.8mm_P1.27mm; symbol ADM3053BRWZ:ADM3053BRWZ-REEL7 -> CholaSymbolsPrjLib:ADM3053
Connections:
- net 5V: now also U20.6 (VIO), U20.8 (VCC)
- net CAN_2_H_IC: now also U20.17 (CANH)
- net CAN_2_L_IC: now also U20.15 (CANL)
- net CAN_ISO_GND: now also U20.11 (GND2), U20.13 (GND2), U20.16 (GND2), U20.18 (RS), U20.20 (GND2)
- net CAN_ISO_VCC: now also U20.12 (VISOOUT), U20.19 (VISOIN)
- net GNDREF: now also U20.1 (GND1), U20.10 (GND1), U20.3 (GND1), U20.7 (GND1), U20.9 (GND1)
- net RX_SHIFT: now also U20.4 (RXD)
- net TX_SHIFT: now also U20.5 (TXD)

Commit message: initialize branch
Parts:
- renumbered C1 to C205, C1 to C206, C1 to C207, C1 to C208, C1 to C209, C1 to C210, C1 to C211, C1 to C212, FB1 to FB12, FB1 to FB13, J22 to J33, Q3 to Q21, Q3 to Q22, R2 to R193, R2 to R194, R2 to R195, R2 to R196, R2 to R197, R2 to R198, R4 to R199, U20 to U23
