File: Tangenta/CAN_Channel_2.kicad_sch (KiCad schematic)
At the start: 21 parts, among them J22 Conn_01x02_Pin, Q3 BSS138, U20 ADM3053

Commit message: ...
Parts:
- C1: symbol CholaSymbolsPrjLib:C_Small -> LocalPrjLib:C_Small
- FB1: symbol CholaSymbolsPrjLib:GZ2012D101TF -> LocalPrjLib:GZ2012D101TF
- J22: symbol CholaSymbolsPrjLib:Conn_01x02_Pin -> LocalPrjLib:Conn_01x02_Pin
- Q3: symbol CholaSymbolsPrjLib:BSS138 -> LocalPrjLib:BSS138
- R2, R4: symbol CholaSymbolsPrjLib:R_Small_US -> LocalPrjLib:R_Small_US
- U20: symbol CholaSymbolsPrjLib:ADM3053 -> LocalPrjLib:ADM3053
Changed lines of the file:
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@@
     (effects (font (size 1.27 1.27)) (justify left))
   )
-  (symbol (lib_id "CholaSymbolsPrjLib:R_Small_US") (at 80.01 134.62 180) (unit 1)
+  (symbol (lib_id "LocalPrjLib:R_Small_US") (at 80.01 134.62 180) (unit 1)
     (in_bom yes) (on_board yes) (dnp no)
     (property "Reference" "R2" (at 78.74 133.35 0)
@@
     )
   )
-  (symbol (lib_id "CholaSymbolsPrjLib:BSS138") (at 66.04 138.43 270) (unit 1)
+  (symbol (lib_id "LocalPrjLib:BSS138") (at 66.04 138.43 270) (unit 1)
     (in_bom yes) (on_board yes) (dnp no)
     (property "Reference" "Q3" (at 68.58 135.89 90)
@@
     )
   )
-  (symbol (lib_id "CholaSymbolsPrjLib:C_Small") (at 132.08 135.89 180) (unit 1)
+  (symbol (lib_id "LocalPrjLib:C_Small") (at 132.08 135.89 180) (unit 1)
     (in_bom yes) (on_board yes) (dnp no)
     (property "Reference" "C1" (at 129.5399 133.9849 0)
@@
     )
   )
-  (symbol (lib_id "CholaSymbolsPrjLib:C_Small") (at 124.46 116.84 180) (unit 1)
+  (symbol (lib_id "LocalPrjLib:C_Small") (at 124.46 116.84 180) (unit 1)
     (in_bom yes) (on_board yes) (dnp no)
     (property "Reference" "C1" (at 121.9199 114.9349 0)
@@
     )
   )
-  (symbol (lib_id "CholaSymbolsPrjLib:R_Small_US") (at 53.34 134.62 180) (unit 1)
+  (symbol (lib_id "LocalPrjLib:R_Small_US") (at 53.34 134.62 180) (unit 1)
     (in_bom yes) (on_board yes) (dnp no)
     (property "Reference" "R2" (at 52.07 133.35 0)
@@
     )
   )
-  (symbol (lib_id "CholaSymbolsPrjLib:BSS138") (at 66.04 117.475 270) (unit 1)
+  (symbol (lib_id "LocalPrjLib:BSS138") (at 66.04 117.475 270) (unit 1)
     (in_bom yes) (on_board yes) (dnp no)
     (property "Reference" "Q3" (at 68.58 114.935 90)
@@
     )
   )
-  (symbol (lib_id "CholaSymbolsPrjLib:Conn_01x02_Pin") (at 139.065 153.67 270) (unit 1)
+  (symbol (lib_id "LocalPrjLib:Conn_01x02_Pin") (at 139.065 153.67 270) (unit 1)
     (in_bom yes) (on_board yes) (dnp no)
     (property "Reference" "J22" (at 135.89 152.4 90)
@@
     )
   )
-  (symbol (lib_id "CholaSymbolsPrjLib:C_Small") (at 159.385 135.89 0) (mirror x) (unit 1)
+  (symbol (lib_id "LocalPrjLib:C_Small") (at 159.385 135.89 0) (mirror x) (unit 1)
     (in_bom yes) (on_board yes) (dnp no)
     (property "Reference" "C1" (at 161.9251 133.9849 0)
@@
     )
   )
-  (symbol (lib_id "CholaSymbolsPrjLib:R_Small_US") (at 80.01 113.665 180) (unit 1)
+  (symbol (lib_id "LocalPrjLib:R_Small_US") (at 80.01 113.665 180) (unit 1)
     (in_bom yes) (on_board yes) (dnp no)
     (property "Reference" "R2" (at 78.74 112.395 0)
@@
     )
   )
-  (symbol (lib_id "CholaSymbolsPrjLib:C_Small") (at 124.46 135.89 180) (unit 1)
+  (symbol (lib_id "LocalPrjLib:C_Small") (at 124.46 135.89 180) (unit 1)
     (in_bom yes) (on_board yes) (dnp no)
     (property "Reference" "C1" (at 121.9199 133.9849 0)
@@
     )
   )
-  (symbol (lib_id "CholaSymbolsPrjLib:C_Small") (at 132.08 116.84 180) (unit 1)
+  (symbol (lib_id "LocalPrjLib:C_Small") (at 132.08 116.84 180) (unit 1)
     (in_bom yes) (on_board yes) (dnp no)
     (property "Reference" "C1" (at 129.5399 114.9349 0)
@@
     )
   )
-  (symbol (lib_id "CholaSymbolsPrjLib:C_Small") (at 141.605 116.84 0) (mirror x) (unit 1)
+  (symbol (lib_id "LocalPrjLib:C_Small") (at 141.605 116.84 0) (mirror x) (unit 1)
     (in_bom yes) (on_board yes) (dnp no)
     (property "Reference" "C1" (at 144.1451 114.9349 0)
@@
     )
   )
-  (symbol (lib_id "CholaSymbolsPrjLib:R_Small_US") (at 193.675 73.66 0) (unit 1)
+  (symbol (lib_id "LocalPrjLib:R_Small_US") (at 193.675 73.66 0) (unit 1)
     (in_bom yes) (on_board yes) (dnp no)
     (property "Reference" "R4" (at 197.485 72.39 0)
@@
     )
   )
-  (symbol (lib_id "CholaSymbolsPrjLib:GZ2012D101TF") (at 168.91 130.81 0) (unit 1)
+  (symbol (lib_id "LocalPrjLib:GZ2012D101TF") (at 168.91 130.81 0) (unit 1)
     (in_bom yes) (on_board yes) (dnp no)
     (property "Reference" "FB1" (at 168.91 128.27 0)
@@
     )
   )
-  (symbol (lib_id "CholaSymbolsPrjLib:C_Small") (at 160.655 116.84 0) (mirror x) (unit 1)
+  (symbol (lib_id "LocalPrjLib:C_Small") (at 160.655 116.84 0) (mirror x) (unit 1)
     (in_bom yes) (on_board yes) (dnp no)
     (property "Reference" "C1" (at 163.1951 114.9349 0)
@@
     )
   )
-  (symbol (lib_id "CholaSymbolsPrjLib:R_Small_US") (at 53.34 113.665 180) (unit 1)
+  (symbol (lib_id "LocalPrjLib:R_Small_US") (at 53.34 113.665 180) (unit 1)
     (in_bom yes) (on_board yes) (dnp no)
     (property "Reference" "R2" (at 52.07 112.395 0)
@@
     )
   )
-  (symbol (lib_id "CholaSymbolsPrjLib:R_Small_US") (at 186.69 77.47 270) (unit 1)
+  (symbol (lib_id "LocalPrjLib:R_Small_US") (at 186.69 77.47 270) (unit 1)
     (in_bom yes) (on_board yes) (dnp no)
     (property "Reference" "R2" (at 179.705 76.2 90)
@@
     )
   )
-  (symbol (lib_id "CholaSymbolsPrjLib:R_Small_US") (at 186.69 69.85 270) (unit 1)
+  (symbol (lib_id "LocalPrjLib:R_Small_US") (at 186.69 69.85 270) (unit 1)
     (in_bom yes) (on_board yes) (dnp no)
     (property "Reference" "R2" (at 179.705 68.58 90)
@@
     )
   )
-  (symbol (lib_id "CholaSymbolsPrjLib:ADM3053") (at 137.16 74.93 0) (unit 1)
+  (symbol (lib_id "LocalPrjLib:ADM3053") (at 137.16 74.93 0) (unit 1)
     (in_bom yes) (on_board yes) (dnp no) (fields_autoplaced)
     (property "Reference" "U20" (at 137.16 52.07 0)
@@
     )
   )
-  (symbol (lib_id "CholaSymbolsPrjLib:GZ2012D101TF") (at 168.91 140.97 0) (unit 1)
+  (symbol (lib_id "LocalPrjLib:GZ2012D101TF") (at 168.91 140.97 0) (unit 1)
     (in_bom yes) (on_board yes) (dnp no)
     (property "Reference" "FB1" (at 168.91 138.43 0)
@@
     )
   )
-  (symbol (lib_id "CholaSymbolsPrjLib:C_Small") (at 178.435 135.89 0) (mirror x) (unit 1)
+  (symbol (lib_id "LocalPrjLib:C_Small") (at 178.435 135.89 0) (mirror x) (unit 1)
     (in_bom yes) (on_board yes) (dnp no)
     (property "Reference" "C1" (at 180.9751 133.9849 0)
