File: Tangenta/CAN_Channel_1.kicad_sch (KiCad schematic)
At the start: 21 parts, among them J32 Conn_01x02_Pin, Q19 BSS138, Q20 BSS138, U22 ADM3053

Commit message: Removing component association with previous project (local) libraries.
Parts:
- C197, C198, C199, C200, C201, C202, C203, C204: symbol CholaSymbolsPrjLib:C_Small -> C_Small:C_Small
- FB10, FB11: footprint CholaFootprintsPrjLib:Ferrite_Bead_100 -> Ferrite_Bead_100:Ferrite_Bead_100; symbol CholaSymbolsPrjLib:GZ2012D101TF -> GZ2012D101TF:GZ2012D101TF
- J32: symbol CholaSymbolsPrjLib:Conn_01x02_Pin -> Conn_01x02_Pin:Conn_01x02_Pin
- Q19, Q20: symbol CholaSymbolsPrjLib:BSS138 -> BSS138:BSS138
- R186, R187, R188, R189, R190, R191, R192: symbol CholaSymbolsPrjLib:R_Small_US -> R_Small_US:R_Small_US
- U22: symbol CholaSymbolsPrjLib:ADM3053 -> ADM3053:ADM3053
Changed lines of the file:
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@@
 	)
 	(symbol
-		(lib_id "CholaSymbolsPrjLib:GZ2012D101TF")
+		(lib_id "GZ2012D101TF:GZ2012D101TF")
 		(at 168.91 140.97 0)
 		(unit 1)
@@
 			)
 		)
-		(property "Footprint" "CholaFootprintsPrjLib:Ferrite_Bead_100"
+		(property "Footprint" "Ferrite_Bead_100:Ferrite_Bead_100"
 			(at 181.483 151.003 0)
 			(effects
@@
 	)
 	(symbol
-		(lib_id "CholaSymbolsPrjLib:C_Small")
+		(lib_id "C_Small:C_Small")
 		(at 132.08 116.84 180)
 		(unit 1)
@@
 	)
 	(symbol
-		(lib_id "CholaSymbolsPrjLib:C_Small")
+		(lib_id "C_Small:C_Small")
 		(at 159.385 135.89 0)
 		(mirror x)
@@
 	)
 	(symbol
-		(lib_id "CholaSymbolsPrjLib:C_Small")
+		(lib_id "C_Small:C_Small")
 		(at 124.46 116.84 180)
 		(unit 1)
@@
 	)
 	(symbol
-		(lib_id "CholaSymbolsPrjLib:C_Small")
+		(lib_id "C_Small:C_Small")
 		(at 132.08 135.89 180)
 		(unit 1)
@@
 	)
 	(symbol
-		(lib_id "CholaSymbolsPrjLib:BSS138")
+		(lib_id "BSS138:BSS138")
 		(at 66.04 117.475 270)
 		(unit 1)
@@
 	)
 	(symbol
-		(lib_id "CholaSymbolsPrjLib:R_Small_US")
+		(lib_id "R_Small_US:R_Small_US")
 		(at 186.69 69.85 270)
 		(unit 1)
@@
 	)
 	(symbol
-		(lib_id "CholaSymbolsPrjLib:C_Small")
+		(lib_id "C_Small:C_Small")
 		(at 141.605 116.84 0)
 		(mirror x)
@@
 	)
 	(symbol
-		(lib_id "CholaSymbolsPrjLib:C_Small")
+		(lib_id "C_Small:C_Small")
 		(at 160.655 116.84 0)
 		(mirror x)
@@
 	)
 	(symbol
-		(lib_id "CholaSymbolsPrjLib:Conn_01x02_Pin")
+		(lib_id "Conn_01x02_Pin:Conn_01x02_Pin")
 		(at 139.065 153.67 270)
 		(unit 1)
@@
 	)
 	(symbol
-		(lib_id "CholaSymbolsPrjLib:BSS138")
+		(lib_id "BSS138:BSS138")
 		(at 66.04 138.43 270)
 		(unit 1)
@@
 	)
 	(symbol
-		(lib_id "CholaSymbolsPrjLib:C_Small")
+		(lib_id "C_Small:C_Small")
 		(at 124.46 135.89 180)
 		(unit 1)
@@
 	)
 	(symbol
-		(lib_id "CholaSymbolsPrjLib:R_Small_US")
+		(lib_id "R_Small_US:R_Small_US")
 		(at 80.01 134.62 180)
 		(unit 1)
@@
 	)
 	(symbol
-		(lib_id "CholaSymbolsPrjLib:R_Small_US")
+		(lib_id "R_Small_US:R_Small_US")
 		(at 186.69 77.47 270)
 		(unit 1)
@@
 	)
 	(symbol
-		(lib_id "CholaSymbolsPrjLib:R_Small_US")
+		(lib_id "R_Small_US:R_Small_US")
 		(at 53.34 134.62 180)
 		(unit 1)
@@
 	)
 	(symbol
-		(lib_id "CholaSymbolsPrjLib:C_Small")
+		(lib_id "C_Small:C_Small")
 		(at 178.435 135.89 0)
 		(mirror x)
@@
 	)
 	(symbol
-		(lib_id "CholaSymbolsPrjLib:R_Small_US")
+		(lib_id "R_Small_US:R_Small_US")
 		(at 80.01 113.665 180)
 		(unit 1)
@@
 	)
 	(symbol
-		(lib_id "CholaSymbolsPrjLib:R_Small_US")
+		(lib_id "R_Small_US:R_Small_US")
 		(at 193.675 73.66 0)
 		(unit 1)
@@
 	)
 	(symbol
-		(lib_id "CholaSymbolsPrjLib:ADM3053")
+		(lib_id "ADM3053:ADM3053")
 		(at 137.16 74.93 0)
 		(unit 1)
@@
 	)
 	(symbol
-		(lib_id "CholaSymbolsPrjLib:R_Small_US")
+		(lib_id "R_Small_US:R_Small_US")
 		(at 53.34 113.665 180)
 		(unit 1)
@@
 	(symbol
 		(lib_name "GZ2012D101TF_1")
-		(lib_id "CholaSymbolsPrjLib:GZ2012D101TF")
+		(lib_id "GZ2012D101TF:GZ2012D101TF")
 		(at 168.91 130.81 0)
 		(unit 1)
@@
 			)
 		)
-		(property "Footprint" "CholaFootprintsPrjLib:Ferrite_Bead_100"
+		(property "Footprint" "Ferrite_Bead_100:Ferrite_Bead_100"
 			(at 181.483 140.843 0)
 			(effects

Commit message: Fixes, before checks.
Parts:
- C197, C198, C199, C200, C201, C202, C203, C204: symbol C_Small:C_Small -> Device:C_Small
- FB10, FB11: symbol GZ2012D101TF:GZ2012D101TF -> Ferrite_Bead_100:GZ2012D101TF
- J32: symbol Conn_01x02_Pin:Conn_01x02_Pin -> Connector_Generic:Conn_01x02
- Q19, Q20: symbol BSS138:BSS138 -> Transistor_FET:BSS138
- R186, R187, R188, R189, R190, R191, R192: symbol R_Small_US:R_Small_US -> Device:R_Small_US
- U22: symbol ADM3053:ADM3053 -> ADM3053BRWZ:ADM3053
Changed lines of the file:
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@@
 	)
 	(symbol
-		(lib_id "GZ2012D101TF:GZ2012D101TF")
+		(lib_id "Ferrite_Bead_100:GZ2012D101TF")
 		(at 168.91 140.97 0)
 		(unit 1)
@@
 	)
 	(symbol
-		(lib_id "C_Small:C_Small")
+		(lib_id "Device:C_Small")
 		(at 132.08 116.84 180)
 		(unit 1)
@@
 	)
 	(symbol
-		(lib_id "C_Small:C_Small")
+		(lib_id "Device:C_Small")
 		(at 159.385 135.89 0)
 		(mirror x)
@@
 	)
 	(symbol
-		(lib_id "C_Small:C_Small")
+		(lib_id "Device:C_Small")
 		(at 124.46 116.84 180)
 		(unit 1)
@@
 	)
 	(symbol
-		(lib_id "C_Small:C_Small")
+		(lib_id "Device:C_Small")
 		(at 132.08 135.89 180)
 		(unit 1)
@@
 	)
 	(symbol
-		(lib_id "BSS138:BSS138")
+		(lib_id "Transistor_FET:BSS138")
 		(at 66.04 117.475 270)
 		(unit 1)
@@
 	)
 	(symbol
-		(lib_id "R_Small_US:R_Small_US")
+		(lib_id "Device:R_Small_US")
 		(at 186.69 69.85 270)
 		(unit 1)
@@
 	)
 	(symbol
-		(lib_id "C_Small:C_Small")
+		(lib_id "Device:C_Small")
 		(at 141.605 116.84 0)
 		(mirror x)
@@
 	)
 	(symbol
-		(lib_id "C_Small:C_Small")
+		(lib_id "Device:C_Small")
 		(at 160.655 116.84 0)
 		(mirror x)
@@
 	)
 	(symbol
-		(lib_id "Conn_01x02_Pin:Conn_01x02_Pin")
+		(lib_id "Connector_Generic:Conn_01x02")
 		(at 139.065 153.67 270)
 		(unit 1)
@@
 	)
 	(symbol
-		(lib_id "BSS138:BSS138")
+		(lib_id "Transistor_FET:BSS138")
 		(at 66.04 138.43 270)
 		(unit 1)
@@
 	)
 	(symbol
-		(lib_id "C_Small:C_Small")
+		(lib_id "Device:C_Small")
 		(at 124.46 135.89 180)
 		(unit 1)
@@
 	)
 	(symbol
-		(lib_id "R_Small_US:R_Small_US")
+		(lib_id "Device:R_Small_US")
 		(at 80.01 134.62 180)
 		(unit 1)
@@
 	)
 	(symbol
-		(lib_id "R_Small_US:R_Small_US")
+		(lib_id "Device:R_Small_US")
 		(at 186.69 77.47 270)
 		(unit 1)
@@
 	)
 	(symbol
-		(lib_id "R_Small_US:R_Small_US")
+		(lib_id "Device:R_Small_US")
 		(at 53.34 134.62 180)
 		(unit 1)
@@
 	)
 	(symbol
-		(lib_id "C_Small:C_Small")
+		(lib_id "Device:C_Small")
 		(at 178.435 135.89 0)
 		(mirror x)
@@
 	)
 	(symbol
-		(lib_id "R_Small_US:R_Small_US")
+		(lib_id "Device:R_Small_US")
 		(at 80.01 113.665 180)
 		(unit 1)
@@
 	)
 	(symbol
-		(lib_id "R_Small_US:R_Small_US")
+		(lib_id "Device:R_Small_US")
 		(at 193.675 73.66 0)
 		(unit 1)
@@
 	)
 	(symbol
-		(lib_id "ADM3053:ADM3053")
+		(lib_id "ADM3053BRWZ:ADM3053")
 		(at 137.16 74.93 0)
 		(unit 1)
@@
 	)
 	(symbol
-		(lib_id "R_Small_US:R_Small_US")
+		(lib_id "Device:R_Small_US")
 		(at 53.34 113.665 180)
 		(unit 1)
@@
 	(symbol
 		(lib_name "GZ2012D101TF_1")
-		(lib_id "GZ2012D101TF:GZ2012D101TF")
+		(lib_id "Ferrite_Bead_100:GZ2012D101TF")
 		(at 168.91 130.81 0)
 		(unit 1)

Commit message: Fixes, continued...
Parts:
- U22: value ADM3053 -> ADM3053BRWZ-REEL7; footprint Package_SO:SOIC-20W_7.5x12.8mm_P1.27mm -> ADM3053BRWZ:ADM3053BRWZ; symbol ADM3053BRWZ:ADM3053 -> ADM3053BRWZ:ADM3053BRWZ-REEL7
Connections:
- net 5V: no longer U22.6 (VIO), U22.8 (VCC)
- net CAN_1_H_IC: no longer U22.17 (CANH)
- net CAN_1_L_IC: no longer U22.15 (CANL)
- net CAN_ISO_GND: no longer U22.11 (GND2), U22.13 (GND2), U22.16 (GND2), U22.18 (RS), U22.20 (GND2)
- net CAN_ISO_VCC: no longer U22.12 (VISOOUT), U22.19 (VISOIN)
- net GNDREF: no longer U22.1 (GND1), U22.10 (GND1), U22.3 (GND1), U22.7 (GND1), U22.9 (GND1)
- net RX_SHIFT: no longer U22.4 (RXD)
- net TX_SHIFT: no longer U22.5 (TXD)
Changed lines of the file:
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@@
 	)
 	(symbol
-		(lib_id "ADM3053BRWZ:ADM3053")
+		(lib_id "ADM3053BRWZ:ADM3053BRWZ-REEL7")
 		(at 137.16 74.93 0)
 		(unit 1)
@@
 			)
 		)
-		(property "Value" "ADM3053"
+		(property "Value" "ADM3053BRWZ-REEL7"
 			(at 137.16 54.61 0)
 			(effects
@@
 			)
 		)
-		(property "Footprint" "Package_SO:SOIC-20W_7.5x12.8mm_P1.27mm"
+		(property "Footprint" "ADM3053BRWZ:ADM3053BRWZ"
 			(at 137.16 96.52 0)
 			(effects

Commit message: Reverting to the original design.
Parts:
- C1: renamed from C199; symbol Device:C_Small -> CholaSymbolsPrjLib:C_Small
- C1: renamed from C202; symbol Device:C_Small -> CholaSymbolsPrjLib:C_Small
- C1: renamed from C197; symbol Device:C_Small -> CholaSymbolsPrjLib:C_Small
- C1: renamed from C200; symbol Device:C_Small -> CholaSymbolsPrjLib:C_Small
- C1: renamed from C201; symbol Device:C_Small -> CholaSymbolsPrjLib:C_Small
- C1: renamed from C203; symbol Device:C_Small -> CholaSymbolsPrjLib:C_Small
- C1: renamed from C198; symbol Device:C_Small -> CholaSymbolsPrjLib:C_Small
- C1: renamed from C204; symbol Device:C_Small -> CholaSymbolsPrjLib:C_Small
- FB1: renamed from FB11; symbol Ferrite_Bead_100:GZ2012D101TF -> CholaSymbolsPrjLib:GZ2012D101TF
- FB1: renamed from FB10; symbol Ferrite_Bead_100:GZ2012D101TF -> CholaSymbolsPrjLib:GZ2012D101TF
- J22: renamed from J32; symbol Connector_Generic:Conn_01x02 -> CholaSymbolsPrjLib:Conn_01x02_Pin
- Q3: renamed from Q19; symbol Transistor_FET:BSS138 -> CholaSymbolsPrjLib:BSS138
- Q3: renamed from Q20; symbol Transistor_FET:BSS138 -> CholaSymbolsPrjLib:BSS138
- R2: renamed from R190; symbol Device:R_Small_US -> CholaSymbolsPrjLib:R_Small_US
- R2: renamed from R189; symbol Device:R_Small_US -> CholaSymbolsPrjLib:R_Small_US
- R2: renamed from R191; symbol Device:R_Small_US -> CholaSymbolsPrjLib:R_Small_US
- R2: renamed from R187; symbol Device:R_Small_US -> CholaSymbolsPrjLib:R_Small_US
- R2: renamed from R188; symbol Device:R_Small_US -> CholaSymbolsPrjLib:R_Small_US
- R2: renamed from R186; symbol Device:R_Small_US -> CholaSymbolsPrjLib:R_Small_US
- R4: renamed from R192; symbol Device:R_Small_US -> CholaSymbolsPrjLib:R_Small_US
- U22: value ADM3053BRWZ-REEL7 -> ADM3053; footprint ADM3053BRWZ:ADM3053BRWZ -> Package_SO:SOIC-20W_7.5x12.8mm_P1.27mm; symbol ADM3053BRWZ:ADM3053BRWZ-REEL7 -> CholaSymbolsPrjLib:ADM3053
Connections:
- net 5V: now also U22.6 (VIO), U22.8 (VCC)
- net CAN_1_H_IC: now also U22.17 (CANH)
- net CAN_1_L_IC: now also U22.15 (CANL)
- net CAN_ISO_GND: now also U22.11 (GND2), U22.13 (GND2), U22.16 (GND2), U22.18 (RS), U22.20 (GND2)
- net CAN_ISO_VCC: now also U22.12 (VISOOUT), U22.19 (VISOIN)
- net GNDREF: now also U22.1 (GND1), U22.10 (GND1), U22.3 (GND1), U22.7 (GND1), U22.9 (GND1)
- net RX_SHIFT: now also U22.4 (RXD)
- net TX_SHIFT: now also U22.5 (TXD)

Commit message: initialize branch
Parts:
- renumbered C1 to C197, C1 to C198, C1 to C199, C1 to C200, C1 to C201, C1 to C202, C1 to C203, C1 to C204, FB1 to FB10, FB1 to FB11, J22 to J32, Q3 to Q19, Q3 to Q20, R2 to R186, R2 to R187, R2 to R188, R2 to R189, R2 to R190, R2 to R191, R4 to R192

Commit message: FB5-FB13, D6
Parts:
- FB10, FB11: footprint Ferrite_Bead_100:Ferrite_Bead_100 -> CholaFootprintsPrjLib:Ferrite_Bead_100
Changed lines of the file:
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@@
       (effects (font (size 1.27 1.27)) hide)
     )
-    (property "Footprint" "Ferrite_Bead_100:Ferrite_Bead_100" (at 181.483 151.003 0)
+    (property "Footprint" "CholaFootprintsPrjLib:Ferrite_Bead_100" (at 181.483 151.003 0)
       (effects (font (size 1.27 1.27) italic) hide)
     )
@@
     )
   )
-  (symbol (lib_id "CholaSymbolsPrjLib:GZ2012D101TF") (at 168.91 130.81 0) (unit 1)
+  (symbol (lib_name "GZ2012D101TF_1") (lib_id "CholaSymbolsPrjLib:GZ2012D101TF") (at 168.91 130.81 0) (unit 1)
     (in_bom yes) (on_board yes) (dnp no)
     (property "Reference" "FB10" (at 168.91 128.27 0)
@@
       (effects (font (size 1.27 1.27)) hide)
     )
-    (property "Footprint" "Ferrite_Bead_100:Ferrite_Bead_100" (at 181.483 140.843 0)
+    (property "Footprint" "CholaFootprintsPrjLib:Ferrite_Bead_100" (at 181.483 140.843 0)
       (effects (font (size 1.27 1.27) italic) hide)
     )
