File: Tangenta/MobileModem.kicad_sch (KiCad schematic)
At the start: 12 parts, among them J7 1-2199230-5, J8 HYC90-SIM06-180

Commit message: Removing component association with previous project (local) libraries.
Parts:
- C70, C71, C72: symbol CholaSymbolsPrjLib:C_Small -> C_Small:C_Small
- H10, H11: symbol CholaSymbolsPrjLib:MountingHole -> MountingHole:MountingHole
- J7: footprint CholaFootprintsPrjLib:M2_Slot -> M2_Slot:M2_Slot; symbol CholaSymbolsPrjLib:1-2199230-5 -> 1-2199230-5:1-2199230-5
- J8: footprint CholaFootprintsPrjLib:SIM-SMD_HYC90-SIM06-180 -> SIM-SMD_HYC90-SIM06-180:SIM-SMD_HYC90-SIM06-180; symbol CholaSymbolsPrjLib:HYC90-SIM06-180 -> HYC90-SIM06-180:HYC90-SIM06-180
- R42, R43, R44, R45, R46: symbol CholaSymbolsPrjLib:R_Small_US -> R_Small_US:R_Small_US
Changed lines of the file:
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@@
 	)
 	(symbol
-		(lib_id "CholaSymbolsPrjLib:HYC90-SIM06-180")
+		(lib_id "HYC90-SIM06-180:HYC90-SIM06-180")
 		(at 148.59 87.63 0)
 		(unit 1)
@@
 			)
 		)
-		(property "Footprint" "CholaFootprintsPrjLib:SIM-SMD_HYC90-SIM06-180"
+		(property "Footprint" "SIM-SMD_HYC90-SIM06-180:SIM-SMD_HYC90-SIM06-180"
 			(at 149.86 80.01 0)
 			(effects
@@
 	)
 	(symbol
-		(lib_id "CholaSymbolsPrjLib:MountingHole")
+		(lib_id "MountingHole:MountingHole")
 		(at 186.055 76.2 0)
 		(unit 1)
@@
 	)
 	(symbol
-		(lib_id "CholaSymbolsPrjLib:C_Small")
+		(lib_id "C_Small:C_Small")
 		(at 140.97 68.58 180)
 		(unit 1)
@@
 	)
 	(symbol
-		(lib_id "CholaSymbolsPrjLib:C_Small")
+		(lib_id "C_Small:C_Small")
 		(at 156.21 68.58 180)
 		(unit 1)
@@
 	)
 	(symbol
-		(lib_id "CholaSymbolsPrjLib:R_Small_US")
+		(lib_id "R_Small_US:R_Small_US")
 		(at 173.99 74.93 180)
 		(unit 1)
@@
 	)
 	(symbol
-		(lib_id "CholaSymbolsPrjLib:R_Small_US")
+		(lib_id "R_Small_US:R_Small_US")
 		(at 54.61 77.47 90)
 		(unit 1)
@@
 	)
 	(symbol
-		(lib_id "CholaSymbolsPrjLib:C_Small")
+		(lib_id "C_Small:C_Small")
 		(at 124.46 95.25 180)
 		(unit 1)
@@
 	)
 	(symbol
-		(lib_id "CholaSymbolsPrjLib:MountingHole")
+		(lib_id "MountingHole:MountingHole")
 		(at 186.055 83.82 0)
 		(unit 1)
@@
 	)
 	(symbol
-		(lib_id "CholaSymbolsPrjLib:R_Small_US")
+		(lib_id "R_Small_US:R_Small_US")
 		(at 92.71 57.15 270)
 		(mirror x)
@@
 	)
 	(symbol
-		(lib_id "CholaSymbolsPrjLib:R_Small_US")
+		(lib_id "R_Small_US:R_Small_US")
 		(at 54.61 128.27 90)
 		(unit 1)
@@
 	)
 	(symbol
-		(lib_id "CholaSymbolsPrjLib:R_Small_US")
+		(lib_id "R_Small_US:R_Small_US")
 		(at 124.46 104.14 180)
 		(unit 1)
@@
 	)
 	(symbol
-		(lib_id "CholaSymbolsPrjLib:1-2199230-5")
+		(lib_id "1-2199230-5:1-2199230-5")
 		(at 73.66 44.45 90)
 		(mirror x)
@@
 			)
 		)
-		(property "Footprint" "CholaFootprintsPrjLib:M2_Slot"
+		(property "Footprint" "M2_Slot:M2_Slot"
 			(at 163.5 139.7 0)
 			(effects
