File: Tangenta/DSI_HDMI.kicad_sch (KiCad schematic)
At the start: 45 parts, among them J9 HDMI_19PIN_043, Q3 BSS138, Q4 BSS138, U15 LT8912B

Commit message: Removing component association with previous project (local) libraries.
Parts:
- C73, C74, C75, C76, C77, C78, C79, C80, C81, C82, C83, C84, C85, C86, C87, C88, C89, C90, C91, C92, C93, C94, C95, C96, C97: symbol CholaSymbolsPrjLib:C_Small -> C_Small:C_Small
- D6: footprint CholaFootprintsPrjLib:B540C-13-F -> B540C-13-F:B540C-13-F; symbol CholaSymbolsPrjLib:B540C-13-F -> B540C-13-F:B540C-13-F
- FB2, FB3, FB4, FB5, FB6, FB7, FB8, FB9: footprint CholaFootprintsPrjLib:Ferrite_Bead_100 -> Ferrite_Bead_100:Ferrite_Bead_100; symbol CholaSymbolsPrjLib:GZ2012D101TF -> GZ2012D101TF:GZ2012D101TF
- J9: footprint CholaFootprintsPrjLib:HDMI_CONNECTOR -> HDMI_CONNECTOR:HDMI_CONNECTOR; symbol CholaSymbolsPrjLib:HDMI_19PIN_043 -> HDMI_19PIN_043:HDMI_19PIN_043
- OSC1: footprint CholaFootprintsPrjLib:25MHZ_OSCILLATOR -> 25MHZ_OSCILLATOR:25MHZ_OSCILLATOR; symbol CholaSymbolsPrjLib:OT322525MJBA4SL -> OT322525MJBA4SL:OT322525MJBA4SL
- Q3, Q4: symbol CholaSymbolsPrjLib:BSS138 -> BSS138:BSS138
- R47, R48, R49, R50, R51, R52: symbol CholaSymbolsPrjLib:R_Small_US -> R_Small_US:R_Small_US
- U15: footprint CholaFootprintsPrjLib:LT8912B -> LT8912B:LT8912B; symbol CholaSymbolsPrjLib:LT8912B -> LT8912B:LT8912B
Changed lines of the file:
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@@
 	)
 	(symbol
-		(lib_id "CholaSymbolsPrjLib:C_Small")
+		(lib_id "C_Small:C_Small")
 		(at 295.91 53.34 270)
 		(unit 1)
@@
 	)
 	(symbol
-		(lib_id "CholaSymbolsPrjLib:C_Small")
+		(lib_id "C_Small:C_Small")
 		(at 46.99 254 180)
 		(unit 1)
@@
 	)
 	(symbol
-		(lib_id "CholaSymbolsPrjLib:C_Small")
+		(lib_id "C_Small:C_Small")
 		(at 124.46 254 180)
 		(unit 1)
@@
 	(symbol
 		(lib_name "LT8912B_1")
-		(lib_id "CholaSymbolsPrjLib:LT8912B")
+		(lib_id "LT8912B:LT8912B")
 		(at 264.16 228.6 0)
 		(unit 1)
@@
 			)
 		)
-		(property "Footprint" "CholaFootprintsPrjLib:LT8912B"
+		(property "Footprint" "LT8912B:LT8912B"
 			(at 257.81 247.65 0)
 			(effects
@@
 	)
 	(symbol
-		(lib_id "CholaSymbolsPrjLib:C_Small")
+		(lib_id "C_Small:C_Small")
 		(at 62.23 254 180)
 		(unit 1)
@@
 	)
 	(symbol
-		(lib_id "CholaSymbolsPrjLib:R_Small_US")
+		(lib_id "R_Small_US:R_Small_US")
 		(at 68.58 142.24 180)
 		(unit 1)
@@
 	)
 	(symbol
-		(lib_id "CholaSymbolsPrjLib:C_Small")
+		(lib_id "C_Small:C_Small")
 		(at 109.22 254 180)
 		(unit 1)
@@
 	)
 	(symbol
-		(lib_id "CholaSymbolsPrjLib:C_Small")
+		(lib_id "C_Small:C_Small")
 		(at 116.84 238.76 180)
 		(unit 1)
@@
 	(symbol
 		(lib_name "LT8912B_2")
-		(lib_id "CholaSymbolsPrjLib:LT8912B")
+		(lib_id "LT8912B:LT8912B")
 		(at 264.16 151.13 0)
 		(unit 2)
@@
 			)
 		)
-		(property "Footprint" "CholaFootprintsPrjLib:LT8912B"
+		(property "Footprint" "LT8912B:LT8912B"
 			(at 257.81 170.18 0)
 			(effects
@@
 	)
 	(symbol
-		(lib_id "CholaSymbolsPrjLib:C_Small")
+		(lib_id "C_Small:C_Small")
 		(at 116.84 223.52 180)
 		(unit 1)
@@
 	(symbol
 		(lib_name "GZ2012D101TF_7")
-		(lib_id "CholaSymbolsPrjLib:GZ2012D101TF")
+		(lib_id "GZ2012D101TF:GZ2012D101TF")
 		(at 94.615 233.68 0)
 		(unit 1)
@@
 			)
 		)
-		(property "Footprint" "CholaFootprintsPrjLib:Ferrite_Bead_100"
+		(property "Footprint" "Ferrite_Bead_100:Ferrite_Bead_100"
 			(at 107.188 243.713 0)
 			(effects
@@
 	)
 	(symbol
-		(lib_id "CholaSymbolsPrjLib:C_Small")
+		(lib_id "C_Small:C_Small")
 		(at 54.61 254 180)
 		(unit 1)
@@
 	)
 	(symbol
-		(lib_id "CholaSymbolsPrjLib:C_Small")
+		(lib_id "C_Small:C_Small")
 		(at 53.34 173.99 180)
 		(unit 1)
@@
 	)
 	(symbol
-		(lib_id "CholaSymbolsPrjLib:C_Small")
+		(lib_id "C_Small:C_Small")
 		(at 40.64 173.99 180)
 		(unit 1)
@@
 	)
 	(symbol
-		(lib_id "CholaSymbolsPrjLib:C_Small")
+		(lib_id "C_Small:C_Small")
 		(at 46.99 238.76 180)
 		(unit 1)
@@
 	)
 	(symbol
-		(lib_id "CholaSymbolsPrjLib:HDMI_19PIN_043")
+		(lib_id "HDMI_19PIN_043:HDMI_19PIN_043")
 		(at 368.3 214.63 0)
 		(unit 1)
@@
 			)
 		)
-		(property "Footprint" "CholaFootprintsPrjLib:HDMI_CONNECTOR"
+		(property "Footprint" "HDMI_CONNECTOR:HDMI_CONNECTOR"
 			(at 372.11 246.38 0)
 			(effects
@@
 	)
 	(symbol
-		(lib_id "CholaSymbolsPrjLib:C_Small")
+		(lib_id "C_Small:C_Small")
 		(at 73.66 273.05 180)
 		(unit 1)
@@
 	)
 	(symbol
-		(lib_id "CholaSymbolsPrjLib:B540C-13-F")
+		(lib_id "B540C-13-F:B540C-13-F")
 		(at 346.71 232.41 180)
 		(unit 1)
@@
 			)
 		)
-		(property "Footprint" "CholaFootprintsPrjLib:B540C-13-F"
+		(property "Footprint" "B540C-13-F:B540C-13-F"
 			(at 346.583 220.853 0)
 			(effects
@@
 	(symbol
 		(lib_name "GZ2012D101TF_3")
-		(lib_id "CholaSymbolsPrjLib:GZ2012D101TF")
+		(lib_id "GZ2012D101TF:GZ2012D101TF")
 		(at 32.385 233.68 0)
 		(unit 1)
@@
 			)
 		)
-		(property "Footprint" "CholaFootprintsPrjLib:Ferrite_Bead_100"
+		(property "Footprint" "Ferrite_Bead_100:Ferrite_Bead_100"
 			(at 44.958 243.713 0)
 			(effects
@@
 	)
 	(symbol
-		(lib_id "CholaSymbolsPrjLib:R_Small_US")
+		(lib_id "R_Small_US:R_Small_US")
 		(at 41.91 142.24 180)
 		(unit 1)
@@
 	)
 	(symbol
-		(lib_id "CholaSymbolsPrjLib:C_Small")
+		(lib_id "C_Small:C_Small")
 		(at 46.99 173.99 180)
 		(unit 1)
@@
 	)
 	(symbol
-		(lib_id "CholaSymbolsPrjLib:R_Small_US")
+		(lib_id "R_Small_US:R_Small_US")
 		(at 217.17 54.61 180)
 		(unit 1)
@@
 	)
 	(symbol
-		(lib_id "CholaSymbolsPrjLib:C_Small")
+		(lib_id "C_Small:C_Small")
 		(at 124.46 223.52 180)
 		(unit 1)
@@
 	)
 	(symbol
-		(lib_id "CholaSymbolsPrjLib:C_Small")
+		(lib_id "C_Small:C_Small")
 		(at 109.22 238.76 180)
 		(unit 1)
@@
 	)
 	(symbol
-		(lib_id "CholaSymbolsPrjLib:C_Small")
+		(lib_id "C_Small:C_Small")
 		(at 124.46 238.76 180)
 		(unit 1)
@@
 	)
 	(symbol
-		(lib_id "CholaSymbolsPrjLib:R_Small_US")
+		(lib_id "R_Small_US:R_Small_US")
 		(at 41.91 116.84 180)
 		(unit 1)
@@
 	)
 	(symbol
-		(lib_id "CholaSymbolsPrjLib:GZ2012D101TF")
+		(lib_id "GZ2012D101TF:GZ2012D101TF")
 		(at 94.615 248.92 0)
 		(unit 1)
@@
 			)
 		)
-		(property "Footprint" "CholaFootprintsPrjLib:Ferrite_Bead_100"
+		(property "Footprint" "Ferrite_Bead_100:Ferrite_Bead_100"
 			(at 107.188 258.953 0)
 			(effects
@@
 	)
 	(symbol
-		(lib_id "CholaSymbolsPrjLib:C_Small")
+		(lib_id "C_Small:C_Small")
 		(at 46.99 223.52 180)
 		(unit 1)
@@
 	)
 	(symbol
-		(lib_id "CholaSymbolsPrjLib:C_Small")
+		(lib_id "C_Small:C_Small")
 		(at 54.61 238.76 180)
 		(unit 1)
@@
 	)
 	(symbol
-		(lib_id "CholaSymbolsPrjLib:LT8912B")
+		(lib_id "LT8912B:LT8912B")
 		(at 264.16 68.58 0)
 		(unit 3)
@@
 			)
 		)
-		(property "Footprint" "CholaFootprintsPrjLib:LT8912B"
+		(property "Footprint" "LT8912B:LT8912B"
 			(at 257.81 87.63 0)
 			(effects
@@
 	(symbol
 		(lib_name "GZ2012D101TF_6")
-		(lib_id "CholaSymbolsPrjLib:GZ2012D101TF")
+		(lib_id "GZ2012D101TF:GZ2012D101TF")
 		(at 94.615 218.44 0)
 		(unit 1)
@@
 			)
 		)
-		(property "Footprint" "CholaFootprintsPrjLib:Ferrite_Bead_100"
+		(property "Footprint" "Ferrite_Bead_100:Ferrite_Bead_100"
 			(at 107.188 228.473 0)
 			(effects
@@
 	)
 	(symbol
-		(lib_id "CholaSymbolsPrjLib:C_Small")
+		(lib_id "C_Small:C_Small")
 		(at 116.84 254 180)
 		(unit 1)
@@
 	)
 	(symbol
-		(lib_id "CholaSymbolsPrjLib:C_Small")
+		(lib_id "C_Small:C_Small")
 		(at 88.9 273.05 180)
 		(unit 1)
@@
 	)
 	(symbol
-		(lib_id "CholaSymbolsPrjLib:C_Small")
+		(lib_id "C_Small:C_Small")
 		(at 109.22 223.52 180)
 		(unit 1)
@@
 	(symbol
 		(lib_name "GZ2012D101TF_1")
-		(lib_id "CholaSymbolsPrjLib:GZ2012D101TF")
+		(lib_id "GZ2012D101TF:GZ2012D101TF")
 		(at 30.48 166.37 0)
 		(unit 1)
@@
 			)
 		)
-		(property "Footprint" "CholaFootprintsPrjLib:Ferrite_Bead_100"
+		(property "Footprint" "Ferrite_Bead_100:Ferrite_Bead_100"
 			(at 43.053 176.403 0)
 			(effects
@@
 	(symbol
 		(lib_name "GZ2012D101TF_5")
-		(lib_id "CholaSymbolsPrjLib:GZ2012D101TF")
+		(lib_id "GZ2012D101TF:GZ2012D101TF")
 		(at 59.055 267.97 0)
 		(unit 1)
@@
 			)
 		)
-		(property "Footprint" "CholaFootprintsPrjLib:Ferrite_Bead_100"
+		(property "Footprint" "Ferrite_Bead_100:Ferrite_Bead_100"
 			(at 71.628 278.003 0)
 			(effects
@@
 	)
 	(symbol
-		(lib_id "CholaSymbolsPrjLib:C_Small")
+		(lib_id "C_Small:C_Small")
 		(at 62.23 238.76 180)
 		(unit 1)
@@
 	)
 	(symbol
-		(lib_id "CholaSymbolsPrjLib:C_Small")
+		(lib_id "C_Small:C_Small")
 		(at 81.28 273.05 180)
 		(unit 1)
@@
 	)
 	(symbol
-		(lib_id "CholaSymbolsPrjLib:C_Small")
+		(lib_id "C_Small:C_Small")
 		(at 54.61 223.52 180)
 		(unit 1)
@@
 	)
 	(symbol
-		(lib_id "CholaSymbolsPrjLib:BSS138")
+		(lib_id "BSS138:BSS138")
 		(at 53.34 146.05 270)
 		(unit 1)
@@
 	)
 	(symbol
-		(lib_id "CholaSymbolsPrjLib:C_Small")
+		(lib_id "C_Small:C_Small")
 		(at 62.23 223.52 180)
 		(unit 1)
@@
 	)
 	(symbol
-		(lib_id "CholaSymbolsPrjLib:OT322525MJBA4SL")
+		(lib_id "OT322525MJBA4SL:OT322525MJBA4SL")
 		(at 80.01 173.99 0)
 		(unit 1)
@@
 			)
 		)
-		(property "Footprint" "CholaFootprintsPrjLib:25MHZ_OSCILLATOR"
+		(property "Footprint" "25MHZ_OSCILLATOR:25MHZ_OSCILLATOR"
 			(at 81.534 186.055 0)
 			(effects
@@
 	(symbol
 		(lib_name "GZ2012D101TF_2")
-		(lib_id "CholaSymbolsPrjLib:GZ2012D101TF")
+		(lib_id "GZ2012D101TF:GZ2012D101TF")
 		(at 32.385 218.44 0)
 		(unit 1)
@@
 			)
 		)
-		(property "Footprint" "CholaFootprintsPrjLib:Ferrite_Bead_100"
+		(property "Footprint" "Ferrite_Bead_100:Ferrite_Bead_100"
 			(at 44.958 228.473 0)
 			(effects
@@
 	(symbol
 		(lib_name "GZ2012D101TF_4")
-		(lib_id "CholaSymbolsPrjLib:GZ2012D101TF")
+		(lib_id "GZ2012D101TF:GZ2012D101TF")
 		(at 32.385 248.92 0)
 		(unit 1)
@@
 			)
 		)
-		(property "Footprint" "CholaFootprintsPrjLib:Ferrite_Bead_100"
+		(property "Footprint" "Ferrite_Bead_100:Ferrite_Bead_100"
 			(at 44.958 258.953 0)
 			(effects
@@
 	)
 	(symbol
-		(lib_id "CholaSymbolsPrjLib:BSS138")
+		(lib_id "BSS138:BSS138")
 		(at 53.34 120.65 270)
 		(unit 1)
@@
 	)
 	(symbol
-		(lib_id "CholaSymbolsPrjLib:R_Small_US")
+		(lib_id "R_Small_US:R_Small_US")
 		(at 300.99 48.26 270)
 		(unit 1)
@@
 	)
 	(symbol
-		(lib_id "CholaSymbolsPrjLib:R_Small_US")
+		(lib_id "R_Small_US:R_Small_US")
 		(at 68.58 116.84 180)
 		(unit 1)

Commit message: Fixes, before checks.
Parts:
- C73, C74, C75, C76, C77, C78, C79, C80, C81, C82, C83, C84, C85, C86, C87, C88, C89, C90, C91, C92, C93, C94, C95, C96, C97: symbol C_Small:C_Small -> Device:C_Small
- FB2, FB3, FB4, FB5, FB6, FB7, FB8, FB9: symbol GZ2012D101TF:GZ2012D101TF -> Ferrite_Bead_100:GZ2012D101TF
- J9: symbol HDMI_19PIN_043:HDMI_19PIN_043 -> HDMI_CONNECTOR:HDMI_19PIN_043
- OSC1: symbol OT322525MJBA4SL:OT322525MJBA4SL -> 25MHZ_OSCILLATOR:OT322525MJBA4SL
- Q3, Q4: symbol BSS138:BSS138 -> Transistor_FET:BSS138
- R47, R48, R49, R50, R51, R52: symbol R_Small_US:R_Small_US -> Device:R_Small_US
Changed lines of the file:
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@@
 	)
 	(symbol
-		(lib_id "C_Small:C_Small")
+		(lib_id "Device:C_Small")
 		(at 295.91 53.34 270)
 		(unit 1)
@@
 	)
 	(symbol
-		(lib_id "C_Small:C_Small")
+		(lib_id "Device:C_Small")
 		(at 46.99 254 180)
 		(unit 1)
@@
 	)
 	(symbol
-		(lib_id "C_Small:C_Small")
+		(lib_id "Device:C_Small")
 		(at 124.46 254 180)
 		(unit 1)
@@
 	)
 	(symbol
-		(lib_id "C_Small:C_Small")
+		(lib_id "Device:C_Small")
 		(at 62.23 254 180)
 		(unit 1)
@@
 	)
 	(symbol
-		(lib_id "R_Small_US:R_Small_US")
+		(lib_id "Device:R_Small_US")
 		(at 68.58 142.24 180)
 		(unit 1)
@@
 	)
 	(symbol
-		(lib_id "C_Small:C_Small")
+		(lib_id "Device:C_Small")
 		(at 109.22 254 180)
 		(unit 1)
@@
 	)
 	(symbol
-		(lib_id "C_Small:C_Small")
+		(lib_id "Device:C_Small")
 		(at 116.84 238.76 180)
 		(unit 1)
@@
 	)
 	(symbol
-		(lib_id "C_Small:C_Small")
+		(lib_id "Device:C_Small")
 		(at 116.84 223.52 180)
 		(unit 1)
@@
 	(symbol
 		(lib_name "GZ2012D101TF_7")
-		(lib_id "GZ2012D101TF:GZ2012D101TF")
+		(lib_id "Ferrite_Bead_100:GZ2012D101TF")
 		(at 94.615 233.68 0)
 		(unit 1)
@@
 	)
 	(symbol
-		(lib_id "C_Small:C_Small")
+		(lib_id "Device:C_Small")
 		(at 54.61 254 180)
 		(unit 1)
@@
 	)
 	(symbol
-		(lib_id "C_Small:C_Small")
+		(lib_id "Device:C_Small")
 		(at 53.34 173.99 180)
 		(unit 1)
@@
 	)
 	(symbol
-		(lib_id "C_Small:C_Small")
+		(lib_id "Device:C_Small")
 		(at 40.64 173.99 180)
 		(unit 1)
@@
 	)
 	(symbol
-		(lib_id "C_Small:C_Small")
+		(lib_id "Device:C_Small")
 		(at 46.99 238.76 180)
 		(unit 1)
@@
 	)
 	(symbol
-		(lib_id "HDMI_19PIN_043:HDMI_19PIN_043")
+		(lib_id "HDMI_CONNECTOR:HDMI_19PIN_043")
 		(at 368.3 214.63 0)
 		(unit 1)
@@
 	)
 	(symbol
-		(lib_id "C_Small:C_Small")
+		(lib_id "Device:C_Small")
 		(at 73.66 273.05 180)
 		(unit 1)
@@
 	(symbol
 		(lib_name "GZ2012D101TF_3")
-		(lib_id "GZ2012D101TF:GZ2012D101TF")
+		(lib_id "Ferrite_Bead_100:GZ2012D101TF")
 		(at 32.385 233.68 0)
 		(unit 1)
@@
 	)
 	(symbol
-		(lib_id "R_Small_US:R_Small_US")
+		(lib_id "Device:R_Small_US")
 		(at 41.91 142.24 180)
 		(unit 1)
@@
 	)
 	(symbol
-		(lib_id "C_Small:C_Small")
+		(lib_id "Device:C_Small")
 		(at 46.99 173.99 180)
 		(unit 1)
@@
 	)
 	(symbol
-		(lib_id "R_Small_US:R_Small_US")
+		(lib_id "Device:R_Small_US")
 		(at 217.17 54.61 180)
 		(unit 1)
@@
 	)
 	(symbol
-		(lib_id "C_Small:C_Small")
+		(lib_id "Device:C_Small")
 		(at 124.46 223.52 180)
 		(unit 1)
@@
 	)
 	(symbol
-		(lib_id "C_Small:C_Small")
+		(lib_id "Device:C_Small")
 		(at 109.22 238.76 180)
 		(unit 1)
@@
 	)
 	(symbol
-		(lib_id "C_Small:C_Small")
+		(lib_id "Device:C_Small")
 		(at 124.46 238.76 180)
 		(unit 1)
@@
 	)
 	(symbol
-		(lib_id "R_Small_US:R_Small_US")
+		(lib_id "Device:R_Small_US")
 		(at 41.91 116.84 180)
 		(unit 1)
@@
 	)
 	(symbol
-		(lib_id "GZ2012D101TF:GZ2012D101TF")
+		(lib_id "Ferrite_Bead_100:GZ2012D101TF")
 		(at 94.615 248.92 0)
 		(unit 1)
@@
 	)
 	(symbol
-		(lib_id "C_Small:C_Small")
+		(lib_id "Device:C_Small")
 		(at 46.99 223.52 180)
 		(unit 1)
@@
 	)
 	(symbol
-		(lib_id "C_Small:C_Small")
+		(lib_id "Device:C_Small")
 		(at 54.61 238.76 180)
 		(unit 1)
@@
 	(symbol
 		(lib_name "GZ2012D101TF_6")
-		(lib_id "GZ2012D101TF:GZ2012D101TF")
+		(lib_id "Ferrite_Bead_100:GZ2012D101TF")
 		(at 94.615 218.44 0)
 		(unit 1)
@@
 	)
 	(symbol
-		(lib_id "C_Small:C_Small")
+		(lib_id "Device:C_Small")
 		(at 116.84 254 180)
 		(unit 1)
@@
 	)
 	(symbol
-		(lib_id "C_Small:C_Small")
+		(lib_id "Device:C_Small")
 		(at 88.9 273.05 180)
 		(unit 1)
@@
 	)
 	(symbol
-		(lib_id "C_Small:C_Small")
+		(lib_id "Device:C_Small")
 		(at 109.22 223.52 180)
 		(unit 1)
@@
 	(symbol
 		(lib_name "GZ2012D101TF_1")
-		(lib_id "GZ2012D101TF:GZ2012D101TF")
+		(lib_id "Ferrite_Bead_100:GZ2012D101TF")
 		(at 30.48 166.37 0)
 		(unit 1)
@@
 	(symbol
 		(lib_name "GZ2012D101TF_5")
-		(lib_id "GZ2012D101TF:GZ2012D101TF")
+		(lib_id "Ferrite_Bead_100:GZ2012D101TF")
 		(at 59.055 267.97 0)
 		(unit 1)
@@
 	)
 	(symbol
-		(lib_id "C_Small:C_Small")
+		(lib_id "Device:C_Small")
 		(at 62.23 238.76 180)
 		(unit 1)
@@
 	)
 	(symbol
-		(lib_id "C_Small:C_Small")
+		(lib_id "Device:C_Small")
 		(at 81.28 273.05 180)
 		(unit 1)
@@
 	)
 	(symbol
-		(lib_id "C_Small:C_Small")
+		(lib_id "Device:C_Small")
 		(at 54.61 223.52 180)
 		(unit 1)
@@
 	)
 	(symbol
-		(lib_id "BSS138:BSS138")
+		(lib_id "Transistor_FET:BSS138")
 		(at 53.34 146.05 270)
 		(unit 1)
@@
 	)
 	(symbol
-		(lib_id "C_Small:C_Small")
+		(lib_id "Device:C_Small")
 		(at 62.23 223.52 180)
 		(unit 1)
@@
 	)
 	(symbol
-		(lib_id "OT322525MJBA4SL:OT322525MJBA4SL")
+		(lib_id "25MHZ_OSCILLATOR:OT322525MJBA4SL")
 		(at 80.01 173.99 0)
 		(unit 1)
@@
 	(symbol
 		(lib_name "GZ2012D101TF_2")
-		(lib_id "GZ2012D101TF:GZ2012D101TF")
+		(lib_id "Ferrite_Bead_100:GZ2012D101TF")
 		(at 32.385 218.44 0)
 		(unit 1)
@@
 	(symbol
 		(lib_name "GZ2012D101TF_4")
-		(lib_id "GZ2012D101TF:GZ2012D101TF")
+		(lib_id "Ferrite_Bead_100:GZ2012D101TF")
 		(at 32.385 248.92 0)
 		(unit 1)
@@
 	)
 	(symbol
-		(lib_id "BSS138:BSS138")
+		(lib_id "Transistor_FET:BSS138")
 		(at 53.34 120.65 270)
 		(unit 1)
@@
 	)
 	(symbol
-		(lib_id "R_Small_US:R_Small_US")
+		(lib_id "Device:R_Small_US")
 		(at 300.99 48.26 270)
 		(unit 1)
@@
 	)
 	(symbol
-		(lib_id "R_Small_US:R_Small_US")
+		(lib_id "Device:R_Small_US")
 		(at 68.58 116.84 180)
 		(unit 1)
