File: Tangenta/Ethernet_Switch.kicad_sch (KiCad schematic)
At the start: 48 parts, among them J26 Conn_01x08_Pin, U21 RTL8367S-CG, X2 X322525MOB4SI

Commit message: CAP_L5, CR2032_HOL, Ferrite_Bead, XTAL_24-25
Parts:
- C195, C196: footprint CAP_L5:CAP_L5 -> CholaFootprintsPrjLib:CAP_L5
- X2: footprint XTAL_25MHZ:XTAL_25MHZ -> CholaFootprintsPrjLib:XTAL_25MHZ
Changed lines of the file:
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@@
       (effects (font (size 1.27 1.27)) hide)
     )
-    (property "Footprint" "XTAL_25MHZ:XTAL_25MHZ" (at 223.139 271.526 0)
+    (property "Footprint" "CholaFootprintsPrjLib:XTAL_25MHZ" (at 223.139 271.526 0)
       (effects (font (size 1.27 1.27) italic) hide)
     )
@@
       (effects (font (size 1.27 1.27)) (justify left))
     )
-    (property "Footprint" "CAP_L5:CAP_L5" (at 372.11 238.76 0)
+    (property "Footprint" "CholaFootprintsPrjLib:CAP_L5" (at 372.11 238.76 0)
       (effects (font (size 1.27 1.27) italic) hide)
     )
@@
     )
   )
-  (symbol (lib_id "CholaSymbolsPrjLib:16CE47FSS") (at 373.38 235.585 0) (unit 1)
+  (symbol (lib_name "16CE47FSS_1") (lib_id "CholaSymbolsPrjLib:16CE47FSS") (at 373.38 235.585 0) (unit 1)
     (in_bom yes) (on_board yes) (dnp no)
     (property "Reference" "C196" (at 374.65 233.68 0)
@@
       (effects (font (size 1.27 1.27)) (justify left))
     )
-    (property "Footprint" "CAP_L5:CAP_L5" (at 372.11 253.365 0)
+    (property "Footprint" "CholaFootprintsPrjLib:CAP_L5" (at 372.11 253.365 0)
       (effects (font (size 1.27 1.27) italic) hide)
     )

Commit message: CAP_L5, NTZD3154NT1G
Parts:
- C193, C194: footprint CAP_TANTAL_A:CAP_TANTAL_A -> CholaFootprintsPrjLib:CAP_TANTAL_A
Changed lines of the file:
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@@
     )
   )
-  (symbol (lib_id "CholaSymbolsPrjLib:CA45-A-6_3V-47UF-K") (at 361.95 236.22 270) (mirror x) (unit 1)
+  (symbol (lib_name "CA45-A-6_3V-47UF-K_1") (lib_id "CholaSymbolsPrjLib:CA45-A-6_3V-47UF-K") (at 361.95 236.22 270) (mirror x) (unit 1)
     (in_bom yes) (on_board yes) (dnp no)
     (property "Reference" "C194" (at 367.665 234.315 90)
@@
       (effects (font (size 1.27 1.27)) (justify right))
     )
-    (property "Footprint" "CAP_TANTAL_A:CAP_TANTAL_A" (at 350.266 233.172 0)
+    (property "Footprint" "CholaFootprintsPrjLib:CAP_TANTAL_A" (at 350.266 233.172 0)
       (effects (font (size 1.27 1.27) italic) hide)
     )
@@
       (effects (font (size 1.27 1.27)) (justify right))
     )
-    (property "Footprint" "CAP_TANTAL_A:CAP_TANTAL_A" (at 350.266 218.567 0)
+    (property "Footprint" "CholaFootprintsPrjLib:CAP_TANTAL_A" (at 350.266 218.567 0)
       (effects (font (size 1.27 1.27) italic) hide)
     )
@@
     )
   )
-  (symbol (lib_name "16CE47FSS_1") (lib_id "CholaSymbolsPrjLib:16CE47FSS") (at 373.38 235.585 0) (unit 1)
+  (symbol (lib_id "CholaSymbolsPrjLib:16CE47FSS") (at 373.38 235.585 0) (unit 1)
     (in_bom yes) (on_board yes) (dnp no)
     (property "Reference" "C196" (at 374.65 233.68 0)

Commit message: Removing component association with previous project (local) libraries.
Parts:
- C170, C171, C172, C173, C174, C175, C176, C177, C178, C179, C180, C181, C182, C183, C184, C185, C186, C187, C188, C189, C190, C191, C192: symbol CholaSymbolsPrjLib:C_Small -> C_Small:C_Small
- C193, C194: footprint CholaFootprintsPrjLib:CAP_TANTAL_A -> CAP_TANTAL_A:CAP_TANTAL_A; symbol CholaSymbolsPrjLib:CA45-A-6_3V-47UF-K -> CA45-A-6_3V-47UF-K:CA45-A-6_3V-47UF-K
- C195, C196: footprint CholaFootprintsPrjLib:CAP_L5 -> CAP_L5:CAP_L5; symbol CholaSymbolsPrjLib:16CE47FSS -> 16CE47FSS:16CE47FSS
- J26: symbol CholaSymbolsPrjLib:Conn_01x08_Pin -> Conn_01x08_Pin:Conn_01x08_Pin
- R152, R153, R154, R155, R156, R157, R158, R159, R160, R161, R162, R163, R164, R165, R166, R167, R168, R169: symbol CholaSymbolsPrjLib:R_Small_US -> R_Small_US:R_Small_US
- U21: footprint CholaFootprintsPrjLib:RTL8367S-CG -> RTL8367S-CG:RTL8367S-CG; symbol CholaSymbolsPrjLib:RTL8367S-CG -> RTL8367S-CG:RTL8367S-CG
- X2: footprint CholaFootprintsPrjLib:XTAL_25MHZ -> XTAL_25MHZ:XTAL_25MHZ; symbol CholaSymbolsPrjLib:X322525MOB4SI -> X322525MOB4SI:X322525MOB4SI
Changed lines of the file:
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@@
 	)
 	(symbol
-		(lib_id "CholaSymbolsPrjLib:R_Small_US")
+		(lib_id "R_Small_US:R_Small_US")
 		(at 191.135 234.315 180)
 		(unit 1)
@@
 	)
 	(symbol
-		(lib_id "CholaSymbolsPrjLib:R_Small_US")
+		(lib_id "R_Small_US:R_Small_US")
 		(at 213.995 234.315 180)
 		(unit 1)
@@
 	)
 	(symbol
-		(lib_id "CholaSymbolsPrjLib:C_Small")
+		(lib_id "C_Small:C_Small")
 		(at 331.47 235.585 180)
 		(unit 1)
@@
 	)
 	(symbol
-		(lib_id "CholaSymbolsPrjLib:C_Small")
+		(lib_id "C_Small:C_Small")
 		(at 345.44 235.585 180)
 		(unit 1)
@@
 	)
 	(symbol
-		(lib_id "CholaSymbolsPrjLib:C_Small")
+		(lib_id "C_Small:C_Small")
 		(at 73.025 67.31 270)
 		(unit 1)
@@
 	)
 	(symbol
-		(lib_id "CholaSymbolsPrjLib:C_Small")
+		(lib_id "C_Small:C_Small")
 		(at 316.23 235.585 180)
 		(unit 1)
@@
 	)
 	(symbol
-		(lib_id "CholaSymbolsPrjLib:C_Small")
+		(lib_id "C_Small:C_Small")
 		(at 222.25 269.24 180)
 		(unit 1)
@@
 	)
 	(symbol
-		(lib_id "CholaSymbolsPrjLib:C_Small")
+		(lib_id "C_Small:C_Small")
 		(at 337.82 220.98 180)
 		(unit 1)
@@
 	)
 	(symbol
-		(lib_id "CholaSymbolsPrjLib:R_Small_US")
+		(lib_id "R_Small_US:R_Small_US")
 		(at 99.695 275.59 90)
 		(unit 1)
@@
 	)
 	(symbol
-		(lib_id "CholaSymbolsPrjLib:C_Small")
+		(lib_id "C_Small:C_Small")
 		(at 73.025 74.93 270)
 		(unit 1)
@@
 	)
 	(symbol
-		(lib_id "CholaSymbolsPrjLib:R_Small_US")
+		(lib_id "R_Small_US:R_Small_US")
 		(at 99.695 270.51 90)
 		(unit 1)
@@
 	)
 	(symbol
-		(lib_id "CholaSymbolsPrjLib:C_Small")
+		(lib_id "C_Small:C_Small")
 		(at 62.23 49.53 270)
 		(unit 1)
@@
 	)
 	(symbol
-		(lib_id "CholaSymbolsPrjLib:C_Small")
+		(lib_id "C_Small:C_Small")
 		(at 323.85 235.585 180)
 		(unit 1)
@@
 	)
 	(symbol
-		(lib_id "CholaSymbolsPrjLib:R_Small_US")
+		(lib_id "R_Small_US:R_Small_US")
 		(at 278.765 99.695 180)
 		(unit 1)
@@
 	)
 	(symbol
-		(lib_id "CholaSymbolsPrjLib:RTL8367S-CG")
+		(lib_id "RTL8367S-CG:RTL8367S-CG")
 		(at 184.785 133.35 0)
 		(unit 1)
@@
 			)
 		)
-		(property "Footprint" "CholaFootprintsPrjLib:RTL8367S-CG"
+		(property "Footprint" "RTL8367S-CG:RTL8367S-CG"
 			(at 184.785 143.51 0)
 			(effects
@@
 	)
 	(symbol
-		(lib_id "CholaSymbolsPrjLib:R_Small_US")
+		(lib_id "R_Small_US:R_Small_US")
 		(at 264.795 138.43 90)
 		(unit 1)
@@
 	)
 	(symbol
-		(lib_id "CholaSymbolsPrjLib:C_Small")
+		(lib_id "C_Small:C_Small")
 		(at 351.79 235.585 180)
 		(unit 1)
@@
 	)
 	(symbol
-		(lib_id "CholaSymbolsPrjLib:X322525MOB4SI")
+		(lib_id "X322525MOB4SI:X322525MOB4SI")
 		(at 231.775 255.27 0)
 		(unit 1)
@@
 			)
 		)
-		(property "Footprint" "CholaFootprintsPrjLib:XTAL_25MHZ"
+		(property "Footprint" "XTAL_25MHZ:XTAL_25MHZ"
 			(at 223.139 271.526 0)
 			(effects
@@
 	)
 	(symbol
-		(lib_id "CholaSymbolsPrjLib:R_Small_US")
+		(lib_id "R_Small_US:R_Small_US")
 		(at 193.675 234.315 180)
 		(unit 1)
@@
 	)
 	(symbol
-		(lib_id "CholaSymbolsPrjLib:C_Small")
+		(lib_id "C_Small:C_Small")
 		(at 316.23 220.98 180)
 		(unit 1)
@@
 	)
 	(symbol
-		(lib_id "CholaSymbolsPrjLib:R_Small_US")
+		(lib_id "R_Small_US:R_Small_US")
 		(at 188.595 234.315 180)
 		(unit 1)
@@
 	)
 	(symbol
-		(lib_id "CholaSymbolsPrjLib:R_Small_US")
+		(lib_id "R_Small_US:R_Small_US")
 		(at 232.41 266.7 90)
 		(unit 1)
@@
 	)
 	(symbol
-		(lib_id "CholaSymbolsPrjLib:R_Small_US")
+		(lib_id "R_Small_US:R_Small_US")
 		(at 100.965 110.49 90)
 		(unit 1)
@@
 	(symbol
 		(lib_name "CA45-A-6_3V-47UF-K_1")
-		(lib_id "CholaSymbolsPrjLib:CA45-A-6_3V-47UF-K")
+		(lib_id "CA45-A-6_3V-47UF-K:CA45-A-6_3V-47UF-K")
 		(at 361.95 236.22 270)
 		(mirror x)
@@
 			)
 		)
-		(property "Footprint" "CholaFootprintsPrjLib:CAP_TANTAL_A"
+		(property "Footprint" "CAP_TANTAL_A:CAP_TANTAL_A"
 			(at 350.266 233.172 0)
 			(effects
@@
 	)
 	(symbol
-		(lib_id "CholaSymbolsPrjLib:R_Small_US")
+		(lib_id "R_Small_US:R_Small_US")
 		(at 99.695 264.16 90)
 		(unit 1)
@@
 	)
 	(symbol
-		(lib_id "CholaSymbolsPrjLib:R_Small_US")
+		(lib_id "R_Small_US:R_Small_US")
 		(at 203.835 234.315 180)
 		(unit 1)
@@
 	)
 	(symbol
-		(lib_id "CholaSymbolsPrjLib:C_Small")
+		(lib_id "C_Small:C_Small")
 		(at 73.025 52.07 270)
 		(unit 1)
@@
 	)
 	(symbol
-		(lib_id "CholaSymbolsPrjLib:R_Small_US")
+		(lib_id "R_Small_US:R_Small_US")
 		(at 101.6 252.73 90)
 		(unit 1)
@@
 	)
 	(symbol
-		(lib_id "CholaSymbolsPrjLib:R_Small_US")
+		(lib_id "R_Small_US:R_Small_US")
 		(at 201.295 234.315 180)
 		(unit 1)
@@
 	)
 	(symbol
-		(lib_id "CholaSymbolsPrjLib:R_Small_US")
+		(lib_id "R_Small_US:R_Small_US")
 		(at 99.695 259.08 90)
 		(unit 1)
@@
 	)
 	(symbol
-		(lib_id "CholaSymbolsPrjLib:R_Small_US")
+		(lib_id "R_Small_US:R_Small_US")
 		(at 101.6 247.65 90)
 		(unit 1)
@@
 	)
 	(symbol
-		(lib_id "CholaSymbolsPrjLib:Conn_01x08_Pin")
+		(lib_id "Conn_01x08_Pin:Conn_01x08_Pin")
 		(at 144.78 265.43 0)
 		(unit 1)
@@
 	)
 	(symbol
-		(lib_id "CholaSymbolsPrjLib:16CE47FSS")
+		(lib_id "16CE47FSS:16CE47FSS")
 		(at 373.38 220.98 0)
 		(unit 1)
@@
 			)
 		)
-		(property "Footprint" "CholaFootprintsPrjLib:CAP_L5"
+		(property "Footprint" "CAP_L5:CAP_L5"
 			(at 372.11 238.76 0)
 			(effects
@@
 	)
 	(symbol
-		(lib_id "CholaSymbolsPrjLib:C_Small")
+		(lib_id "C_Small:C_Small")
 		(at 337.82 235.585 180)
 		(unit 1)
@@
 	)
 	(symbol
-		(lib_id "CholaSymbolsPrjLib:C_Small")
+		(lib_id "C_Small:C_Small")
 		(at 278.765 110.49 180)
 		(unit 1)
@@
 	)
 	(symbol
-		(lib_id "CholaSymbolsPrjLib:C_Small")
+		(lib_id "C_Small:C_Small")
 		(at 62.23 72.39 270)
 		(unit 1)
@@
 	)
 	(symbol
-		(lib_id "CholaSymbolsPrjLib:C_Small")
+		(lib_id "C_Small:C_Small")
 		(at 351.79 220.98 180)
 		(unit 1)
@@
 	)
 	(symbol
-		(lib_id "CholaSymbolsPrjLib:C_Small")
+		(lib_id "C_Small:C_Small")
 		(at 62.23 64.77 270)
 		(unit 1)
@@
 	)
 	(symbol
-		(lib_id "CholaSymbolsPrjLib:R_Small_US")
+		(lib_id "R_Small_US:R_Small_US")
 		(at 264.795 123.19 90)
 		(unit 1)
@@
 	)
 	(symbol
-		(lib_id "CholaSymbolsPrjLib:R_Small_US")
+		(lib_id "R_Small_US:R_Small_US")
 		(at 264.795 130.81 90)
 		(unit 1)
@@
 	)
 	(symbol
-		(lib_id "CholaSymbolsPrjLib:C_Small")
+		(lib_id "C_Small:C_Small")
 		(at 345.44 220.98 180)
 		(unit 1)
@@
 	)
 	(symbol
-		(lib_id "CholaSymbolsPrjLib:CA45-A-6_3V-47UF-K")
+		(lib_id "CA45-A-6_3V-47UF-K:CA45-A-6_3V-47UF-K")
 		(at 361.95 221.615 270)
 		(mirror x)
@@
 			)
 		)
-		(property "Footprint" "CholaFootprintsPrjLib:CAP_TANTAL_A"
+		(property "Footprint" "CAP_TANTAL_A:CAP_TANTAL_A"
 			(at 350.266 218.567 0)
 			(effects
@@
 	)
 	(symbol
-		(lib_id "CholaSymbolsPrjLib:C_Small")
+		(lib_id "C_Small:C_Small")
 		(at 62.23 57.15 270)
 		(unit 1)
@@
 	)
 	(symbol
-		(lib_id "CholaSymbolsPrjLib:16CE47FSS")
+		(lib_id "16CE47FSS:16CE47FSS")
 		(at 373.38 235.585 0)
 		(unit 1)
@@
 			)
 		)
-		(property "Footprint" "CholaFootprintsPrjLib:CAP_L5"
+		(property "Footprint" "CAP_L5:CAP_L5"
 			(at 372.11 253.365 0)
 			(effects
@@
 	)
 	(symbol
-		(lib_id "CholaSymbolsPrjLib:C_Small")
+		(lib_id "C_Small:C_Small")
 		(at 241.3 269.24 180)
 		(unit 1)
@@
 	)
 	(symbol
-		(lib_id "CholaSymbolsPrjLib:C_Small")
+		(lib_id "C_Small:C_Small")
 		(at 323.85 220.98 180)
 		(unit 1)
@@
 	)
 	(symbol
-		(lib_id "CholaSymbolsPrjLib:C_Small")
+		(lib_id "C_Small:C_Small")
 		(at 331.47 220.98 180)
 		(unit 1)
@@
 	)
 	(symbol
-		(lib_id "CholaSymbolsPrjLib:C_Small")
+		(lib_id "C_Small:C_Small")
 		(at 73.025 59.69 270)
 		(unit 1)

Commit message: Fixes, continued...
Parts:
- C170, C171, C172, C173, C174, C175, C176, C177, C178, C179, C180, C181, C182, C183, C184, C185, C186, C187, C188, C189, C190, C191, C192: symbol C_Small:C_Small -> Device:C_Small
- J26: symbol Conn_01x08_Pin:Conn_01x08_Pin -> Connector_Generic:Conn_01x08_Pin
- R152, R153, R154, R155, R156, R157, R158, R159, R160, R161, R162, R163, R164, R165, R166, R167, R168, R169: symbol R_Small_US:R_Small_US -> Device:R_Small_US
Connections:
- net 1V1: no longer C182.2, C184.2, C186.2, C188.2, C190.2, C192.2
- net 3V3: no longer C181.2, C183.2, C185.2, C187.2, C189.2, C191.2, R157.2, R166.2, R167.2, R169.2
- net DL: no longer R167.1
- net EN_PL: no longer R168.1
- net GNDREF: no longer C178.1, C179.1, C180.1, C181.1, C182.1, C183.1, C184.1, C185.1, C186.1, C187.1, C188.1, C189.1, C190.1, C191.1, C192.1, J26.1 (Pin_1), R156.1, R158.2, R159.1, R160.1, R161.1, R162.1, R163.1, R164.1, R168.2
- net GPIO_03: no longer J26.4 (Pin_4)
- net I2C_SCL: no longer R155.2
- net I2C_SDA: no longer R153.2
- net MDIREF: no longer R156.2
- net MGMT_CLK: no longer R154.1, R155.1
- net MGMT_DATA: no longer R152.1, R153.1
- net P0_MDI_A_N: no longer C174.1
- net P0_MDI_A_P: no longer C170.1
- net P0_MDI_B_N: no longer C175.1
- net P0_MDI_B_P: no longer C171.1
- net P0_MDI_C_N: no longer C176.1
- net P0_MDI_C_P: no longer C172.1
- net P0_MDI_D_N: no longer C177.1
- net P0_MDI_D_P: no longer C173.1
- net P1_LED_0: no longer R166.1
- net RXD_GPIO_01: no longer J26.2 (Pin_2)
- net SMI_SEL: no longer R157.1, R158.1
- net SPI_CLK: no longer J26.5 (Pin_5)
- net SPI_CS: no longer J26.8 (Pin_8)
- net SPI_D0: no longer J26.6 (Pin_6)
- net SPI_D1: no longer J26.7 (Pin_7)
- net TXD_GPIO_02: no longer J26.3 (Pin_3)
- net UPLINK_A_N: no longer C174.2
- net UPLINK_A_P: no longer C170.2
- net UPLINK_B_N: no longer C175.2
- net UPLINK_B_P: no longer C171.2
- net UPLINK_C_N: no longer C176.2
- net UPLINK_C_P: no longer C172.2
- net UPLINK_D_N: no longer C177.2
- net UPLINK_D_P: no longer C173.2
- net UPLINK_MDC: no longer R154.2
- net UPLINK_MDIO: no longer R152.2
- net XTALI: no longer C178.2, R165.1
- net XTALO: no longer C179.2, R165.2
- net nRESET: no longer C180.2, R169.1
- net at U21.51 (M2P_TXCLK/M2M_RXCLK/RG2_RXCLK/GPIO07): no longer R160.2
- net at U21.60 (EN_SWR): no longer R164.2
- net at U21.50 (M2P_RXCLK/M2M_TXCLK/RG2_TXCLK/GPIO06): no longer R159.2
- net at U21.52 (M2P_TXEN/M2M_RXDV/RG2_RXCTL/GPIO08): no longer R161.2
- net at U21.55 (M2P_TXD2/M2M_RXD2/RG2_RXD2/GPIO11): no longer R162.2
- net at U21.56 (M2P_TXD3/M2M_RXD3/RG2_RXD3/GPIO12): no longer R163.2
Changed lines of the file:
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@@
 	)
 	(symbol
-		(lib_id "R_Small_US:R_Small_US")
+		(lib_id "Device:R_Small_US")
 		(at 191.135 234.315 180)
 		(unit 1)
@@
 	)
 	(symbol
-		(lib_id "R_Small_US:R_Small_US")
+		(lib_id "Device:R_Small_US")
 		(at 213.995 234.315 180)
 		(unit 1)
@@
 	)
 	(symbol
-		(lib_id "C_Small:C_Small")
+		(lib_id "Device:C_Small")
 		(at 331.47 235.585 180)
 		(unit 1)
@@
 	)
 	(symbol
-		(lib_id "C_Small:C_Small")
+		(lib_id "Device:C_Small")
 		(at 345.44 235.585 180)
 		(unit 1)
@@
 	)
 	(symbol
-		(lib_id "C_Small:C_Small")
+		(lib_id "Device:C_Small")
 		(at 73.025 67.31 270)
 		(unit 1)
@@
 	)
 	(symbol
-		(lib_id "C_Small:C_Small")
+		(lib_id "Device:C_Small")
 		(at 316.23 235.585 180)
 		(unit 1)
@@
 	)
 	(symbol
-		(lib_id "C_Small:C_Small")
+		(lib_id "Device:C_Small")
 		(at 222.25 269.24 180)
 		(unit 1)
@@
 	)
 	(symbol
-		(lib_id "C_Small:C_Small")
+		(lib_id "Device:C_Small")
 		(at 337.82 220.98 180)
 		(unit 1)
@@
 	)
 	(symbol
-		(lib_id "R_Small_US:R_Small_US")
+		(lib_id "Device:R_Small_US")
 		(at 99.695 275.59 90)
 		(unit 1)
@@
 	)
 	(symbol
-		(lib_id "C_Small:C_Small")
+		(lib_id "Device:C_Small")
 		(at 73.025 74.93 270)
 		(unit 1)
@@
 	)
 	(symbol
-		(lib_id "R_Small_US:R_Small_US")
+		(lib_id "Device:R_Small_US")
 		(at 99.695 270.51 90)
 		(unit 1)
@@
 	)
 	(symbol
-		(lib_id "C_Small:C_Small")
+		(lib_id "Device:C_Small")
 		(at 62.23 49.53 270)
 		(unit 1)
@@
 	)
 	(symbol
-		(lib_id "C_Small:C_Small")
+		(lib_id "Device:C_Small")
 		(at 323.85 235.585 180)
 		(unit 1)
@@
 	)
 	(symbol
-		(lib_id "R_Small_US:R_Small_US")
+		(lib_id "Device:R_Small_US")
 		(at 278.765 99.695 180)
 		(unit 1)
@@
 	)
 	(symbol
-		(lib_id "R_Small_US:R_Small_US")
+		(lib_id "Device:R_Small_US")
 		(at 264.795 138.43 90)
 		(unit 1)
@@
 	)
 	(symbol
-		(lib_id "C_Small:C_Small")
+		(lib_id "Device:C_Small")
 		(at 351.79 235.585 180)
 		(unit 1)
@@
 	)
 	(symbol
-		(lib_id "R_Small_US:R_Small_US")
+		(lib_id "Device:R_Small_US")
 		(at 193.675 234.315 180)
 		(unit 1)
@@
 	)
 	(symbol
-		(lib_id "C_Small:C_Small")
+		(lib_id "Device:C_Small")
 		(at 316.23 220.98 180)
 		(unit 1)
@@
 	)
 	(symbol
-		(lib_id "R_Small_US:R_Small_US")
+		(lib_id "Device:R_Small_US")
 		(at 188.595 234.315 180)
 		(unit 1)
@@
 	)
 	(symbol
-		(lib_id "R_Small_US:R_Small_US")
+		(lib_id "Device:R_Small_US")
 		(at 232.41 266.7 90)
 		(unit 1)
@@
 	)
 	(symbol
-		(lib_id "R_Small_US:R_Small_US")
+		(lib_id "Device:R_Small_US")
 		(at 100.965 110.49 90)
 		(unit 1)
@@
 	)
 	(symbol
-		(lib_id "R_Small_US:R_Small_US")
+		(lib_id "Device:R_Small_US")
 		(at 99.695 264.16 90)
 		(unit 1)
@@
 	)
 	(symbol
-		(lib_id "R_Small_US:R_Small_US")
+		(lib_id "Device:R_Small_US")
 		(at 203.835 234.315 180)
 		(unit 1)
@@
 	)
 	(symbol
-		(lib_id "C_Small:C_Small")
+		(lib_id "Device:C_Small")
 		(at 73.025 52.07 270)
 		(unit 1)
@@
 	)
 	(symbol
-		(lib_id "R_Small_US:R_Small_US")
+		(lib_id "Device:R_Small_US")
 		(at 101.6 252.73 90)
 		(unit 1)
@@
 	)
 	(symbol
-		(lib_id "R_Small_US:R_Small_US")
+		(lib_id "Device:R_Small_US")
 		(at 201.295 234.315 180)
 		(unit 1)
@@
 	)
 	(symbol
-		(lib_id "R_Small_US:R_Small_US")
+		(lib_id "Device:R_Small_US")
 		(at 99.695 259.08 90)
 		(unit 1)
@@
 	)
 	(symbol
-		(lib_id "R_Small_US:R_Small_US")
+		(lib_id "Device:R_Small_US")
 		(at 101.6 247.65 90)
 		(unit 1)
@@
 	)
 	(symbol
-		(lib_id "Conn_01x08_Pin:Conn_01x08_Pin")
+		(lib_id "Connector_Generic:Conn_01x08_Pin")
 		(at 144.78 265.43 0)
 		(unit 1)
@@
 	)
 	(symbol
-		(lib_id "C_Small:C_Small")
+		(lib_id "Device:C_Small")
 		(at 337.82 235.585 180)
 		(unit 1)
@@
 	)
 	(symbol
-		(lib_id "C_Small:C_Small")
+		(lib_id "Device:C_Small")
 		(at 278.765 110.49 180)
 		(unit 1)
@@
 	)
 	(symbol
-		(lib_id "C_Small:C_Small")
+		(lib_id "Device:C_Small")
 		(at 62.23 72.39 270)
 		(unit 1)
@@
 	)
 	(symbol
-		(lib_id "C_Small:C_Small")
+		(lib_id "Device:C_Small")
 		(at 351.79 220.98 180)
 		(unit 1)
@@
 	)
 	(symbol
-		(lib_id "C_Small:C_Small")
+		(lib_id "Device:C_Small")
 		(at 62.23 64.77 270)
 		(unit 1)
@@
 	)
 	(symbol
-		(lib_id "R_Small_US:R_Small_US")
+		(lib_id "Device:R_Small_US")
 		(at 264.795 123.19 90)
 		(unit 1)
@@
 	)
 	(symbol
-		(lib_id "R_Small_US:R_Small_US")
+		(lib_id "Device:R_Small_US")
 		(at 264.795 130.81 90)
 		(unit 1)
@@
 	)
 	(symbol
-		(lib_id "C_Small:C_Small")
+		(lib_id "Device:C_Small")
 		(at 345.44 220.98 180)
 		(unit 1)
@@
 	)
 	(symbol
-		(lib_id "C_Small:C_Small")
+		(lib_id "Device:C_Small")
 		(at 62.23 57.15 270)
 		(unit 1)
@@
 	)
 	(symbol
-		(lib_id "C_Small:C_Small")
+		(lib_id "Device:C_Small")
 		(at 241.3 269.24 180)
 		(unit 1)
@@
 	)
 	(symbol
-		(lib_id "C_Small:C_Small")
+		(lib_id "Device:C_Small")
 		(at 323.85 220.98 180)
 		(unit 1)
@@
 	)
 	(symbol
-		(lib_id "C_Small:C_Small")
+		(lib_id "Device:C_Small")
 		(at 331.47 220.98 180)
 		(unit 1)
@@
 	)
 	(symbol
-		(lib_id "C_Small:C_Small")
+		(lib_id "Device:C_Small")
 		(at 73.025 59.69 270)
 		(unit 1)
