File: Tangenta/RS_485_422.kicad_sch (KiCad schematic)
At the start: 32 parts, among them J10 Conn_01x02_Pin, Q5 BSS138, Q6 BSS138, Q7 BSS138, Q8 BSS138, U16 ADM2582E, U17 TPCDSOT23-SM712, U18 TPCDSOT23-SM712

Commit message: Fixes, before checks.
Parts:
- C100, C101, C102, C103, C104, C99: symbol C_Small:C_Small -> Device:C_Small
- C98: symbol 16CE47FSS:16CE47FSS -> CAP_L5:16CE47FSS
- J10: symbol Conn_01x02_Pin:Conn_01x02_Pin -> Connector_Generic:Conn_01x02
- Q5, Q6, Q7, Q8: symbol BSS138:BSS138 -> Transistor_FET:BSS138
- R53, R54, R55, R56, R57, R58, R59, R60, R61, R62, R63, R64, R65, R66, R67, R68, R69: symbol R_Small_US:R_Small_US -> Device:R_Small_US
- U16: symbol ADM2582E:ADM2582E -> ADM2582EBRWZ:ADM2582E
- U17, U18: symbol TPCDSOT23-SM712:TPCDSOT23-SM712 -> ESD_RS485:TPCDSOT23-SM712
Changed lines of the file:
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@@
 	)
 	(symbol
-		(lib_id "R_Small_US:R_Small_US")
+		(lib_id "Device:R_Small_US")
 		(at 137.795 40.64 180)
 		(unit 1)
@@
 	)
 	(symbol
-		(lib_id "R_Small_US:R_Small_US")
+		(lib_id "Device:R_Small_US")
 		(at 206.375 75.565 270)
 		(unit 1)
@@
 	)
 	(symbol
-		(lib_id "R_Small_US:R_Small_US")
+		(lib_id "Device:R_Small_US")
 		(at 250.825 80.645 270)
 		(unit 1)
@@
 	)
 	(symbol
-		(lib_id "R_Small_US:R_Small_US")
+		(lib_id "Device:R_Small_US")
 		(at 137.795 82.55 180)
 		(unit 1)
@@
 	)
 	(symbol
-		(lib_id "R_Small_US:R_Small_US")
+		(lib_id "Device:R_Small_US")
 		(at 206.375 91.44 270)
 		(unit 1)
@@
 	)
 	(symbol
-		(lib_id "R_Small_US:R_Small_US")
+		(lib_id "Device:R_Small_US")
 		(at 213.36 79.375 0)
 		(unit 1)
@@
 	)
 	(symbol
-		(lib_id "C_Small:C_Small")
+		(lib_id "Device:C_Small")
 		(at 266.7 36.195 180)
 		(unit 1)
@@
 	)
 	(symbol
-		(lib_id "BSS138:BSS138")
+		(lib_id "Transistor_FET:BSS138")
 		(at 123.825 65.405 270)
 		(unit 1)
@@
 	)
 	(symbol
-		(lib_id "R_Small_US:R_Small_US")
+		(lib_id "Device:R_Small_US")
 		(at 206.375 99.06 270)
 		(unit 1)
@@
 	)
 	(symbol
-		(lib_id "R_Small_US:R_Small_US")
+		(lib_id "Device:R_Small_US")
 		(at 259.08 86.995 0)
 		(unit 1)
@@
 	)
 	(symbol
-		(lib_id "C_Small:C_Small")
+		(lib_id "Device:C_Small")
 		(at 266.7 57.785 180)
 		(unit 1)
@@
 	)
 	(symbol
-		(lib_id "R_Small_US:R_Small_US")
+		(lib_id "Device:R_Small_US")
 		(at 206.375 83.185 270)
 		(unit 1)
@@
 	)
 	(symbol
-		(lib_id "C_Small:C_Small")
+		(lib_id "Device:C_Small")
 		(at 259.08 36.195 180)
 		(unit 1)
@@
 	)
 	(symbol
-		(lib_id "R_Small_US:R_Small_US")
+		(lib_id "Device:R_Small_US")
 		(at 137.795 61.595 180)
 		(unit 1)
@@
 	)
 	(symbol
-		(lib_id "BSS138:BSS138")
+		(lib_id "Transistor_FET:BSS138")
 		(at 123.825 44.45 270)
 		(unit 1)
@@
 	)
 	(symbol
-		(lib_id "16CE47FSS:16CE47FSS")
+		(lib_id "CAP_L5:16CE47FSS")
 		(at 48.26 47.625 0)
 		(unit 1)
@@
 	)
 	(symbol
-		(lib_id "R_Small_US:R_Small_US")
+		(lib_id "Device:R_Small_US")
 		(at 111.125 82.55 180)
 		(unit 1)
@@
 	)
 	(symbol
-		(lib_id "R_Small_US:R_Small_US")
+		(lib_id "Device:R_Small_US")
 		(at 111.125 103.505 180)
 		(unit 1)
@@
 	)
 	(symbol
-		(lib_id "TPCDSOT23-SM712:TPCDSOT23-SM712")
+		(lib_id "ESD_RS485:TPCDSOT23-SM712")
 		(at 216.916 127.635 0)
 		(unit 1)
@@
 	)
 	(symbol
-		(lib_id "R_Small_US:R_Small_US")
+		(lib_id "Device:R_Small_US")
 		(at 111.125 40.64 180)
 		(unit 1)
@@
 	)
 	(symbol
-		(lib_id "C_Small:C_Small")
+		(lib_id "Device:C_Small")
 		(at 274.32 57.785 180)
 		(unit 1)
@@
 	)
 	(symbol
-		(lib_id "BSS138:BSS138")
+		(lib_id "Transistor_FET:BSS138")
 		(at 123.825 86.36 270)
 		(unit 1)
@@
 	)
 	(symbol
-		(lib_id "ADM2582E:ADM2582E")
+		(lib_id "ADM2582EBRWZ:ADM2582E")
 		(at 210.185 49.53 0)
 		(unit 1)
@@
 	)
 	(symbol
-		(lib_id "R_Small_US:R_Small_US")
+		(lib_id "Device:R_Small_US")
 		(at 137.795 103.505 180)
 		(unit 1)
@@
 	)
 	(symbol
-		(lib_id "BSS138:BSS138")
+		(lib_id "Transistor_FET:BSS138")
 		(at 123.825 107.315 270)
 		(unit 1)
@@
 	)
 	(symbol
-		(lib_id "C_Small:C_Small")
+		(lib_id "Device:C_Small")
 		(at 274.32 36.195 180)
 		(unit 1)
@@
 	)
 	(symbol
-		(lib_id "R_Small_US:R_Small_US")
+		(lib_id "Device:R_Small_US")
 		(at 111.125 61.595 180)
 		(unit 1)
@@
 	)
 	(symbol
-		(lib_id "R_Small_US:R_Small_US")
+		(lib_id "Device:R_Small_US")
 		(at 250.825 93.98 270)
 		(unit 1)
@@
 	)
 	(symbol
-		(lib_id "Conn_01x02_Pin:Conn_01x02_Pin")
+		(lib_id "Connector_Generic:Conn_01x02")
 		(at 198.12 154.94 270)
 		(unit 1)
@@
 	)
 	(symbol
-		(lib_id "R_Small_US:R_Small_US")
+		(lib_id "Device:R_Small_US")
 		(at 213.36 95.25 180)
 		(unit 1)
@@
 	(symbol
 		(lib_name "TPCDSOT23-SM712_1")
-		(lib_id "TPCDSOT23-SM712:TPCDSOT23-SM712")
+		(lib_id "ESD_RS485:TPCDSOT23-SM712")
 		(at 216.916 111.125 0)
 		(unit 1)
@@
 	)
 	(symbol
-		(lib_id "C_Small:C_Small")
+		(lib_id "Device:C_Small")
 		(at 259.08 57.785 180)
 		(unit 1)
