File: Tangenta/RS_485_422.kicad_sch (KiCad schematic)
At the start: 32 parts, among them J10 Conn_01x02_Pin, Q5 BSS138, Q6 BSS138, Q7 BSS138, Q8 BSS138, U16 ADM2582E, U17 TPCDSOT23-SM712, U18 TPCDSOT23-SM712

Commit message: Fixes, continued...
Parts:
- U16: value ADM2582E -> ADM2582EBRWZ-REEL7; footprint Package_SO:SOIC-20W_7.5x12.8mm_P1.27mm -> ADM2582EBRWZ:ADM2582EBRWZ; symbol ADM2582EBRWZ:ADM2582E -> ADM2582EBRWZ:ADM2582EBRWZ-REEL7
Connections:
- net 5V: no longer U16.2 (VCC), U16.8 (VCC)
- net A: no longer U16.18 (A)
- net B: no longer U16.17 (B)
- net CTS_1_H: no longer U16.6 (DE)
- net GNDREF: no longer U16.1 (GND1), U16.10 (GND1), U16.3 (GND1), U16.9 (GND1)
- net RS_ISO_5V: no longer U16.12 (Visoout), U16.19 (Visoin)
- net RS_ISO_GND: no longer U16.11 (GND2), U16.14 (GND2), U16.16 (GND2), U16.20 (GND2)
- net RTS_1_H: no longer U16.5 (~{RE})
- net RXD_1_H: no longer U16.4 (RxD)
- net TXD_1_H: no longer U16.7 (TxD)
- net Y: no longer U16.13 (Y)
- net Z: no longer U16.15 (Z)
Changed lines of the file:
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@@
 	)
 	(symbol
-		(lib_id "ADM2582EBRWZ:ADM2582E")
+		(lib_id "ADM2582EBRWZ:ADM2582EBRWZ-REEL7")
 		(at 210.185 49.53 0)
 		(unit 1)
@@
 			)
 		)
-		(property "Value" "ADM2582E"
+		(property "Value" "ADM2582EBRWZ-REEL7"
 			(at 210.185 66.675 0)
 			(effects
@@
 			)
 		)
-		(property "Footprint" "Package_SO:SOIC-20W_7.5x12.8mm_P1.27mm"
+		(property "Footprint" "ADM2582EBRWZ:ADM2582EBRWZ"
 			(at 210.185 67.31 0)
 			(effects

Commit message: Reverting to the original design.
Parts:
- C1: renamed from C101; symbol Device:C_Small -> CholaSymbolsPrjLib:C_Small
- C1: renamed from C102; symbol Device:C_Small -> CholaSymbolsPrjLib:C_Small
- C1: renamed from C99; symbol Device:C_Small -> CholaSymbolsPrjLib:C_Small
- C1: renamed from C104; symbol Device:C_Small -> CholaSymbolsPrjLib:C_Small
- C1: renamed from C103; symbol Device:C_Small -> CholaSymbolsPrjLib:C_Small
- C1: renamed from C100; symbol Device:C_Small -> CholaSymbolsPrjLib:C_Small
- C178: renamed from C98; symbol CAP_L5:16CE47FSS -> CholaSymbolsPrjLib:16CE47FSS
- J10: symbol Connector_Generic:Conn_01x02 -> CholaSymbolsPrjLib:Conn_01x02_Pin
- Q3: renamed from Q6; symbol Transistor_FET:BSS138 -> CholaSymbolsPrjLib:BSS138
- Q3: renamed from Q5; symbol Transistor_FET:BSS138 -> CholaSymbolsPrjLib:BSS138
- Q3: renamed from Q7; symbol Transistor_FET:BSS138 -> CholaSymbolsPrjLib:BSS138
- Q3: renamed from Q8; symbol Transistor_FET:BSS138 -> CholaSymbolsPrjLib:BSS138
- R2: renamed from R57; symbol Device:R_Small_US -> CholaSymbolsPrjLib:R_Small_US
- R2: renamed from R61; symbol Device:R_Small_US -> CholaSymbolsPrjLib:R_Small_US
- R2: renamed from R59; symbol Device:R_Small_US -> CholaSymbolsPrjLib:R_Small_US
- R2: renamed from R63; symbol Device:R_Small_US -> CholaSymbolsPrjLib:R_Small_US
- R2: renamed from R64; symbol Device:R_Small_US -> CholaSymbolsPrjLib:R_Small_US
- R2: renamed from R62; symbol Device:R_Small_US -> CholaSymbolsPrjLib:R_Small_US
- R2: renamed from R58; symbol Device:R_Small_US -> CholaSymbolsPrjLib:R_Small_US
- R2: renamed from R55; symbol Device:R_Small_US -> CholaSymbolsPrjLib:R_Small_US
- R2: renamed from R56; symbol Device:R_Small_US -> CholaSymbolsPrjLib:R_Small_US
- R2: renamed from R53; symbol Device:R_Small_US -> CholaSymbolsPrjLib:R_Small_US
- R2: renamed from R60; symbol Device:R_Small_US -> CholaSymbolsPrjLib:R_Small_US
- R2: renamed from R54; symbol Device:R_Small_US -> CholaSymbolsPrjLib:R_Small_US
- R4: renamed from R67; symbol Device:R_Small_US -> CholaSymbolsPrjLib:R_Small_US
- R4: renamed from R65; symbol Device:R_Small_US -> CholaSymbolsPrjLib:R_Small_US
- R4: renamed from R69; symbol Device:R_Small_US -> CholaSymbolsPrjLib:R_Small_US
- R4: renamed from R68; symbol Device:R_Small_US -> CholaSymbolsPrjLib:R_Small_US
- R4: renamed from R66; symbol Device:R_Small_US -> CholaSymbolsPrjLib:R_Small_US
- U16: value ADM2582EBRWZ-REEL7 -> ADM2582E; footprint ADM2582EBRWZ:ADM2582EBRWZ -> Package_SO:SOIC-20W_7.5x12.8mm_P1.27mm; symbol ADM2582EBRWZ:ADM2582EBRWZ-REEL7 -> CholaSymbolsPrjLib:ADM2582E
- U17, U18: symbol ESD_RS485:TPCDSOT23-SM712 -> CholaSymbolsPrjLib:TPCDSOT23-SM712
Connections:
- net 5V: now also U16.2 (VCC), U16.8 (VCC)
- net A: now also U16.18 (A)
- net B: now also U16.17 (B)
- net CTS_1_H: now also U16.6 (DE)
- net GNDREF: now also U16.1 (GND1), U16.10 (GND1), U16.3 (GND1), U16.9 (GND1)
- net RS_ISO_5V: now also U16.12 (Visoout), U16.19 (Visoin)
- net RS_ISO_GND: now also U16.11 (GND2), U16.14 (GND2), U16.16 (GND2), U16.20 (GND2)
- net RTS_1_H: now also U16.5 (~{RE})
- net RXD_1_H: now also U16.4 (RxD)
- net TXD_1_H: now also U16.7 (TxD)
- net Y: now also U16.13 (Y)
- net Z: now also U16.15 (Z)

Commit message: ...
Parts:
- C1: symbol CholaSymbolsPrjLib:C_Small -> LocalPrjLib:C_Small
- C178: symbol CholaSymbolsPrjLib:16CE47FSS -> LocalPrjLib:16CE47FSS
- J10: symbol CholaSymbolsPrjLib:Conn_01x02_Pin -> LocalPrjLib:Conn_01x02_Pin
- Q3: symbol CholaSymbolsPrjLib:BSS138 -> LocalPrjLib:BSS138
- R2, R4: symbol CholaSymbolsPrjLib:R_Small_US -> LocalPrjLib:R_Small_US
- U16: symbol CholaSymbolsPrjLib:ADM2582E -> LocalPrjLib:ADM2582E
- U17, U18: symbol CholaSymbolsPrjLib:TPCDSOT23-SM712 -> LocalPrjLib:TPCDSOT23-SM712
Changed lines of the file:
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@@
     )
   )
-  (symbol (lib_id "CholaSymbolsPrjLib:R_Small_US") (at 137.795 40.64 180) (unit 1)
+  (symbol (lib_id "LocalPrjLib:R_Small_US") (at 137.795 40.64 180) (unit 1)
     (in_bom yes) (on_board yes) (dnp no)
     (property "Reference" "R2" (at 136.525 39.37 0)
@@
     )
   )
-  (symbol (lib_id "CholaSymbolsPrjLib:R_Small_US") (at 206.375 75.565 270) (unit 1)
+  (symbol (lib_id "LocalPrjLib:R_Small_US") (at 206.375 75.565 270) (unit 1)
     (in_bom yes) (on_board yes) (dnp no)
     (property "Reference" "R2" (at 199.39 74.295 90)
@@
     )
   )
-  (symbol (lib_id "CholaSymbolsPrjLib:R_Small_US") (at 250.825 80.645 270) (unit 1)
+  (symbol (lib_id "LocalPrjLib:R_Small_US") (at 250.825 80.645 270) (unit 1)
     (in_bom no) (on_board yes) (dnp yes)
     (property "Reference" "R4" (at 246.38 79.375 90)
@@
     )
   )
-  (symbol (lib_id "CholaSymbolsPrjLib:R_Small_US") (at 137.795 82.55 180) (unit 1)
+  (symbol (lib_id "LocalPrjLib:R_Small_US") (at 137.795 82.55 180) (unit 1)
     (in_bom yes) (on_board yes) (dnp no)
     (property "Reference" "R2" (at 136.525 81.28 0)
@@
     )
   )
-  (symbol (lib_id "CholaSymbolsPrjLib:R_Small_US") (at 206.375 91.44 270) (unit 1)
+  (symbol (lib_id "LocalPrjLib:R_Small_US") (at 206.375 91.44 270) (unit 1)
     (in_bom yes) (on_board yes) (dnp no)
     (property "Reference" "R2" (at 199.39 90.17 90)
@@
     )
   )
-  (symbol (lib_id "CholaSymbolsPrjLib:R_Small_US") (at 213.36 79.375 0) (unit 1)
+  (symbol (lib_id "LocalPrjLib:R_Small_US") (at 213.36 79.375 0) (unit 1)
     (in_bom yes) (on_board yes) (dnp no)
     (property "Reference" "R4" (at 217.17 78.105 0)
@@
     )
   )
-  (symbol (lib_id "CholaSymbolsPrjLib:C_Small") (at 266.7 36.195 180) (unit 1)
+  (symbol (lib_id "LocalPrjLib:C_Small") (at 266.7 36.195 180) (unit 1)
     (in_bom yes) (on_board yes) (dnp no)
     (property "Reference" "C1" (at 264.1599 34.2899 0)
@@
     )
   )
-  (symbol (lib_id "CholaSymbolsPrjLib:BSS138") (at 123.825 65.405 270) (unit 1)
+  (symbol (lib_id "LocalPrjLib:BSS138") (at 123.825 65.405 270) (unit 1)
     (in_bom yes) (on_board yes) (dnp no)
     (property "Reference" "Q3" (at 126.365 62.865 90)
@@
     )
   )
-  (symbol (lib_id "CholaSymbolsPrjLib:R_Small_US") (at 206.375 99.06 270) (unit 1)
+  (symbol (lib_id "LocalPrjLib:R_Small_US") (at 206.375 99.06 270) (unit 1)
     (in_bom yes) (on_board yes) (dnp no)
     (property "Reference" "R2" (at 199.39 97.79 90)
@@
     )
   )
-  (symbol (lib_id "CholaSymbolsPrjLib:R_Small_US") (at 259.08 86.995 0) (unit 1)
+  (symbol (lib_id "LocalPrjLib:R_Small_US") (at 259.08 86.995 0) (unit 1)
     (in_bom no) (on_board yes) (dnp yes)
     (property "Reference" "R4" (at 262.89 86.36 0)
@@
     )
   )
-  (symbol (lib_id "CholaSymbolsPrjLib:C_Small") (at 266.7 57.785 180) (unit 1)
+  (symbol (lib_id "LocalPrjLib:C_Small") (at 266.7 57.785 180) (unit 1)
     (in_bom yes) (on_board yes) (dnp no)
     (property "Reference" "C1" (at 264.1599 55.8799 0)
@@
     )
   )
-  (symbol (lib_id "CholaSymbolsPrjLib:R_Small_US") (at 206.375 83.185 270) (unit 1)
+  (symbol (lib_id "LocalPrjLib:R_Small_US") (at 206.375 83.185 270) (unit 1)
     (in_bom yes) (on_board yes) (dnp no)
     (property "Reference" "R2" (at 199.39 81.915 90)
@@
     )
   )
-  (symbol (lib_id "CholaSymbolsPrjLib:C_Small") (at 259.08 36.195 180) (unit 1)
+  (symbol (lib_id "LocalPrjLib:C_Small") (at 259.08 36.195 180) (unit 1)
     (in_bom yes) (on_board yes) (dnp no)
     (property "Reference" "C1" (at 256.5399 34.2899 0)
@@
     )
   )
-  (symbol (lib_id "CholaSymbolsPrjLib:R_Small_US") (at 137.795 61.595 180) (unit 1)
+  (symbol (lib_id "LocalPrjLib:R_Small_US") (at 137.795 61.595 180) (unit 1)
     (in_bom yes) (on_board yes) (dnp no)
     (property "Reference" "R2" (at 136.525 60.325 0)
@@
     )
   )
-  (symbol (lib_id "CholaSymbolsPrjLib:BSS138") (at 123.825 44.45 270) (unit 1)
+  (symbol (lib_id "LocalPrjLib:BSS138") (at 123.825 44.45 270) (unit 1)
     (in_bom yes) (on_board yes) (dnp no)
     (property "Reference" "Q3" (at 126.365 41.91 90)
@@
     )
   )
-  (symbol (lib_id "CholaSymbolsPrjLib:16CE47FSS") (at 48.26 47.625 0) (unit 1)
+  (symbol (lib_id "LocalPrjLib:16CE47FSS") (at 48.26 47.625 0) (unit 1)
     (in_bom yes) (on_board yes) (dnp no)
     (property "Reference" "C178" (at 49.53 45.72 0)
@@
     )
   )
-  (symbol (lib_id "CholaSymbolsPrjLib:R_Small_US") (at 111.125 82.55 180) (unit 1)
+  (symbol (lib_id "LocalPrjLib:R_Small_US") (at 111.125 82.55 180) (unit 1)
     (in_bom yes) (on_board yes) (dnp no)
     (property "Reference" "R2" (at 109.855 81.28 0)
@@
     )
   )
-  (symbol (lib_id "CholaSymbolsPrjLib:R_Small_US") (at 111.125 103.505 180) (unit 1)
+  (symbol (lib_id "LocalPrjLib:R_Small_US") (at 111.125 103.505 180) (unit 1)
     (in_bom yes) (on_board yes) (dnp no)
     (property "Reference" "R2" (at 109.855 102.235 0)
@@
     )
   )
-  (symbol (lib_id "CholaSymbolsPrjLib:TPCDSOT23-SM712") (at 216.916 127.635 0) (unit 1)
+  (symbol (lib_id "LocalPrjLib:TPCDSOT23-SM712") (at 216.916 127.635 0) (unit 1)
     (in_bom yes) (on_board yes) (dnp no)
     (property "Reference" "U18" (at 210.566 121.285 0)
@@
     )
   )
-  (symbol (lib_id "CholaSymbolsPrjLib:R_Small_US") (at 111.125 40.64 180) (unit 1)
+  (symbol (lib_id "LocalPrjLib:R_Small_US") (at 111.125 40.64 180) (unit 1)
     (in_bom yes) (on_board yes) (dnp no)
     (property "Reference" "R2" (at 109.855 39.37 0)
@@
     )
   )
-  (symbol (lib_id "CholaSymbolsPrjLib:C_Small") (at 274.32 57.785 180) (unit 1)
+  (symbol (lib_id "LocalPrjLib:C_Small") (at 274.32 57.785 180) (unit 1)
     (in_bom yes) (on_board yes) (dnp no)
     (property "Reference" "C1" (at 271.7799 55.8799 0)
@@
     )
   )
-  (symbol (lib_id "CholaSymbolsPrjLib:BSS138") (at 123.825 86.36 270) (unit 1)
+  (symbol (lib_id "LocalPrjLib:BSS138") (at 123.825 86.36 270) (unit 1)
     (in_bom yes) (on_board yes) (dnp no)
     (property "Reference" "Q3" (at 126.365 83.82 90)
@@
     )
   )
-  (symbol (lib_id "CholaSymbolsPrjLib:ADM2582E") (at 210.185 49.53 0) (unit 1)
+  (symbol (lib_id "LocalPrjLib:ADM2582E") (at 210.185 49.53 0) (unit 1)
     (in_bom yes) (on_board yes) (dnp no)
     (property "Reference" "U16" (at 210.185 30.48 0)
@@
     )
   )
-  (symbol (lib_id "CholaSymbolsPrjLib:R_Small_US") (at 137.795 103.505 180) (unit 1)
+  (symbol (lib_id "LocalPrjLib:R_Small_US") (at 137.795 103.505 180) (unit 1)
     (in_bom yes) (on_board yes) (dnp no)
     (property "Reference" "R2" (at 136.525 102.235 0)
@@
     )
   )
-  (symbol (lib_id "CholaSymbolsPrjLib:BSS138") (at 123.825 107.315 270) (unit 1)
+  (symbol (lib_id "LocalPrjLib:BSS138") (at 123.825 107.315 270) (unit 1)
     (in_bom yes) (on_board yes) (dnp no)
     (property "Reference" "Q3" (at 126.365 104.775 90)
@@
     )
   )
-  (symbol (lib_id "CholaSymbolsPrjLib:C_Small") (at 274.32 36.195 180) (unit 1)
+  (symbol (lib_id "LocalPrjLib:C_Small") (at 274.32 36.195 180) (unit 1)
     (in_bom yes) (on_board yes) (dnp no)
     (property "Reference" "C1" (at 271.7799 34.2899 0)
@@
     )
   )
-  (symbol (lib_id "CholaSymbolsPrjLib:R_Small_US") (at 111.125 61.595 180) (unit 1)
+  (symbol (lib_id "LocalPrjLib:R_Small_US") (at 111.125 61.595 180) (unit 1)
     (in_bom yes) (on_board yes) (dnp no)
     (property "Reference" "R2" (at 109.855 60.325 0)
@@
     )
   )
-  (symbol (lib_id "CholaSymbolsPrjLib:R_Small_US") (at 250.825 93.98 270) (unit 1)
+  (symbol (lib_id "LocalPrjLib:R_Small_US") (at 250.825 93.98 270) (unit 1)
     (in_bom no) (on_board yes) (dnp yes)
     (property "Reference" "R4" (at 246.38 92.71 90)
@@
     )
   )
-  (symbol (lib_id "CholaSymbolsPrjLib:Conn_01x02_Pin") (at 198.12 154.94 270) (unit 1)
+  (symbol (lib_id "LocalPrjLib:Conn_01x02_Pin") (at 198.12 154.94 270) (unit 1)
     (in_bom yes) (on_board yes) (dnp no)
     (property "Reference" "J10" (at 194.945 153.67 90)
@@
     )
   )
-  (symbol (lib_id "CholaSymbolsPrjLib:R_Small_US") (at 213.36 95.25 180) (unit 1)
+  (symbol (lib_id "LocalPrjLib:R_Small_US") (at 213.36 95.25 180) (unit 1)
     (in_bom yes) (on_board yes) (dnp no)
     (property "Reference" "R4" (at 217.17 93.98 0)
@@
     )
   )
-  (symbol (lib_id "CholaSymbolsPrjLib:TPCDSOT23-SM712") (at 216.916 111.125 0) (unit 1)
+  (symbol (lib_id "LocalPrjLib:TPCDSOT23-SM712") (at 216.916 111.125 0) (unit 1)
     (in_bom yes) (on_board yes) (dnp no)
     (property "Reference" "U17" (at 210.566 104.775 0)
@@
     )
   )
-  (symbol (lib_id "CholaSymbolsPrjLib:C_Small") (at 259.08 57.785 180) (unit 1)
+  (symbol (lib_id "LocalPrjLib:C_Small") (at 259.08 57.785 180) (unit 1)
     (in_bom yes) (on_board yes) (dnp no)
     (property "Reference" "C1" (at 256.5399 55.8799 0)

Commit message: Fixes, new approach.
Parts:
- C1: symbol LocalPrjLib:C_Small -> LocalSymbolsPrjLib:C_Small
- C178: symbol LocalPrjLib:16CE47FSS -> LocalSymbolsPrjLib:16CE47FSS
- J10: symbol LocalPrjLib:Conn_01x02_Pin -> LocalSymbolsPrjLib:Conn_01x02_Pin
- Q3: symbol LocalPrjLib:BSS138 -> LocalSymbolsPrjLib:BSS138
- R2, R4: symbol LocalPrjLib:R_Small_US -> LocalSymbolsPrjLib:R_Small_US
- U16: symbol LocalPrjLib:ADM2582E -> LocalSymbolsPrjLib:ADM2582E
- U17, U18: symbol LocalPrjLib:TPCDSOT23-SM712 -> LocalSymbolsPrjLib:TPCDSOT23-SM712
Changed lines of the file:
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@@
     )
   )
-  (symbol (lib_id "LocalPrjLib:R_Small_US") (at 137.795 40.64 180) (unit 1)
+  (symbol (lib_id "LocalSymbolsPrjLib:R_Small_US") (at 137.795 40.64 180) (unit 1)
     (in_bom yes) (on_board yes) (dnp no)
     (property "Reference" "R2" (at 136.525 39.37 0)
@@
     )
   )
-  (symbol (lib_id "LocalPrjLib:R_Small_US") (at 206.375 75.565 270) (unit 1)
+  (symbol (lib_id "LocalSymbolsPrjLib:R_Small_US") (at 206.375 75.565 270) (unit 1)
     (in_bom yes) (on_board yes) (dnp no)
     (property "Reference" "R2" (at 199.39 74.295 90)
@@
     )
   )
-  (symbol (lib_id "LocalPrjLib:R_Small_US") (at 250.825 80.645 270) (unit 1)
+  (symbol (lib_id "LocalSymbolsPrjLib:R_Small_US") (at 250.825 80.645 270) (unit 1)
     (in_bom no) (on_board yes) (dnp yes)
     (property "Reference" "R4" (at 246.38 79.375 90)
@@
     )
   )
-  (symbol (lib_id "LocalPrjLib:R_Small_US") (at 137.795 82.55 180) (unit 1)
+  (symbol (lib_id "LocalSymbolsPrjLib:R_Small_US") (at 137.795 82.55 180) (unit 1)
     (in_bom yes) (on_board yes) (dnp no)
     (property "Reference" "R2" (at 136.525 81.28 0)
@@
     )
   )
-  (symbol (lib_id "LocalPrjLib:R_Small_US") (at 206.375 91.44 270) (unit 1)
+  (symbol (lib_id "LocalSymbolsPrjLib:R_Small_US") (at 206.375 91.44 270) (unit 1)
     (in_bom yes) (on_board yes) (dnp no)
     (property "Reference" "R2" (at 199.39 90.17 90)
@@
     )
   )
-  (symbol (lib_id "LocalPrjLib:R_Small_US") (at 213.36 79.375 0) (unit 1)
+  (symbol (lib_id "LocalSymbolsPrjLib:R_Small_US") (at 213.36 79.375 0) (unit 1)
     (in_bom yes) (on_board yes) (dnp no)
     (property "Reference" "R4" (at 217.17 78.105 0)
@@
     )
   )
-  (symbol (lib_id "LocalPrjLib:C_Small") (at 266.7 36.195 180) (unit 1)
+  (symbol (lib_id "LocalSymbolsPrjLib:C_Small") (at 266.7 36.195 180) (unit 1)
     (in_bom yes) (on_board yes) (dnp no)
     (property "Reference" "C1" (at 264.1599 34.2899 0)
@@
     )
   )
-  (symbol (lib_id "LocalPrjLib:BSS138") (at 123.825 65.405 270) (unit 1)
+  (symbol (lib_id "LocalSymbolsPrjLib:BSS138") (at 123.825 65.405 270) (unit 1)
     (in_bom yes) (on_board yes) (dnp no)
     (property "Reference" "Q3" (at 126.365 62.865 90)
@@
     )
   )
-  (symbol (lib_id "LocalPrjLib:R_Small_US") (at 206.375 99.06 270) (unit 1)
+  (symbol (lib_id "LocalSymbolsPrjLib:R_Small_US") (at 206.375 99.06 270) (unit 1)
     (in_bom yes) (on_board yes) (dnp no)
     (property "Reference" "R2" (at 199.39 97.79 90)
@@
     )
   )
-  (symbol (lib_id "LocalPrjLib:R_Small_US") (at 259.08 86.995 0) (unit 1)
+  (symbol (lib_id "LocalSymbolsPrjLib:R_Small_US") (at 259.08 86.995 0) (unit 1)
     (in_bom no) (on_board yes) (dnp yes)
     (property "Reference" "R4" (at 262.89 86.36 0)
@@
     )
   )
-  (symbol (lib_id "LocalPrjLib:C_Small") (at 266.7 57.785 180) (unit 1)
+  (symbol (lib_id "LocalSymbolsPrjLib:C_Small") (at 266.7 57.785 180) (unit 1)
     (in_bom yes) (on_board yes) (dnp no)
     (property "Reference" "C1" (at 264.1599 55.8799 0)
@@
     )
   )
-  (symbol (lib_id "LocalPrjLib:R_Small_US") (at 206.375 83.185 270) (unit 1)
+  (symbol (lib_id "LocalSymbolsPrjLib:R_Small_US") (at 206.375 83.185 270) (unit 1)
     (in_bom yes) (on_board yes) (dnp no)
     (property "Reference" "R2" (at 199.39 81.915 90)
@@
     )
   )
-  (symbol (lib_id "LocalPrjLib:C_Small") (at 259.08 36.195 180) (unit 1)
+  (symbol (lib_id "LocalSymbolsPrjLib:C_Small") (at 259.08 36.195 180) (unit 1)
     (in_bom yes) (on_board yes) (dnp no)
     (property "Reference" "C1" (at 256.5399 34.2899 0)
@@
     )
   )
-  (symbol (lib_id "LocalPrjLib:R_Small_US") (at 137.795 61.595 180) (unit 1)
+  (symbol (lib_id "LocalSymbolsPrjLib:R_Small_US") (at 137.795 61.595 180) (unit 1)
     (in_bom yes) (on_board yes) (dnp no)
     (property "Reference" "R2" (at 136.525 60.325 0)
@@
     )
   )
-  (symbol (lib_id "LocalPrjLib:BSS138") (at 123.825 44.45 270) (unit 1)
+  (symbol (lib_id "LocalSymbolsPrjLib:BSS138") (at 123.825 44.45 270) (unit 1)
     (in_bom yes) (on_board yes) (dnp no)
     (property "Reference" "Q3" (at 126.365 41.91 90)
@@
     )
   )
-  (symbol (lib_id "LocalPrjLib:16CE47FSS") (at 48.26 47.625 0) (unit 1)
+  (symbol (lib_id "LocalSymbolsPrjLib:16CE47FSS") (at 48.26 47.625 0) (unit 1)
     (in_bom yes) (on_board yes) (dnp no)
     (property "Reference" "C178" (at 49.53 45.72 0)
@@
     )
   )
-  (symbol (lib_id "LocalPrjLib:R_Small_US") (at 111.125 82.55 180) (unit 1)
+  (symbol (lib_id "LocalSymbolsPrjLib:R_Small_US") (at 111.125 82.55 180) (unit 1)
     (in_bom yes) (on_board yes) (dnp no)
     (property "Reference" "R2" (at 109.855 81.28 0)
@@
     )
   )
-  (symbol (lib_id "LocalPrjLib:R_Small_US") (at 111.125 103.505 180) (unit 1)
+  (symbol (lib_id "LocalSymbolsPrjLib:R_Small_US") (at 111.125 103.505 180) (unit 1)
     (in_bom yes) (on_board yes) (dnp no)
     (property "Reference" "R2" (at 109.855 102.235 0)
@@
     )
   )
-  (symbol (lib_id "LocalPrjLib:TPCDSOT23-SM712") (at 216.916 127.635 0) (unit 1)
+  (symbol (lib_id "LocalSymbolsPrjLib:TPCDSOT23-SM712") (at 216.916 127.635 0) (unit 1)
     (in_bom yes) (on_board yes) (dnp no)
     (property "Reference" "U18" (at 210.566 121.285 0)
@@
     )
   )
-  (symbol (lib_id "LocalPrjLib:R_Small_US") (at 111.125 40.64 180) (unit 1)
+  (symbol (lib_id "LocalSymbolsPrjLib:R_Small_US") (at 111.125 40.64 180) (unit 1)
     (in_bom yes) (on_board yes) (dnp no)
     (property "Reference" "R2" (at 109.855 39.37 0)
@@
     )
   )
-  (symbol (lib_id "LocalPrjLib:C_Small") (at 274.32 57.785 180) (unit 1)
+  (symbol (lib_id "LocalSymbolsPrjLib:C_Small") (at 274.32 57.785 180) (unit 1)
     (in_bom yes) (on_board yes) (dnp no)
     (property "Reference" "C1" (at 271.7799 55.8799 0)
@@
     )
   )
-  (symbol (lib_id "LocalPrjLib:BSS138") (at 123.825 86.36 270) (unit 1)
+  (symbol (lib_id "LocalSymbolsPrjLib:BSS138") (at 123.825 86.36 270) (unit 1)
     (in_bom yes) (on_board yes) (dnp no)
     (property "Reference" "Q3" (at 126.365 83.82 90)
@@
     )
   )
-  (symbol (lib_id "LocalPrjLib:ADM2582E") (at 210.185 49.53 0) (unit 1)
+  (symbol (lib_id "LocalSymbolsPrjLib:ADM2582E") (at 210.185 49.53 0) (unit 1)
     (in_bom yes) (on_board yes) (dnp no)
     (property "Reference" "U16" (at 210.185 30.48 0)
@@
     )
   )
-  (symbol (lib_id "LocalPrjLib:R_Small_US") (at 137.795 103.505 180) (unit 1)
+  (symbol (lib_id "LocalSymbolsPrjLib:R_Small_US") (at 137.795 103.505 180) (unit 1)
     (in_bom yes) (on_board yes) (dnp no)
     (property "Reference" "R2" (at 136.525 102.235 0)
@@
     )
   )
-  (symbol (lib_id "LocalPrjLib:BSS138") (at 123.825 107.315 270) (unit 1)
+  (symbol (lib_id "LocalSymbolsPrjLib:BSS138") (at 123.825 107.315 270) (unit 1)
     (in_bom yes) (on_board yes) (dnp no)
     (property "Reference" "Q3" (at 126.365 104.775 90)
@@
     )
   )
-  (symbol (lib_id "LocalPrjLib:C_Small") (at 274.32 36.195 180) (unit 1)
+  (symbol (lib_id "LocalSymbolsPrjLib:C_Small") (at 274.32 36.195 180) (unit 1)
     (in_bom yes) (on_board yes) (dnp no)
     (property "Reference" "C1" (at 271.7799 34.2899 0)
@@
     )
   )
-  (symbol (lib_id "LocalPrjLib:R_Small_US") (at 111.125 61.595 180) (unit 1)
+  (symbol (lib_id "LocalSymbolsPrjLib:R_Small_US") (at 111.125 61.595 180) (unit 1)
     (in_bom yes) (on_board yes) (dnp no)
     (property "Reference" "R2" (at 109.855 60.325 0)
@@
     )
   )
-  (symbol (lib_id "LocalPrjLib:R_Small_US") (at 250.825 93.98 270) (unit 1)
+  (symbol (lib_id "LocalSymbolsPrjLib:R_Small_US") (at 250.825 93.98 270) (unit 1)
     (in_bom no) (on_board yes) (dnp yes)
     (property "Reference" "R4" (at 246.38 92.71 90)
@@
     )
   )
-  (symbol (lib_id "LocalPrjLib:Conn_01x02_Pin") (at 198.12 154.94 270) (unit 1)
+  (symbol (lib_id "LocalSymbolsPrjLib:Conn_01x02_Pin") (at 198.12 154.94 270) (unit 1)
     (in_bom yes) (on_board yes) (dnp no)
     (property "Reference" "J10" (at 194.945 153.67 90)
@@
     )
   )
-  (symbol (lib_id "LocalPrjLib:R_Small_US") (at 213.36 95.25 180) (unit 1)
+  (symbol (lib_id "LocalSymbolsPrjLib:R_Small_US") (at 213.36 95.25 180) (unit 1)
     (in_bom yes) (on_board yes) (dnp no)
     (property "Reference" "R4" (at 217.17 93.98 0)
@@
     )
   )
-  (symbol (lib_id "LocalPrjLib:TPCDSOT23-SM712") (at 216.916 111.125 0) (unit 1)
+  (symbol (lib_id "LocalSymbolsPrjLib:TPCDSOT23-SM712") (at 216.916 111.125 0) (unit 1)
     (in_bom yes) (on_board yes) (dnp no)
     (property "Reference" "U17" (at 210.566 104.775 0)
@@
     )
   )
-  (symbol (lib_id "LocalPrjLib:C_Small") (at 259.08 57.785 180) (unit 1)
+  (symbol (lib_id "LocalSymbolsPrjLib:C_Small") (at 259.08 57.785 180) (unit 1)
     (in_bom yes) (on_board yes) (dnp no)
     (property "Reference" "C1" (at 256.5399 55.8799 0)

Commit message: Fixes...
Parts:
- renumbered C1 to C100, C1 to C101, C1 to C102, C1 to C103, C1 to C104, C178 to C98, C1 to C99, Q3 to Q5, Q3 to Q6, Q3 to Q7, Q3 to Q8, R2 to R53, R2 to R54, R2 to R55, R2 to R56, R2 to R57, R2 to R58, R2 to R59, R2 to R60, R2 to R61, R2 to R62, R2 to R63, R2 to R64, R4 to R65, R4 to R66, R4 to R67, R4 to R68, R4 to R69
