File: Tangenta/JTAG.kicad_sch (KiCad schematic)
At the start: 1 part, among them J34 Conn_02x05_Odd_Even

Commit message: Removing component association with previous project (local) libraries.
Parts:
- J34: symbol CholaSymbolsPrjLib:Conn_02x05_Odd_Even -> Conn_02x05_Odd_Even:Conn_02x05_Odd_Even
Changed lines of the file:
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@@
 	)
 	(symbol
-		(lib_id "CholaSymbolsPrjLib:Conn_02x05_Odd_Even")
+		(lib_id "Conn_02x05_Odd_Even:Conn_02x05_Odd_Even")
 		(at 167.005 81.28 0)
 		(mirror y)

Commit message: Fixes, continued...
Parts:
- J34: symbol Conn_02x05_Odd_Even:Conn_02x05_Odd_Even -> Connector_Generic:Conn_02x05_Odd_Even
Connections:
- net GNDREF: no longer J34.3 (Pin_3), J34.5 (Pin_5)
- net JTAG.TCK: no longer J34.4 (Pin_4)
- net JTAG.TDI: no longer J34.8 (Pin_8)
- net JTAG.TDO: no longer J34.6 (Pin_6)
- net JTAG.TMS: no longer J34.2 (Pin_2)
- net JTAG.VREF: no longer J34.1 (Pin_1)
- net JTAG.nTRST: no longer J34.10 (Pin_10)
Changed lines of the file:
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@@
 	)
 	(symbol
-		(lib_id "Conn_02x05_Odd_Even:Conn_02x05_Odd_Even")
+		(lib_id "Connector_Generic:Conn_02x05_Odd_Even")
 		(at 167.005 81.28 0)
 		(mirror y)

Commit message: Fixes, continued...
Parts:
- J34: symbol Connector_Generic:Conn_02x05_Odd_Even -> Conn_02x05_Odd_Even:Conn_02x05_Odd_Even
Connections:
- net GNDREF: now also J34.3 (Pin_3), J34.5 (Pin_5)
- net JTAG.TCK: now also J34.4 (Pin_4)
- net JTAG.TDI: now also J34.8 (Pin_8)
- net JTAG.TDO: now also J34.6 (Pin_6)
- net JTAG.TMS: now also J34.2 (Pin_2)
- net JTAG.VREF: now also J34.1 (Pin_1)
- net JTAG.nTRST: now also J34.10 (Pin_10)
Changed lines of the file:
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@@
 	)
 	(symbol
-		(lib_id "Connector_Generic:Conn_02x05_Odd_Even")
+		(lib_id "Conn_02x05_Odd_Even:Conn_02x05_Odd_Even")
 		(at 167.005 81.28 0)
 		(mirror y)

Commit message: Fixes, before checks.
Parts:
- J34: symbol Conn_02x05_Odd_Even:Conn_02x05_Odd_Even -> Connector_Generic:Conn_02x05_Odd_Even
Changed lines of the file:
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@@
 	)
 	(symbol
-		(lib_id "Conn_02x05_Odd_Even:Conn_02x05_Odd_Even")
+		(lib_id "Connector_Generic:Conn_02x05_Odd_Even")
 		(at 167.005 81.28 0)
 		(mirror y)

Commit message: Reverting to the original design.
Parts:
- J34: symbol Connector_Generic:Conn_02x05_Odd_Even -> CholaSymbolsPrjLib:Conn_02x05_Odd_Even
