File: Tangenta/Ethernet_SFP_Port_4.kicad_sch (KiCad schematic)
At the start: 17 parts, among them J9 HC-SFP-01L

Commit message: Fixes, new approach.
Parts:
- C1: symbol LocalPrjLib:C_Small -> LocalSymbolsPrjLib:C_Small
- J9: symbol LocalPrjLib:HC-SFP-01L -> LocalSymbolsPrjLib:HC-SFP-01L
- R4: symbol LocalPrjLib:R_Small_US -> LocalSymbolsPrjLib:R_Small_US
- S1: symbol LocalPrjLib:HC-SFP-20P -> LocalSymbolsPrjLib:HC-SFP-20P
Changed lines of the file:
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@@
     (effects (font (size 1.27 1.27)) (justify right))
   )
-  (symbol (lib_id "LocalPrjLib:C_Small") (at 66.04 64.77 270) (unit 1)
+  (symbol (lib_id "LocalSymbolsPrjLib:C_Small") (at 66.04 64.77 270) (unit 1)
     (in_bom yes) (on_board yes) (dnp no)
     (property "Reference" "C1" (at 62.23 63.5 90)
@@
     )
   )
-  (symbol (lib_id "LocalPrjLib:R_Small_US") (at 224.79 128.905 180) (unit 1)
+  (symbol (lib_id "LocalSymbolsPrjLib:R_Small_US") (at 224.79 128.905 180) (unit 1)
     (in_bom yes) (on_board yes) (dnp no)
     (property "Reference" "R4" (at 220.98 128.27 0)
@@
     )
   )
-  (symbol (lib_id "LocalPrjLib:R_Small_US") (at 139.7 118.11 90) (unit 1)
+  (symbol (lib_id "LocalSymbolsPrjLib:R_Small_US") (at 139.7 118.11 90) (unit 1)
     (in_bom yes) (on_board yes) (dnp no)
     (property "Reference" "R4" (at 135.255 116.84 90)
@@
     )
   )
-  (symbol (lib_id "LocalPrjLib:HC-SFP-01L") (at 159.385 76.835 0) (unit 1)
+  (symbol (lib_id "LocalSymbolsPrjLib:HC-SFP-01L") (at 159.385 76.835 0) (unit 1)
     (in_bom yes) (on_board yes) (dnp no)
     (property "Reference" "J9" (at 159.385 61.341 0)
@@
     )
   )
-  (symbol (lib_id "LocalPrjLib:R_Small_US") (at 217.17 140.335 180) (unit 1)
+  (symbol (lib_id "LocalSymbolsPrjLib:R_Small_US") (at 217.17 140.335 180) (unit 1)
     (in_bom no) (on_board yes) (dnp yes)
     (property "Reference" "R4" (at 213.36 139.7 0)
@@
     )
   )
-  (symbol (lib_id "LocalPrjLib:R_Small_US") (at 139.7 133.35 90) (unit 1)
+  (symbol (lib_id "LocalSymbolsPrjLib:R_Small_US") (at 139.7 133.35 90) (unit 1)
     (in_bom yes) (on_board yes) (dnp no)
     (property "Reference" "R4" (at 135.255 132.08 90)
@@
     )
   )
-  (symbol (lib_id "LocalPrjLib:C_Small") (at 78.74 59.69 270) (unit 1)
+  (symbol (lib_id "LocalSymbolsPrjLib:C_Small") (at 78.74 59.69 270) (unit 1)
     (in_bom yes) (on_board yes) (dnp no)
     (property "Reference" "C1" (at 74.93 58.42 90)
@@
     )
   )
-  (symbol (lib_id "LocalPrjLib:HC-SFP-20P") (at 159.385 127 0) (unit 1)
+  (symbol (lib_id "LocalSymbolsPrjLib:HC-SFP-20P") (at 159.385 127 0) (unit 1)
     (in_bom yes) (on_board yes) (dnp no)
     (property "Reference" "S1" (at 159.385 111.506 0)
@@
     )
   )
-  (symbol (lib_id "LocalPrjLib:R_Small_US") (at 217.17 128.905 180) (unit 1)
+  (symbol (lib_id "LocalSymbolsPrjLib:R_Small_US") (at 217.17 128.905 180) (unit 1)
     (in_bom yes) (on_board yes) (dnp no)
     (property "Reference" "R4" (at 213.36 128.27 0)
@@
     )
   )
-  (symbol (lib_id "LocalPrjLib:R_Small_US") (at 198.755 113.03 180) (unit 1)
+  (symbol (lib_id "LocalSymbolsPrjLib:R_Small_US") (at 198.755 113.03 180) (unit 1)
     (in_bom yes) (on_board yes) (dnp no)
     (property "Reference" "R4" (at 194.945 112.395 0)
@@
     )
   )
-  (symbol (lib_id "LocalPrjLib:C_Small") (at 78.74 67.31 270) (unit 1)
+  (symbol (lib_id "LocalSymbolsPrjLib:C_Small") (at 78.74 67.31 270) (unit 1)
     (in_bom yes) (on_board yes) (dnp no)
     (property "Reference" "C1" (at 74.93 66.04 90)
@@
     )
   )
-  (symbol (lib_id "LocalPrjLib:R_Small_US") (at 224.79 140.335 180) (unit 1)
+  (symbol (lib_id "LocalSymbolsPrjLib:R_Small_US") (at 224.79 140.335 180) (unit 1)
     (in_bom no) (on_board yes) (dnp yes)
     (property "Reference" "R4" (at 220.98 139.7 0)
@@
     )
   )
-  (symbol (lib_id "LocalPrjLib:C_Small") (at 66.04 57.15 270) (unit 1)
+  (symbol (lib_id "LocalSymbolsPrjLib:C_Small") (at 66.04 57.15 270) (unit 1)
     (in_bom yes) (on_board yes) (dnp no)
     (property "Reference" "C1" (at 62.23 55.88 90)
@@
     )
   )
-  (symbol (lib_id "LocalPrjLib:R_Small_US") (at 198.755 125.095 180) (unit 1)
+  (symbol (lib_id "LocalSymbolsPrjLib:R_Small_US") (at 198.755 125.095 180) (unit 1)
     (in_bom no) (on_board yes) (dnp yes)
     (property "Reference" "R4" (at 194.945 124.46 0)
@@
     )
   )
-  (symbol (lib_id "LocalPrjLib:R_Small_US") (at 206.375 113.03 180) (unit 1)
+  (symbol (lib_id "LocalSymbolsPrjLib:R_Small_US") (at 206.375 113.03 180) (unit 1)
     (in_bom yes) (on_board yes) (dnp no)
     (property "Reference" "R4" (at 202.565 112.395 0)
@@
     )
   )
-  (symbol (lib_id "LocalPrjLib:R_Small_US") (at 139.7 128.27 90) (unit 1)
+  (symbol (lib_id "LocalSymbolsPrjLib:R_Small_US") (at 139.7 128.27 90) (unit 1)
     (in_bom yes) (on_board yes) (dnp no)
     (property "Reference" "R4" (at 135.255 127 90)
@@
     )
   )
-  (symbol (lib_id "LocalPrjLib:R_Small_US") (at 206.375 125.095 180) (unit 1)
+  (symbol (lib_id "LocalSymbolsPrjLib:R_Small_US") (at 206.375 125.095 180) (unit 1)
     (in_bom no) (on_board yes) (dnp yes)
     (property "Reference" "R4" (at 202.565 124.46 0)

Commit message: Fixes...
Parts:
- renumbered C1 to C166, C1 to C167, C1 to C168, C1 to C169, J9 to J25, R4 to R141, R4 to R142, R4 to R143, R4 to R144, R4 to R145, R4 to R146, R4 to R147, R4 to R148, R4 to R149, R4 to R150, R4 to R151
