File: Tangenta/FANs.kicad_sch (KiCad schematic)
At the start: 8 parts, among them M1 Fan_4pin, M2 Fan_4pin, Q3 BSS138

Commit message: Fixes, new approach.
Parts:
- M1, M2: symbol LocalPrjLib:Fan_4pin -> LocalSymbolsPrjLib:Fan_4pin
- Q3: symbol LocalPrjLib:BSS138 -> LocalSymbolsPrjLib:BSS138
- R2: symbol LocalPrjLib:R_Small_US -> LocalSymbolsPrjLib:R_Small_US
Changed lines of the file:
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@@
     (effects (font (size 1.27 1.27)) (justify right))
   )
-  (symbol (lib_id "LocalPrjLib:R_Small_US") (at 127 111.76 180) (unit 1)
+  (symbol (lib_id "LocalSymbolsPrjLib:R_Small_US") (at 127 111.76 180) (unit 1)
     (in_bom yes) (on_board yes) (dnp no)
     (property "Reference" "R2" (at 125.73 110.49 0)
@@
     )
   )
-  (symbol (lib_id "LocalPrjLib:R_Small_US") (at 127 78.105 180) (unit 1)
+  (symbol (lib_id "LocalSymbolsPrjLib:R_Small_US") (at 127 78.105 180) (unit 1)
     (in_bom yes) (on_board yes) (dnp no)
     (property "Reference" "R2" (at 125.73 76.835 0)
@@
     )
   )
-  (symbol (lib_id "LocalPrjLib:Fan_4pin") (at 181.61 115.57 0) (unit 1)
+  (symbol (lib_id "LocalSymbolsPrjLib:Fan_4pin") (at 181.61 115.57 0) (unit 1)
     (in_bom yes) (on_board yes) (dnp no)
     (property "Reference" "M2" (at 185.42 114.3 0)
@@
     )
   )
-  (symbol (lib_id "LocalPrjLib:BSS138") (at 139.7 115.57 270) (unit 1)
+  (symbol (lib_id "LocalSymbolsPrjLib:BSS138") (at 139.7 115.57 270) (unit 1)
     (in_bom yes) (on_board yes) (dnp no)
     (property "Reference" "Q3" (at 142.24 113.03 90)
@@
     )
   )
-  (symbol (lib_id "LocalPrjLib:R_Small_US") (at 153.67 111.76 180) (unit 1)
+  (symbol (lib_id "LocalSymbolsPrjLib:R_Small_US") (at 153.67 111.76 180) (unit 1)
     (in_bom yes) (on_board yes) (dnp no)
     (property "Reference" "R2" (at 152.4 110.49 0)
@@
     )
   )
-  (symbol (lib_id "LocalPrjLib:R_Small_US") (at 153.67 78.105 180) (unit 1)
+  (symbol (lib_id "LocalSymbolsPrjLib:R_Small_US") (at 153.67 78.105 180) (unit 1)
     (in_bom yes) (on_board yes) (dnp no)
     (property "Reference" "R2" (at 152.4 76.835 0)
@@
     )
   )
-  (symbol (lib_id "LocalPrjLib:Fan_4pin") (at 181.61 81.915 0) (unit 1)
+  (symbol (lib_id "LocalSymbolsPrjLib:Fan_4pin") (at 181.61 81.915 0) (unit 1)
     (in_bom yes) (on_board yes) (dnp no)
     (property "Reference" "M1" (at 185.42 80.645 0)
@@
     )
   )
-  (symbol (lib_id "LocalPrjLib:BSS138") (at 139.7 81.915 270) (unit 1)
+  (symbol (lib_id "LocalSymbolsPrjLib:BSS138") (at 139.7 81.915 270) (unit 1)
     (in_bom yes) (on_board yes) (dnp no)
     (property "Reference" "Q3" (at 142.24 79.375 90)

Commit message: Fixes...
Parts:
- renumbered Q3 to Q23, Q3 to Q24, R2 to R204, R2 to R205, R2 to R206, R2 to R207
