File: Tangenta/PCIE_Slot_2.kicad_sch (KiCad schematic)
At the start: 12 parts, among them J10 1-2199230-5

Commit message: ...
Parts:
- C24: symbol CholaSymbolsPrjLib:CA45-A-6_3V-47UF-K -> LocalPrjLib:CA45-A-6_3V-47UF-K
- H10: symbol CholaSymbolsPrjLib:MountingHole -> LocalPrjLib:MountingHole
- J10: symbol CholaSymbolsPrjLib:1-2199230-5 -> LocalPrjLib:1-2199230-5
- R2: symbol CholaSymbolsPrjLib:R_Small_US -> LocalPrjLib:R_Small_US
- TP3: symbol CholaSymbolsPrjLib:TestPoint_Small -> LocalPrjLib:TestPoint_Small
Changed lines of the file:
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@@
     (effects (font (size 1.27 1.27)) (justify left))
   )
-  (symbol (lib_id "CholaSymbolsPrjLib:MountingHole") (at 163.195 175.26 0) (unit 1)
+  (symbol (lib_id "LocalPrjLib:MountingHole") (at 163.195 175.26 0) (unit 1)
     (in_bom yes) (on_board yes) (dnp no)
     (property "Reference" "H10" (at 165.735 175.26 0)
@@
     )
   )
-  (symbol (lib_id "CholaSymbolsPrjLib:MountingHole") (at 163.195 185.42 0) (unit 1)
+  (symbol (lib_id "LocalPrjLib:MountingHole") (at 163.195 185.42 0) (unit 1)
     (in_bom yes) (on_board yes) (dnp no)
     (property "Reference" "H10" (at 165.735 185.42 0)
@@
     )
   )
-  (symbol (lib_id "CholaSymbolsPrjLib:R_Small_US") (at 161.29 48.26 270) (unit 1)
+  (symbol (lib_id "LocalPrjLib:R_Small_US") (at 161.29 48.26 270) (unit 1)
     (in_bom yes) (on_board yes) (dnp no)
     (property "Reference" "R2" (at 154.305 46.99 90)
@@
     )
   )
-  (symbol (lib_id "CholaSymbolsPrjLib:1-2199230-5") (at 135.89 33.02 90) (mirror x) (unit 1)
+  (symbol (lib_id "LocalPrjLib:1-2199230-5") (at 135.89 33.02 90) (mirror x) (unit 1)
     (in_bom yes) (on_board yes) (dnp no)
     (property "Reference" "J10" (at 128.27 36.83 90)
@@
     )
   )
-  (symbol (lib_id "CholaSymbolsPrjLib:CA45-A-6_3V-47UF-K") (at 140.97 148.59 270) (mirror x) (unit 1)
+  (symbol (lib_id "LocalPrjLib:CA45-A-6_3V-47UF-K") (at 140.97 148.59 270) (mirror x) (unit 1)
     (in_bom yes) (on_board yes) (dnp no)
     (property "Reference" "C24" (at 148.59 147.32 90)
@@
     )
   )
-  (symbol (lib_id "CholaSymbolsPrjLib:MountingHole") (at 163.195 180.34 0) (unit 1)
+  (symbol (lib_id "LocalPrjLib:MountingHole") (at 163.195 180.34 0) (unit 1)
     (in_bom yes) (on_board yes) (dnp no)
     (property "Reference" "H10" (at 165.735 180.34 0)
@@
     )
   )
-  (symbol (lib_id "CholaSymbolsPrjLib:R_Small_US") (at 161.29 45.72 270) (unit 1)
+  (symbol (lib_id "LocalPrjLib:R_Small_US") (at 161.29 45.72 270) (unit 1)
     (in_bom yes) (on_board yes) (dnp no)
     (property "Reference" "R2" (at 154.305 44.45 90)
@@
     )
   )
-  (symbol (lib_id "CholaSymbolsPrjLib:R_Small_US") (at 163.83 91.44 270) (unit 1)
+  (symbol (lib_id "LocalPrjLib:R_Small_US") (at 163.83 91.44 270) (unit 1)
     (in_bom yes) (on_board yes) (dnp no)
     (property "Reference" "R2" (at 156.845 90.17 90)
@@
     )
   )
-  (symbol (lib_id "CholaSymbolsPrjLib:CA45-A-6_3V-47UF-K") (at 130.175 148.59 270) (mirror x) (unit 1)
+  (symbol (lib_id "LocalPrjLib:CA45-A-6_3V-47UF-K") (at 130.175 148.59 270) (mirror x) (unit 1)
     (in_bom yes) (on_board yes) (dnp no)
     (property "Reference" "C24" (at 137.795 147.32 90)
@@
     )
   )
-  (symbol (lib_id "CholaSymbolsPrjLib:TestPoint_Small") (at 113.03 114.3 0) (mirror y) (unit 1)
+  (symbol (lib_id "LocalPrjLib:TestPoint_Small") (at 113.03 114.3 0) (mirror y) (unit 1)
     (in_bom yes) (on_board yes) (dnp no)
     (property "Reference" "TP3" (at 112.395 114.3 0)
@@
     )
   )
-  (symbol (lib_id "CholaSymbolsPrjLib:R_Small_US") (at 163.83 88.9 270) (unit 1)
+  (symbol (lib_id "LocalPrjLib:R_Small_US") (at 163.83 88.9 270) (unit 1)
     (in_bom yes) (on_board yes) (dnp no)
     (property "Reference" "R2" (at 156.845 87.63 90)
@@
     )
   )
-  (symbol (lib_id "CholaSymbolsPrjLib:R_Small_US") (at 34.29 45.72 270) (unit 1)
+  (symbol (lib_id "LocalPrjLib:R_Small_US") (at 34.29 45.72 270) (unit 1)
     (in_bom yes) (on_board yes) (dnp no)
     (property "Reference" "R2" (at 28.575 44.45 90)

Commit message: Fixes, new approach.
Parts:
- C24: symbol LocalPrjLib:CA45-A-6_3V-47UF-K -> LocalSymbolsPrjLib:CA45-A-6_3V-47UF-K
- H10: symbol LocalPrjLib:MountingHole -> LocalSymbolsPrjLib:MountingHole
- J10: symbol LocalPrjLib:1-2199230-5 -> LocalSymbolsPrjLib:1-2199230-5
- R2: symbol LocalPrjLib:R_Small_US -> LocalSymbolsPrjLib:R_Small_US
- TP3: symbol LocalPrjLib:TestPoint_Small -> LocalSymbolsPrjLib:TestPoint_Small
Changed lines of the file:
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@@
     (effects (font (size 1.27 1.27)) (justify left))
   )
-  (symbol (lib_id "LocalPrjLib:MountingHole") (at 163.195 175.26 0) (unit 1)
+  (symbol (lib_id "LocalSymbolsPrjLib:MountingHole") (at 163.195 175.26 0) (unit 1)
     (in_bom yes) (on_board yes) (dnp no)
     (property "Reference" "H10" (at 165.735 175.26 0)
@@
     )
   )
-  (symbol (lib_id "LocalPrjLib:MountingHole") (at 163.195 185.42 0) (unit 1)
+  (symbol (lib_id "LocalSymbolsPrjLib:MountingHole") (at 163.195 185.42 0) (unit 1)
     (in_bom yes) (on_board yes) (dnp no)
     (property "Reference" "H10" (at 165.735 185.42 0)
@@
     )
   )
-  (symbol (lib_id "LocalPrjLib:R_Small_US") (at 161.29 48.26 270) (unit 1)
+  (symbol (lib_id "LocalSymbolsPrjLib:R_Small_US") (at 161.29 48.26 270) (unit 1)
     (in_bom yes) (on_board yes) (dnp no)
     (property "Reference" "R2" (at 154.305 46.99 90)
@@
     )
   )
-  (symbol (lib_id "LocalPrjLib:1-2199230-5") (at 135.89 33.02 90) (mirror x) (unit 1)
+  (symbol (lib_id "LocalSymbolsPrjLib:1-2199230-5") (at 135.89 33.02 90) (mirror x) (unit 1)
     (in_bom yes) (on_board yes) (dnp no)
     (property "Reference" "J10" (at 128.27 36.83 90)
@@
     )
   )
-  (symbol (lib_id "LocalPrjLib:CA45-A-6_3V-47UF-K") (at 140.97 148.59 270) (mirror x) (unit 1)
+  (symbol (lib_id "LocalSymbolsPrjLib:CA45-A-6_3V-47UF-K") (at 140.97 148.59 270) (mirror x) (unit 1)
     (in_bom yes) (on_board yes) (dnp no)
     (property "Reference" "C24" (at 148.59 147.32 90)
@@
     )
   )
-  (symbol (lib_id "LocalPrjLib:MountingHole") (at 163.195 180.34 0) (unit 1)
+  (symbol (lib_id "LocalSymbolsPrjLib:MountingHole") (at 163.195 180.34 0) (unit 1)
     (in_bom yes) (on_board yes) (dnp no)
     (property "Reference" "H10" (at 165.735 180.34 0)
@@
     )
   )
-  (symbol (lib_id "LocalPrjLib:R_Small_US") (at 161.29 45.72 270) (unit 1)
+  (symbol (lib_id "LocalSymbolsPrjLib:R_Small_US") (at 161.29 45.72 270) (unit 1)
     (in_bom yes) (on_board yes) (dnp no)
     (property "Reference" "R2" (at 154.305 44.45 90)
@@
     )
   )
-  (symbol (lib_id "LocalPrjLib:R_Small_US") (at 163.83 91.44 270) (unit 1)
+  (symbol (lib_id "LocalSymbolsPrjLib:R_Small_US") (at 163.83 91.44 270) (unit 1)
     (in_bom yes) (on_board yes) (dnp no)
     (property "Reference" "R2" (at 156.845 90.17 90)
@@
     )
   )
-  (symbol (lib_id "LocalPrjLib:CA45-A-6_3V-47UF-K") (at 130.175 148.59 270) (mirror x) (unit 1)
+  (symbol (lib_id "LocalSymbolsPrjLib:CA45-A-6_3V-47UF-K") (at 130.175 148.59 270) (mirror x) (unit 1)
     (in_bom yes) (on_board yes) (dnp no)
     (property "Reference" "C24" (at 137.795 147.32 90)
@@
     )
   )
-  (symbol (lib_id "LocalPrjLib:TestPoint_Small") (at 113.03 114.3 0) (mirror y) (unit 1)
+  (symbol (lib_id "LocalSymbolsPrjLib:TestPoint_Small") (at 113.03 114.3 0) (mirror y) (unit 1)
     (in_bom yes) (on_board yes) (dnp no)
     (property "Reference" "TP3" (at 112.395 114.3 0)
@@
     )
   )
-  (symbol (lib_id "LocalPrjLib:R_Small_US") (at 163.83 88.9 270) (unit 1)
+  (symbol (lib_id "LocalSymbolsPrjLib:R_Small_US") (at 163.83 88.9 270) (unit 1)
     (in_bom yes) (on_board yes) (dnp no)
     (property "Reference" "R2" (at 156.845 87.63 90)
@@
     )
   )
-  (symbol (lib_id "LocalPrjLib:R_Small_US") (at 34.29 45.72 270) (unit 1)
+  (symbol (lib_id "LocalSymbolsPrjLib:R_Small_US") (at 34.29 45.72 270) (unit 1)
     (in_bom yes) (on_board yes) (dnp no)
     (property "Reference" "R2" (at 28.575 44.45 90)

Commit message: Fixes...
Parts:
- renumbered C24 to C112, C24 to C113, H10 to H16, H10 to H17, H10 to H18, J10 to J19, R2 to R83, R2 to R84, R2 to R85, R2 to R86, R2 to R87, TP3 to TP2
